File: clock.sch (KiCad schematic (older format))
At the start: 20 parts, among them SW1 SW_Push, SW2 SW_SPDT, U23 LM555xN, U24 74LS04, U25 74LS08, U26 74LS32, U27 LM555xN, U28 LM555xN

Commit message: Fixed ZIF
Parts:
- C1, C3, C4, C5: symbol Device:C -> 16bitCpu-rescue:C-Device
- C2: symbol Device:CP -> 16bitCpu-rescue:CP-Device
- R1, R2, R3, R4, R5, R6: symbol Device:R -> 16bitCpu-rescue:R-Device
- RV1: symbol Device:R_POT -> 16bitCpu-rescue:R_POT-Device
- SW1: symbol Switch:SW_Push -> 16bitCpu-rescue:SW_Push-Switch
- SW2: symbol Switch:SW_SPDT -> 16bitCpu-rescue:SW_SPDT-Switch
- U23, U27, U28: symbol Timer:LM555xN -> 16bitCpu-rescue:LM555xN-Timer
- U24: symbol 74xx:74LS04 -> 16bitCpu-rescue:74LS04-74xx
- U25: symbol 74xx:74LS08 -> 16bitCpu-rescue:74LS08-74xx
- U26: symbol 74xx:74LS32 -> 16bitCpu-rescue:74LS32-74xx
Changed lines of the file:
@@
 $EndDescr
 $Comp
-L power:+5V #PWR078
+L 16bitCpu-rescue:+5V-power #PWR078
 U 1 1 5F76260D
 P 2700 1100
+AR Path="/5F76260D" Ref="#PWR078"  Part="1"
+AR Path="/5F75E433/5F76260D" Ref="#PWR078"  Part="1"
 F 0 "#PWR078" H 2700 950 50  0001 C CNN
 F 1 "+5V" H 2715 1273 50  0000 C CNN
@@
 $EndComp
 $Comp
-L power:GND #PWR082
+L 16bitCpu-rescue:GND-power #PWR082
 U 1 1 5F763381
 P 5750 2700
+AR Path="/5F763381" Ref="#PWR082"  Part="1"
+AR Path="/5F75E433/5F763381" Ref="#PWR082"  Part="1"
 F 0 "#PWR082" H 5750 2450 50  0001 C CNN
 F 1 "GND" H 5755 2527 50  0000 C CNN
@@
 $EndComp
 $Comp
-L power:GND #PWR077
+L 16bitCpu-rescue:GND-power #PWR077
 U 1 1 5F7634B3
 P 2450 2650
+AR Path="/5F7634B3" Ref="#PWR077"  Part="1"
+AR Path="/5F75E433/5F7634B3" Ref="#PWR077"  Part="1"
 F 0 "#PWR077" H 2450 2400 50  0001 C CNN
 F 1 "GND" H 2455 2477 50  0000 C CNN
@@
 $EndComp
 $Comp
-L Device:R R1
+L 16bitCpu-rescue:R-Device R1
 U 1 1 5F763CA2
 P 3350 1350
+AR Path="/5F763CA2" Ref="R1"  Part="1"
+AR Path="/5F75E433/5F763CA2" Ref="R1"  Part="1"
 F 0 "R1" H 3420 1396 50  0000 L CNN
 F 1 "1K" H 3420 1305 50  0000 L CNN
@@
 	3350 1900 3350 1850
 $Comp
-L Device:R R2
+L 16bitCpu-rescue:R-Device R2
 U 1 1 5F76554D
 P 3550 2000
+AR Path="/5F76554D" Ref="R2"  Part="1"
+AR Path="/5F75E433/5F76554D" Ref="R2"  Part="1"
 F 0 "R2" H 3620 2046 50  0000 L CNN
 F 1 "1K" H 3620 1955 50  0000 L CNN
@@
 	3350 1850 3350 1500
 $Comp
-L Device:R_POT RV1
+L 16bitCpu-rescue:R_POT-Device RV1
 U 1 1 5F766089
 P 3800 2150
+AR Path="/5F766089" Ref="RV1"  Part="1"
+AR Path="/5F75E433/5F766089" Ref="RV1"  Part="1"
 F 0 "RV1" H 3730 2104 50  0000 R CNN
 F 1 "1M" H 3730 2195 50  0000 R CNN
@@
 Connection ~ 3400 2300
 $Comp
-L Device:C C1
+L 16bitCpu-rescue:C-Device C1
 U 1 1 5F768F08
 P 1600 2500
+AR Path="/5F768F08" Ref="C1"  Part="1"
+AR Path="/5F75E433/5F768F08" Ref="C1"  Part="1"
 F 0 "C1" H 1715 2546 50  0000 L CNN
 F 1 "0.01uF" H 1715 2455 50  0000 L CNN
@@
 	1800 2350 1800 1700
 $Comp
-L Device:CP C2
+L 16bitCpu-rescue:CP-Device C2
 U 1 1 5F76B50A
 P 2050 2500
+AR Path="/5F76B50A" Ref="C2"  Part="1"
+AR Path="/5F75E433/5F76B50A" Ref="C2"  Part="1"
 F 0 "C2" H 2168 2546 50  0000 L CNN
 F 1 "1uF" H 2168 2455 50  0000 L CNN
@@
 Connection ~ 2450 2650
 $Comp
-L power:+5V #PWR081
+L 16bitCpu-rescue:+5V-power #PWR081
 U 1 1 5F76F8D8
 P 5750 1150
+AR Path="/5F76F8D8" Ref="#PWR081"  Part="1"
+AR Path="/5F75E433/5F76F8D8" Ref="#PWR081"  Part="1"
 F 0 "#PWR081" H 5750 1000 50  0001 C CNN
 F 1 "+5V" H 5765 1323 50  0000 C CNN
@@
 	5750 1250 5750 1400
 $Comp
-L Device:R R4
+L 16bitCpu-rescue:R-Device R4
 U 1 1 5F771810
 P 6400 1500
+AR Path="/5F771810" Ref="R4"  Part="1"
+AR Path="/5F75E433/5F771810" Ref="R4"  Part="1"
 F 0 "R4" H 6470 1546 50  0000 L CNN
 F 1 "1M" H 6470 1455 50  0000 L CNN
@@
 Connection ~ 6400 1900
 $Comp
-L Device:C C4
+L 16bitCpu-rescue:C-Device C4
 U 1 1 5F772B51
 P 6400 2350
+AR Path="/5F772B51" Ref="C4"  Part="1"
+AR Path="/5F75E433/5F772B51" Ref="C4"  Part="1"
 F 0 "C4" H 6515 2396 50  0000 L CNN
 F 1 "0.1uF" H 6515 2305 50  0000 L CNN
@@
 	5750 2600 5750 2300
 $Comp
-L Device:C C3
+L 16bitCpu-rescue:C-Device C3
 U 1 1 5F7757C1
 P 5100 2450
+AR Path="/5F7757C1" Ref="C3"  Part="1"
+AR Path="/5F75E433/5F7757C1" Ref="C3"  Part="1"
 F 0 "C3" H 5215 2496 50  0000 L CNN
 F 1 "0.01uF" H 5215 2405 50  0000 L CNN
@@
 	5250 1700 5050 1700
 $Comp
-L Device:R R3
+L 16bitCpu-rescue:R-Device R3
 U 1 1 5F778F11
 P 5050 1550
+AR Path="/5F778F11" Ref="R3"  Part="1"
+AR Path="/5F75E433/5F778F11" Ref="R3"  Part="1"
 F 0 "R3" H 5120 1596 50  0000 L CNN
 F 1 "1K" H 5120 1505 50  0000 L CNN
@@
 	5200 1400 5750 1400
 $Comp
-L Switch:SW_Push SW1
+L 16bitCpu-rescue:SW_Push-Switch SW1
 U 1 1 5F77C300
 P 4800 1700
+AR Path="/5F77C300" Ref="SW1"  Part="1"
+AR Path="/5F75E433/5F77C300" Ref="SW1"  Part="1"
 F 0 "SW1" H 4800 1985 50  0000 C CNN
 F 1 "SW_Push" H 4800 1894 50  0000 C CNN
@@
 Connection ~ 5050 1700
 $Comp
-L power:GND #PWR084
+L 16bitCpu-rescue:GND-power #PWR084
 U 1 1 5F785279
 P 8450 2700
+AR Path="/5F785279" Ref="#PWR084"  Part="1"
+AR Path="/5F75E433/5F785279" Ref="#PWR084"  Part="1"
 F 0 "#PWR084" H 8450 2450 50  0001 C CNN
 F 1 "GND" H 8455 2527 50  0000 C CNN
@@
 $EndComp
 $Comp
-L power:+5V #PWR083
+L 16bitCpu-rescue:+5V-power #PWR083
 U 1 1 5F78527F
 P 8450 1150
+AR Path="/5F78527F" Ref="#PWR083"  Part="1"
+AR Path="/5F75E433/5F78527F" Ref="#PWR083"  Part="1"
 F 0 "#PWR083" H 8450 1000 50  0001 C CNN
 F 1 "+5V" H 8465 1323 50  0000 C CNN
@@
 	8450 2600 8450 2300
 $Comp
-L Device:C C5
+L 16bitCpu-rescue:C-Device C5
 U 1 1 5F7852A0
 P 7800 2450
+AR Path="/5F7852A0" Ref="C5"  Part="1"
+AR Path="/5F75E433/5F7852A0" Ref="C5"  Part="1"
 F 0 "C5" H 7915 2496 50  0000 L CNN
 F 1 "0.01uF" H 7915 2405 50  0000 L CNN
@@
 Connection ~ 7800 2600
 $Comp
-L Device:R R5
+L 16bitCpu-rescue:R-Device R5
 U 1 1 5F7852AF
 P 7750 1400
+AR Path="/5F7852AF" Ref="R5"  Part="1"
+AR Path="/5F75E433/5F7852AF" Ref="R5"  Part="1"
 F 0 "R5" H 7820 1446 50  0000 L CNN
 F 1 "1K" H 7820 1355 50  0000 L CNN
@@
 	8450 1150 8450 1250
 $Comp
-L Switch:SW_SPDT SW2
+L 16bitCpu-rescue:SW_SPDT-Switch SW2
 U 1 1 5F79CC11
 P 7500 1900
+AR Path="/5F79CC11" Ref="SW2"  Part="1"
+AR Path="/5F75E433/5F79CC11" Ref="SW2"  Part="1"
 F 0 "SW2" H 7500 2185 50  0000 C CNN
 F 1 "SW_SPDT" H 7500 2094 50  0000 C CNN
@@
 	7750 1250 7900 1250
 $Comp
-L Device:R R6
+L 16bitCpu-rescue:R-Device R6
 U 1 1 5F7A4B09
 P 7900 1400
+AR Path="/5F7A4B09" Ref="R6"  Part="1"
+AR Path="/5F75E433/5F7A4B09" Ref="R6"  Part="1"
 F 0 "R6" H 7970 1446 50  0000 L CNN
 F 1 "1K" H 7970 1355 50  0000 L CNN
@@
 	7900 2100 7950 2100
 $Comp
-L 74xx:74LS08 U25
+L 16bitCpu-rescue:74LS08-74xx U25
 U 1 1 5F7BE3EA
 P 3600 4100
+AR Path="/5F7BE3EA" Ref="U25"  Part="1"
+AR Path="/5F75E433/5F7BE3EA" Ref="U25"  Part="1"
 F 0 "U25" H 3600 4425 50  0000 C CNN
 F 1 "74LS08" H 3600 4334 50  0000 C CNN
@@
 $EndComp
 $Comp
-L 74xx:74LS08 U25
+L 16bitCpu-rescue:74LS08-74xx U25
 U 2 1 5F7C112B
 P 3600 4650
+AR Path="/5F7C112B" Ref="U25"  Part="2"
+AR Path="/5F75E433/5F7C112B" Ref="U25"  Part="2"
 F 0 "U25" H 3600 4975 50  0000 C CNN
 F 1 "74LS08" H 3600 4884 50  0000 C CNN
@@
 $EndComp
 $Comp
-L 74xx:74LS08 U25
+L 16bitCpu-rescue:74LS08-74xx U25
 U 3 1 5F7C255C
 P 6400 4500
+AR Path="/5F7C255C" Ref="U25"  Part="3"
+AR Path="/5F75E433/5F7C255C" Ref="U25"  Part="3"
 F 0 "U25" H 6400 4825 50  0000 C CNN
 F 1 "74LS08" H 6400 4734 50  0000 C CNN
@@
 $EndComp
 $Comp
-L 74xx:74LS32 U26
+L 16bitCpu-rescue:74LS32-74xx U26
 U 1 1 5F7C6F12
 P 5250 4400
+AR Path="/5F7C6F12" Ref="U26"  Part="1"
+AR Path="/5F75E433/5F7C6F12" Ref="U26"  Part="1"
 F 0 "U26" H 5250 4725 50  0000 C CNN
 F 1 "74LS32" H 5250 4634 50  0000 C CNN
@@
 	3300 3600 3300 4000
 $Comp
-L 74xx:74LS04 U24
+L 16bitCpu-rescue:74LS04-74xx U24
 U 1 1 5F7CE7FD
 P 2700 4550
+AR Path="/5F7CE7FD" Ref="U24"  Part="1"
+AR Path="/5F75E433/5F7CE7FD" Ref="U24"  Part="1"
 F 0 "U24" H 2700 4867 50  0000 C CNN
 F 1 "74LS04" H 2700 4776 50  0000 C CNN
@@
 $EndComp
 $Comp
-L 74xx:74LS04 U24
+L 16bitCpu-rescue:74LS04-74xx U24
 U 2 1 5F7D01D9
 P 3600 5550
+AR Path="/5F7D01D9" Ref="U24"  Part="2"
+AR Path="/5F75E433/5F7D01D9" Ref="U24"  Part="2"
 F 0 "U24" H 3600 5867 50  0000 C CNN
 F 1 "74LS04" H 3600 5776 50  0000 C CNN
@@
 $EndComp
 $Comp
-L 74xx:74LS04 U24
+L 16bitCpu-rescue:74LS04-74xx U24
 U 3 1 5F7D1AFC
 P 7900 3950
+AR Path="/5F7D1AFC" Ref="U24"  Part="3"
+AR Path="/5F75E433/5F7D1AFC" Ref="U24"  Part="3"
 F 0 "U24" H 7900 4267 50  0000 C CNN
 F 1 "74LS04" H 7900 4176 50  0000 C CNN
@@
 Connection ~ 5150 6750
 $Comp
-L power:+5V #PWR079
+L 16bitCpu-rescue:+5V-power #PWR079
 U 1 1 6081D7D4
 P 5150 5750
+AR Path="/6081D7D4" Ref="#PWR079"  Part="1"
+AR Path="/5F75E433/6081D7D4" Ref="#PWR079"  Part="1"
 F 0 "#PWR079" H 5150 5600 50  0001 C CNN
 F 1 "+5V" H 5165 5923 50  0000 C CNN
@@
 $EndComp
 $Comp
-L power:GND #PWR080
+L 16bitCpu-rescue:GND-power #PWR080
 U 1 1 6081E349
 P 5150 6750
+AR Path="/6081E349" Ref="#PWR080"  Part="1"
+AR Path="/5F75E433/6081E349" Ref="#PWR080"  Part="1"
 F 0 "#PWR080" H 5150 6500 50  0001 C CNN
 F 1 "GND" H 5155 6577 50  0000 C CNN
@@
 $EndComp
 $Comp
-L 74xx:74LS04 U24
+L 16bitCpu-rescue:74LS04-74xx U24
 U 7 1 6085491F
 P 4650 6250
+AR Path="/6085491F" Ref="U24"  Part="7"
+AR Path="/5F75E433/6085491F" Ref="U24"  Part="7"
 F 0 "U24" H 4421 6296 50  0000 R CNN
 F 1 "74LS04" H 4421 6205 50  0000 R CNN
@@
 $EndComp
 $Comp
-L 74xx:74LS08 U25
+L 16bitCpu-rescue:74LS08-74xx U25
 U 5 1 6085870D
 P 5150 6250
+AR Path="/6085870D" Ref="U25"  Part="5"
+AR Path="/5F75E433/6085870D" Ref="U25"  Part="5"
 F 0 "U25" H 5380 6296 50  0000 L CNN
 F 1 "74LS08" H 5380 6205 50  0000 L CNN
@@
 $EndComp
 $Comp
-L 74xx:74LS32 U26
+L 16bitCpu-rescue:74LS32-74xx U26
 U 5 1 608654F6
 P 5650 6250
+AR Path="/608654F6" Ref="U26"  Part="5"
+AR Path="/5F75E433/608654F6" Ref="U26"  Part="5"
 F 0 "U26" H 5880 6296 50  0000 L CNN
 F 1 "74LS32" H 5880 6205 50  0000 L CNN
@@
 $EndComp
 $Comp
-L Timer:LM555xN U23
+L 16bitCpu-rescue:LM555xN-Timer U23
 U 1 1 60AA52FF
 P 2700 1900
+AR Path="/60AA52FF" Ref="U23"  Part="1"
+AR Path="/5F75E433/60AA52FF" Ref="U23"  Part="1"
 F 0 "U23" H 2700 2481 50  0000 C CNN
 F 1 "LM555xN" H 2700 2390 50  0000 C CNN
@@
 	1600 1900 1600 2350
 $Comp
-L Timer:LM555xN U27
+L 16bitCpu-rescue:LM555xN-Timer U27
 U 1 1 60AB8137
 P 5750 1900
+AR Path="/60AB8137" Ref="U27"  Part="1"
+AR Path="/5F75E433/60AB8137" Ref="U27"  Part="1"
 F 0 "U27" H 5750 2481 50  0000 C CNN
 F 1 "LM555xN" H 5750 2390 50  0000 C CNN
@@
 $EndComp
 $Comp
-L Timer:LM555xN U28
+L 16bitCpu-rescue:LM555xN-Timer U28
 U 1 1 60AB9E78
 P 8450 1900
+AR Path="/60AB9E78" Ref="U28"  Part="1"
+AR Path="/5F75E433/60AB9E78" Ref="U28"  Part="1"
 F 0 "U28" H 8450 2481 50  0000 C CNN
 F 1 "LM555xN" H 8450 2390 50  0000 C CNN
