File: resgisterx.sch (KiCad schematic (older format))
At the start: 6 parts, among them U11 74LS245, U12 74LS173, U13 74LS173, U14 74LS245, U15 74LS173, U16 74LS173

Commit message: Added X register
Connections:
- net labels added: ~XI, ~XO
- net labels removed: GND-power, ~SI, ~SO
