File: 16bitCpu.kicad_pcb (KiCad board)
At the start: 4 copper layers, 73 parts, among them SW1 SW_Push, SW2 SW_SPDT, U1 74LS245, U10 74LS86, U11 74LS245, U12 74LS173, U13 74LS173, U14 74LS245, U15 74LS173, U16 74LS173, U17 74LS245, U18 74LS173, U19 74LS173, U2 74LS245, U20 74LS245, U21 74LS173, U22 74LS173, U23 LM555xN, U24 74LS04, U25 74LS08, U26 74LS32, U27 LM555xN, U28 LM555xN, U29 74LS245, U3 74LS283, U30 74LS245, U31 74LS161, U32 74LS161, U33 74LS161, U34 74LS161, U35 74HC00, U36 74LS245, U37 74HC04, U38 74LS173, U39 74LS173, U4 74LS283, U40 74LS245, U41 74LS173, U42 74LS173, U43 AS6C6264, U44 AS6C6264, U45 AT28C64B-15PU, U46 AT28C64B-15PU, U47 74LS245, U48 74LS173, U49 74LS173, U5 74LS283, U50 74LS245, U51 74LS173, U52 74LS173, U53 74LS173, U54 74HC02, U55 74HC02, U56 74LS08, U57 74LS08, U6 74LS283, U7 74LS86, U8 74LS86, U9 74LS86

Commit message: made the CU , need to change the IR
Parts:
- added R8: 1K, Resistor_THT:R_Axial_DIN0204_L3.6mm_D1.6mm_P7.62mm_Horizontal, F.Cu at (185.3, 209.0)
- added SW3: SW_Push-Switch, Button_Switch_THT:SW_PUSH-12mm, F.Cu at (186.7, 191.8)
- added U58: 7400, Package_DIP:DIP-14_W7.62mm, F.Cu at (185.5, 212.4)
- added U62: 74LS161-74xx, Package_DIP:DIP-16_W7.62mm, F.Cu at (185.5, 231.5)
- added U63: AT28C64B-15PU, ROM:ZIF-AT28C64B-15PU, F.Cu at (171.9, 219.7)
- added U64: AT28C64B-15PU, ROM:ZIF-AT28C64B-15PU, F.Cu at (146.6, 219.7)
- added U65: AT28C64B-15PU, ROM:ZIF-AT28C64B-15PU, F.Cu at (121.3, 219.7)
- moved U46 159.2 mm to (-1.26, 222.2)
- moved SW1 146.7 mm to (20.6, 128.0)
- moved R1 130.9 mm to (36.6, 88.0)
- moved R2 130.9 mm to (36.6, 90.8)
- moved R3 130.9 mm to (36.6, 93.7)
- moved C3 125.8 mm to (47.5, 91.2)
- moved C4 125.8 mm to (47.5, 97.4)
- moved C5 125.8 mm to (47.5, 103.7)
- moved R5 111.7 mm to (65.4, 83.1), turned to 0 degrees
- moved C2 110.2 mm to (47.5, 84.9)
- moved U45 108.8 mm to (24.1, 222.2)
- moved R6 104.0 mm to (65.4, 97.2)
- moved U29 102.0 mm to (76.2, 53.3)
- moved RV1 100.2 mm to (66.3, 91.8)
- moved SW2 99.4 mm to (65.5, 102.6)
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Connections:
- net /ALU/SU renamed /Control Unit/ALU_SU
- net /ALU/~EO renamed /Control Unit/~ALU_EO
- net /ALU/~FI renamed /Control Unit/~ALU_FI
- U53 pad 16: Net-(U53-Pad16) -> +5V
- U53 pad 8: Net-(U53-Pad8) -> GND
Routing:
- net /ALU/BUS0: track 1.59 -> 0.00 mm
- net /ALU/BUS3: track 1.59 -> 0.00 mm
- net /ALU/BUS2: track 1.59 -> 0.00 mm
- net /ALU/BUS1: track 1.59 -> 0.00 mm

Commit message: back to 13 bit addresses
Parts:
- added U59: 74LS245, Package_DIP:DIP-20_W7.62mm, F.Cu at (77.2, 41.4)
- added U60: 74LS173, Package_DIP:DIP-16_W7.62mm, F.Cu at (99.7, 46.5)
- added U61: 74LS173, Package_DIP:DIP-16_W7.62mm, F.Cu at (99.7, 24.2)
- added U66: 74LS245, Package_DIP:DIP-20_W7.62mm, F.Cu at (65.9, 41.4)
- added U67: 74LS173, Package_DIP:DIP-16_W7.62mm, F.Cu at (88.4, 24.2)
- added U68: 74LS173, Package_DIP:DIP-16_W7.62mm, F.Cu at (88.4, 46.5)
- added U69: 74LS245, Package_DIP:DIP-20_W7.62mm, F.Cu at (-44.2, 48.9)
- added U70: 74LS173, Package_DIP:DIP-16_W7.62mm, F.Cu at (-21.7, 54.0)
- added U71: 74LS173, Package_DIP:DIP-16_W7.62mm, F.Cu at (-21.7, 31.7)
- added U72: 74LS245, Package_DIP:DIP-20_W7.62mm, F.Cu at (-55.5, 48.9)
- added U73: 74LS173, Package_DIP:DIP-16_W7.62mm, F.Cu at (-32.9, 31.7)
- added U74: 74LS173, Package_DIP:DIP-16_W7.62mm, F.Cu at (-32.9, 54.0)
- moved U31 150.7 mm to (195.2, 141.5)
- moved U18 148.6 mm to (217.0, 262.8)
- moved U48 131.9 mm to (172.7, 46.5)
- moved U32 127.9 mm to (195.2, 119.2)
- moved U34 127.8 mm to (183.9, 141.5)
- moved U29 127.3 mm to (172.7, 136.4)
- moved U30 126.7 mm to (161.4, 136.4)
- moved U22 124.6 mm to (205.7, 262.8)
- moved U17 124.4 mm to (194.5, 257.7)
- moved U20 124.2 mm to (183.2, 257.7)
- moved U19 124.1 mm to (217.0, 240.5)
- moved U49 121.7 mm to (172.7, 24.2)
- moved U52 120.9 mm to (161.4, 46.5)
- moved U47 120.2 mm to (150.2, 41.4)
- moved U50 119.5 mm to (138.9, 41.4)
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Connections:
- net /RAM/A13 renamed Net-(U40-Pad7)
- net /sheet5F747766/A0 renamed /Register B/A0
- net /sheet5F747766/A1 renamed /Register B/A1
- net /sheet5F747766/A10 renamed /Register B/A10
- net /sheet5F747766/A11 renamed /Register B/A11
- net /sheet5F747766/A12 renamed /Register B/A12
- net /sheet5F747766/A13 renamed /Register B/A13
- net /sheet5F747766/A14 renamed /Register B/A14
- net /sheet5F747766/A15 renamed /Register B/A15
- net /sheet5F747766/A2 renamed /Register B/A2
- net /sheet5F747766/A3 renamed /Register B/A3
- net /sheet5F747766/A4 renamed /Register B/A4
- net /sheet5F747766/A5 renamed /Register B/A5
- net /sheet5F747766/A6 renamed /Register B/A6
- net /sheet5F747766/A7 renamed /Register B/A7
- net /sheet5F747766/A8 renamed /Register B/A8
- net /sheet5F747766/A9 renamed /Register B/A9
- net /sheet5F747766/CLR renamed /Register B/CLR
- net /sheet5F747766/~AI renamed /Register B/~AI
- net /sheet5F747766/~AO renamed /Register B/~AO
- U24 pad 5: /ALU/CLK -> /Control Unit/CLK
- U25 pad 8: /ALU/CLK -> /Control Unit/CLK
- U37 pad 1: /ALU/CLK -> /Control Unit/CLK
- U38 pad 7: /ALU/CLK -> /Control Unit/CLK
- U39 pad 7: /ALU/CLK -> /Control Unit/CLK
- U40 pad 8: /RAM/A14 -> Net-(U40-Pad8)
- U40 pad 9: /RAM/A15 -> Net-(U40-Pad9)
- U41 pad 7: /ALU/CLK -> /Control Unit/CLK
- U42 pad 5: /RAM/A14 -> GND
- U42 pad 6: /RAM/A15 -> GND
- U42 pad 7: /ALU/CLK -> /Control Unit/CLK
- U48 pad 7: /ALU/CLK -> /Control Unit/CLK
- U49 pad 7: /ALU/CLK -> /Control Unit/CLK
- U51 pad 7: /ALU/CLK -> /Control Unit/CLK
- U52 pad 13: Net-(U52-Pad13) -> /ALU/BUS13
- U52 pad 14: Net-(U52-Pad14) -> /ALU/BUS12
- U52 pad 7: /ALU/CLK -> /Control Unit/CLK
- U62 pad 2: /ALU/CLK -> /Control Unit/CLK
- U63 pad 13: Net-(U63-Pad13) -> /Control Unit/~SI
- U63 pad 15: Net-(U63-Pad15) -> /Control Unit/~SO
- U63 pad 16: Net-(U63-Pad16) -> /Control Unit/~XI
- U63 pad 17: Net-(U63-Pad17) -> /Control Unit/~XO
- U65 pad 16: /Control Unit/~IR_AO -> /Instruction Register/~I0
- U65 pad 17: /Instruction Register/~I0 -> /Control Unit/~IR_8O

Commit message: Let there be light
Parts:
- added D1: LED, LED_THT:LED_D3.0mm, F.Cu at (-77.3, 397.6)
- added D10: LED, LED_THT:LED_D3.0mm, F.Cu at (-83.6, 403.6)
- added D100: LED, LED_THT:LED_D3.0mm, F.Cu at (-356.4, 738.6)
- added D101: LED, LED_THT:LED_D3.0mm, F.Cu at (-356.4, 744.5)
- added D102: LED, LED_THT:LED_D3.0mm, F.Cu at (-356.4, 750.5)
- added D103: LED, LED_THT:LED_D3.0mm, F.Cu at (-356.4, 716.3)
- added D104: LED, LED_THT:LED_D3.0mm, F.Cu at (-356.4, 722.2)
- added D105: LED, LED_THT:LED_D3.0mm, F.Cu at (-356.4, 728.2)
- added D106: LED, LED_THT:LED_D3.0mm, F.Cu at (-356.7, 704.8)
- added D107: LED, LED_THT:LED_D3.0mm, F.Cu at (-356.7, 697.7)
- added D108: LED, LED_THT:LED_D3.0mm, F.Cu at (-356.7, 690.6)
- added D109: LED, LED_THT:LED_D3.0mm, F.Cu at (-356.7, 683.5)
- added D11: LED, LED_THT:LED_D3.0mm, F.Cu at (-72.6, 403.6)
- added D110: LED, LED_THT:LED_D3.0mm, F.Cu at (-356.7, 676.4)
- added D111: LED, LED_THT:LED_D3.0mm, F.Cu at (-356.7, 669.3)
- added D112: LED, LED_THT:LED_D3.0mm, F.Cu at (-356.7, 662.2)
- added D113: LED, LED_THT:LED_D3.0mm, F.Cu at (-445.8, 661.6)
- added D114: LED, LED_THT:LED_D3.0mm, F.Cu at (-376.2, 665.1)
- added D115: LED, LED_THT:LED_D3.0mm, F.Cu at (-376.2, 671.1)
- added D116: LED, LED_THT:LED_D3.0mm, F.Cu at (-445.8, 667.5)
- added D117: LED, LED_THT:LED_D3.0mm, F.Cu at (-428.5, 664.0)
- added D118: LED, LED_THT:LED_D3.0mm, F.Cu at (-434.8, 664.0)
- added D119: LED, LED_THT:LED_D3.0mm, F.Cu at (-348.9, 397.6)
- added D12: LED, LED_THT:LED_D3.0mm, F.Cu at (-61.6, 404.7)
- added D120: LED, LED_THT:LED_D3.0mm, F.Cu at (-355.2, 397.6)
- added D121: LED, LED_THT:LED_D3.0mm, F.Cu at (-333.3, 398.8)
- added D122: LED, LED_THT:LED_D3.0mm, F.Cu at (-327.0, 398.8)
- added D123: LED, LED_THT:LED_D3.0mm, F.Cu at (-327.0, 432.0)
- added D124: LED, LED_THT:LED_D3.0mm, F.Cu at (-327.0, 426.0)
- added D125: LED, LED_THT:LED_D3.0mm, F.Cu at (-327.0, 414.1)
- added D126: LED, LED_THT:LED_D3.0mm, F.Cu at (-327.0, 420.1)
- added D127: LED, LED_THT:LED_D3.0mm, F.Cu at (-327.0, 404.7)
- added D128: LED, LED_THT:LED_D3.0mm, F.Cu at (-355.2, 403.6)
- added D129: LED, LED_THT:LED_D3.0mm, F.Cu at (-344.2, 403.6)
- added D13: LED, LED_THT:LED_D3.0mm, F.Cu at (-61.6, 420.1)
- added D130: LED, LED_THT:LED_D3.0mm, F.Cu at (-333.3, 404.7)
- added D131: LED, LED_THT:LED_D3.0mm, F.Cu at (-333.3, 420.1)
- added D132: LED, LED_THT:LED_D3.0mm, F.Cu at (-333.3, 426.0)
- added D133: LED, LED_THT:LED_D3.0mm, F.Cu at (-333.3, 432.0)
- added D134: LED, LED_THT:LED_D3.0mm, F.Cu at (-333.3, 410.7)
- added D135: LED, LED_THT:LED_D3.0mm, F.Cu at (-439.4, 397.6)
- added D136: LED, LED_THT:LED_D3.0mm, F.Cu at (-445.8, 397.6)
- added D137: LED, LED_THT:LED_D3.0mm, F.Cu at (-423.8, 398.8)
- added D138: LED, LED_THT:LED_D3.0mm, F.Cu at (-417.5, 398.8)
- added D139: LED, LED_THT:LED_D3.0mm, F.Cu at (-417.5, 432.0)
- added D14: LED, LED_THT:LED_D3.0mm, F.Cu at (-61.6, 426.0)
- added D140: LED, LED_THT:LED_D3.0mm, F.Cu at (-417.5, 426.0)
- added D141: LED, LED_THT:LED_D3.0mm, F.Cu at (-417.5, 414.1)
- added D142: LED, LED_THT:LED_D3.0mm, F.Cu at (-417.5, 420.1)
- added D143: LED, LED_THT:LED_D3.0mm, F.Cu at (-417.5, 404.7)
- added D144: LED, LED_THT:LED_D3.0mm, F.Cu at (-445.8, 403.6)
- added D145: LED, LED_THT:LED_D3.0mm, F.Cu at (-434.8, 403.6)
- added D146: LED, LED_THT:LED_D3.0mm, F.Cu at (-423.8, 404.7)
- added D147: LED, LED_THT:LED_D3.0mm, F.Cu at (-423.8, 420.1)
- added D148: LED, LED_THT:LED_D3.0mm, F.Cu at (-423.8, 426.0)
- added D149: LED, LED_THT:LED_D3.0mm, F.Cu at (-423.8, 432.0)
- added D15: LED, LED_THT:LED_D3.0mm, F.Cu at (-61.6, 432.0)
- added D150: LED, LED_THT:LED_D3.0mm, F.Cu at (-423.8, 410.7)
- added D151: LED, LED_THT:LED_D3.0mm, F.Cu at (-194.5, 716.1)
- added D152: LED, LED_THT:LED_D3.0mm, F.Cu at (-200.8, 716.1)
- added D153: LED, LED_THT:LED_D3.0mm, F.Cu at (-178.8, 717.3)
- added D154: LED, LED_THT:LED_D3.0mm, F.Cu at (-172.5, 717.3)
- added D155: LED, LED_THT:LED_D3.0mm, F.Cu at (-172.5, 750.5)
- added D156: LED, LED_THT:LED_D3.0mm, F.Cu at (-172.5, 744.5)
- added D157: LED, LED_THT:LED_D3.0mm, F.Cu at (-172.5, 732.6)
- added D158: LED, LED_THT:LED_D3.0mm, F.Cu at (-172.5, 738.6)
- added D159: LED, LED_THT:LED_D3.0mm, F.Cu at (-172.5, 723.2)
- added D16: LED, LED_THT:LED_D3.0mm, F.Cu at (-61.6, 410.7)
- added D160: LED, LED_THT:LED_D3.0mm, F.Cu at (-200.8, 722.1)
- added D161: LED, LED_THT:LED_D3.0mm, F.Cu at (-189.8, 722.1)
- added D162: LED, LED_THT:LED_D3.0mm, F.Cu at (-178.8, 723.2)
- added D163: LED, LED_THT:LED_D3.0mm, F.Cu at (-178.8, 738.6)
- added D164: LED, LED_THT:LED_D3.0mm, F.Cu at (-178.8, 744.5)
- added D165: LED, LED_THT:LED_D3.0mm, F.Cu at (-178.8, 750.5)
- added D166: LED, LED_THT:LED_D3.0mm, F.Cu at (-178.8, 729.2)
- added D17: LED, LED_THT:LED_D3.0mm, F.Cu at (142.4, 79.0)
- added D18: LED, LED_THT:LED_D3.0mm, F.Cu at (136.1, 79.0)
- added D19: LED, LED_THT:LED_D3.0mm, F.Cu at (158.1, 80.2)
- added D2: LED, LED_THT:LED_D3.0mm, F.Cu at (-83.6, 397.6)
- added D20: LED, LED_THT:LED_D3.0mm, F.Cu at (164.4, 80.2)
- added D21: LED, LED_THT:LED_D3.0mm, F.Cu at (164.4, 113.4)
- added D22: LED, LED_THT:LED_D3.0mm, F.Cu at (164.4, 107.4)
- added D23: LED, LED_THT:LED_D3.0mm, F.Cu at (164.4, 95.5)
- added D24: LED, LED_THT:LED_D3.0mm, F.Cu at (164.4, 101.5)
- added D25: LED, LED_THT:LED_D3.0mm, F.Cu at (164.4, 86.1)
- added D26: LED, LED_THT:LED_D3.0mm, F.Cu at (136.1, 85.0)
- added D27: LED, LED_THT:LED_D3.0mm, F.Cu at (147.1, 85.0)
- added D28: LED, LED_THT:LED_D3.0mm, F.Cu at (158.1, 86.1)
- added D29: LED, LED_THT:LED_D3.0mm, F.Cu at (158.1, 101.5)
- added D3: LED, LED_THT:LED_D3.0mm, F.Cu at (-61.6, 398.8)
- added D30: LED, LED_THT:LED_D3.0mm, F.Cu at (158.1, 107.4)
- added D31: LED, LED_THT:LED_D3.0mm, F.Cu at (158.1, 113.4)
- added D32: LED, LED_THT:LED_D3.0mm, F.Cu at (158.1, 92.1)
- added D33: LED, LED_THT:LED_D3.0mm, F.Cu at (145.0, 139.7)
- added D34: LED, LED_THT:LED_D3.0mm, F.Cu at (138.7, 139.7)
- added D35: LED, LED_THT:LED_D3.0mm, F.Cu at (160.6, 140.9)
- added D36: LED, LED_THT:LED_D3.0mm, F.Cu at (166.9, 140.9)
- added D37: LED, LED_THT:LED_D3.0mm, F.Cu at (166.9, 174.1)
- added D38: LED, LED_THT:LED_D3.0mm, F.Cu at (166.9, 168.1)
- added D39: LED, LED_THT:LED_D3.0mm, F.Cu at (166.9, 156.2)
- added D4: LED, LED_THT:LED_D3.0mm, F.Cu at (-55.3, 398.8)
- added D40: LED, LED_THT:LED_D3.0mm, F.Cu at (166.9, 162.2)
- added D41: LED, LED_THT:LED_D3.0mm, F.Cu at (166.9, 146.8)
- added D42: LED, LED_THT:LED_D3.0mm, F.Cu at (138.7, 145.7)
- added D43: LED, LED_THT:LED_D3.0mm, F.Cu at (149.7, 145.7)
- added D44: LED, LED_THT:LED_D3.0mm, F.Cu at (160.6, 146.8)
- added D45: LED, LED_THT:LED_D3.0mm, F.Cu at (160.6, 162.2)
- added D46: LED, LED_THT:LED_D3.0mm, F.Cu at (160.6, 168.1)
- added D47: LED, LED_THT:LED_D3.0mm, F.Cu at (160.6, 174.1)
- added D48: LED, LED_THT:LED_D3.0mm, F.Cu at (160.6, 152.8)
- added D49: LED, LED_THT:LED_D3.0mm, F.Cu at (-103.9, 716.1)
- added D5: LED, LED_THT:LED_D3.0mm, F.Cu at (-55.3, 432.0)
- added D50: LED, LED_THT:LED_D3.0mm, F.Cu at (-110.2, 716.1)
- added D51: LED, LED_THT:LED_D3.0mm, F.Cu at (-88.3, 717.3)
- added D52: LED, LED_THT:LED_D3.0mm, F.Cu at (-82.0, 717.3)
- added D53: LED, LED_THT:LED_D3.0mm, F.Cu at (-82.0, 750.5)
- added D54: LED, LED_THT:LED_D3.0mm, F.Cu at (-82.0, 744.5)
- added D55: LED, LED_THT:LED_D3.0mm, F.Cu at (-82.0, 732.6)
- added D56: LED, LED_THT:LED_D3.0mm, F.Cu at (-82.0, 738.6)
- added D57: LED, LED_THT:LED_D3.0mm, F.Cu at (-82.0, 723.2)
- added D58: LED, LED_THT:LED_D3.0mm, F.Cu at (-110.2, 722.1)
- added D59: LED, LED_THT:LED_D3.0mm, F.Cu at (-99.3, 722.1)
- added D6: LED, LED_THT:LED_D3.0mm, F.Cu at (-55.3, 426.0)
- added D60: LED, LED_THT:LED_D3.0mm, F.Cu at (-88.3, 723.2)
- added D61: LED, LED_THT:LED_D3.0mm, F.Cu at (-88.3, 738.6)
- added D62: LED, LED_THT:LED_D3.0mm, F.Cu at (-88.3, 744.5)
- added D63: LED, LED_THT:LED_D3.0mm, F.Cu at (-88.3, 750.5)
- added D64: LED, LED_THT:LED_D3.0mm, F.Cu at (-88.3, 729.2)
- added D65: LED, LED_THT:LED_D3.0mm, F.Cu at (-167.8, 397.6)
- added D66: LED, LED_THT:LED_D3.0mm, F.Cu at (-174.1, 397.6)
- added D67: LED, LED_THT:LED_D3.0mm, F.Cu at (-152.2, 398.8)
- added D68: LED, LED_THT:LED_D3.0mm, F.Cu at (-145.9, 398.8)
- added D69: LED, LED_THT:LED_D3.0mm, F.Cu at (-145.9, 432.0)
- added D7: LED, LED_THT:LED_D3.0mm, F.Cu at (-55.3, 414.1)
- added D70: LED, LED_THT:LED_D3.0mm, F.Cu at (-145.9, 426.0)
- added D71: LED, LED_THT:LED_D3.0mm, F.Cu at (-145.9, 414.1)
- added D72: LED, LED_THT:LED_D3.0mm, F.Cu at (-145.9, 420.1)
- added D73: LED, LED_THT:LED_D3.0mm, F.Cu at (-145.9, 404.7)
- added D74: LED, LED_THT:LED_D3.0mm, F.Cu at (-174.1, 403.6)
- added D75: LED, LED_THT:LED_D3.0mm, F.Cu at (-163.2, 403.6)
- added D76: LED, LED_THT:LED_D3.0mm, F.Cu at (-152.2, 404.7)
- added D77: LED, LED_THT:LED_D3.0mm, F.Cu at (-152.2, 420.1)
- added D78: LED, LED_THT:LED_D3.0mm, F.Cu at (-152.2, 426.0)
- added D79: LED, LED_THT:LED_D3.0mm, F.Cu at (-152.2, 432.0)
- added D8: LED, LED_THT:LED_D3.0mm, F.Cu at (-55.3, 420.1)
- added D80: LED, LED_THT:LED_D3.0mm, F.Cu at (-152.2, 410.7)
- added D81: LED, LED_THT:LED_D3.0mm, F.Cu at (-258.4, 397.6)
- added D82: LED, LED_THT:LED_D3.0mm, F.Cu at (-264.7, 397.6)
- added D83: LED, LED_THT:LED_D3.0mm, F.Cu at (-242.7, 398.8)
- added D84: LED, LED_THT:LED_D3.0mm, F.Cu at (-236.4, 398.8)
- added D85: LED, LED_THT:LED_D3.0mm, F.Cu at (-236.4, 432.0)
- added D86: LED, LED_THT:LED_D3.0mm, F.Cu at (-236.4, 426.0)
- added D87: LED, LED_THT:LED_D3.0mm, F.Cu at (-236.4, 414.1)
- added D88: LED, LED_THT:LED_D3.0mm, F.Cu at (-236.4, 420.1)
- added D89: LED, LED_THT:LED_D3.0mm, F.Cu at (-236.4, 404.7)
- added D9: LED, LED_THT:LED_D3.0mm, F.Cu at (-55.3, 404.7)
- added D90: LED, LED_THT:LED_D3.0mm, F.Cu at (-264.7, 403.6)
- added D91: LED, LED_THT:LED_D3.0mm, F.Cu at (-253.7, 403.6)
- added D92: LED, LED_THT:LED_D3.0mm, F.Cu at (-242.7, 404.7)
- added D93: LED, LED_THT:LED_D3.0mm, F.Cu at (-242.7, 420.1)
- added D94: LED, LED_THT:LED_D3.0mm, F.Cu at (-242.7, 426.0)
- added D95: LED, LED_THT:LED_D3.0mm, F.Cu at (-242.7, 432.0)
- added D96: LED, LED_THT:LED_D3.0mm, F.Cu at (-242.7, 410.7)
- added D97: LED, LED_THT:LED_D3.0mm, F.Cu at (-407.1, 660.4)
- added D98: LED, LED_THT:LED_D3.0mm, F.Cu at (-413.4, 660.4)
- added D99: LED, LED_THT:LED_D3.0mm, F.Cu at (-419.7, 660.4)
- added R10: 220, Resistor_THT:R_Axial_DIN0204_L3.6mm_D1.6mm_P7.62mm_Horizontal, F.Cu at (-83.8, 408.3)
- added R100: 220, Resistor_THT:R_Axial_DIN0204_L3.6mm_D1.6mm_P7.62mm_Horizontal, F.Cu at (-264.9, 419.0)
- added R101: 220, Resistor_THT:R_Axial_DIN0204_L3.6mm_D1.6mm_P7.62mm_Horizontal, F.Cu at (-264.9, 422.5)
- added R102: 220, Resistor_THT:R_Axial_DIN0204_L3.6mm_D1.6mm_P7.62mm_Horizontal, F.Cu at (-264.9, 426.1)
- added R103: 220, Resistor_THT:R_Axial_DIN0204_L3.6mm_D1.6mm_P7.62mm_Horizontal, F.Cu at (-264.9, 429.6)
- added R104: 220, Resistor_THT:R_Axial_DIN0204_L3.6mm_D1.6mm_P7.62mm_Horizontal, F.Cu at (-264.9, 433.2)
- added R105: 220, Resistor_THT:R_Axial_DIN0204_L3.6mm_D1.6mm_P7.62mm_Horizontal, F.Cu at (-435.0, 672.3)
- added R106: 220, Resistor_THT:R_Axial_DIN0204_L3.6mm_D1.6mm_P7.62mm_Horizontal, F.Cu at (-445.9, 672.3)
- added R107: 220, Resistor_THT:R_Axial_DIN0204_L3.6mm_D1.6mm_P7.62mm_Horizontal, F.Cu at (-419.9, 665.2)
- added R108: 220, Resistor_THT:R_Axial_DIN0204_L3.6mm_D1.6mm_P7.62mm_Horizontal, F.Cu at (-419.9, 668.7)
- added R109: 220, Resistor_THT:R_Axial_DIN0204_L3.6mm_D1.6mm_P7.62mm_Horizontal, F.Cu at (-409.0, 665.2)
- added R11: 220, Resistor_THT:R_Axial_DIN0204_L3.6mm_D1.6mm_P7.62mm_Horizontal, F.Cu at (-83.8, 411.9)
- added R110: 220, Resistor_THT:R_Axial_DIN0204_L3.6mm_D1.6mm_P7.62mm_Horizontal, F.Cu at (-409.0, 668.7)
- added R111: 220, Resistor_THT:R_Axial_DIN0204_L3.6mm_D1.6mm_P7.62mm_Horizontal, F.Cu at (-409.0, 672.3)
- added R112: 220, Resistor_THT:R_Axial_DIN0204_L3.6mm_D1.6mm_P7.62mm_Horizontal, F.Cu at (-419.9, 672.3)
- added R113: 220, Resistor_THT:R_Axial_DIN0204_L3.6mm_D1.6mm_P7.62mm_Horizontal, F.Cu at (-367.9, 663.4)
- added R114: 220, Resistor_THT:R_Axial_DIN0204_L3.6mm_D1.6mm_P7.62mm_Horizontal, F.Cu at (-367.9, 667.0)
- added R115: 220, Resistor_THT:R_Axial_DIN0204_L3.6mm_D1.6mm_P7.62mm_Horizontal, F.Cu at (-367.9, 670.5)
- added R116: 220, Resistor_THT:R_Axial_DIN0204_L3.6mm_D1.6mm_P7.62mm_Horizontal, F.Cu at (-367.9, 674.1)
- added R117: 220, Resistor_THT:R_Axial_DIN0204_L3.6mm_D1.6mm_P7.62mm_Horizontal, F.Cu at (-367.9, 677.6)
- added R118: 220, Resistor_THT:R_Axial_DIN0204_L3.6mm_D1.6mm_P7.62mm_Horizontal, F.Cu at (-367.9, 681.2)
- added R119: 220, Resistor_THT:R_Axial_DIN0204_L3.6mm_D1.6mm_P7.62mm_Horizontal, F.Cu at (-367.9, 684.7)
- added R12: 220, Resistor_THT:R_Axial_DIN0204_L3.6mm_D1.6mm_P7.62mm_Horizontal, F.Cu at (-72.8, 411.9)
- added R120: 220, Resistor_THT:R_Axial_DIN0204_L3.6mm_D1.6mm_P7.62mm_Horizontal, F.Cu at (-367.9, 688.3)
- added R121: 220, Resistor_THT:R_Axial_DIN0204_L3.6mm_D1.6mm_P7.62mm_Horizontal, F.Cu at (-367.9, 691.8)
- added R122: 220, Resistor_THT:R_Axial_DIN0204_L3.6mm_D1.6mm_P7.62mm_Horizontal, F.Cu at (-367.9, 695.4)
- added R123: 220, Resistor_THT:R_Axial_DIN0204_L3.6mm_D1.6mm_P7.62mm_Horizontal, F.Cu at (-367.9, 698.9)
- added R124: 220, Resistor_THT:R_Axial_DIN0204_L3.6mm_D1.6mm_P7.62mm_Horizontal, F.Cu at (-367.9, 702.5)
- added R125: 220, Resistor_THT:R_Axial_DIN0204_L3.6mm_D1.6mm_P7.62mm_Horizontal, F.Cu at (-367.9, 706.0)
- added R126: 220, Resistor_THT:R_Axial_DIN0204_L3.6mm_D1.6mm_P7.62mm_Horizontal, F.Cu at (-367.9, 709.6)
- added R127: 220, Resistor_THT:R_Axial_DIN0204_L3.6mm_D1.6mm_P7.62mm_Horizontal, F.Cu at (-344.4, 408.3)
- added R128: 220, Resistor_THT:R_Axial_DIN0204_L3.6mm_D1.6mm_P7.62mm_Horizontal, F.Cu at (-355.4, 408.3)
- added R129: 220, Resistor_THT:R_Axial_DIN0204_L3.6mm_D1.6mm_P7.62mm_Horizontal, F.Cu at (-355.4, 411.9)
- added R13: 220, Resistor_THT:R_Axial_DIN0204_L3.6mm_D1.6mm_P7.62mm_Horizontal, F.Cu at (-72.8, 433.2)
- added R130: 220, Resistor_THT:R_Axial_DIN0204_L3.6mm_D1.6mm_P7.62mm_Horizontal, F.Cu at (-344.4, 411.9)
- added R131: 220, Resistor_THT:R_Axial_DIN0204_L3.6mm_D1.6mm_P7.62mm_Horizontal, F.Cu at (-344.4, 433.2)
- added R132: 220, Resistor_THT:R_Axial_DIN0204_L3.6mm_D1.6mm_P7.62mm_Horizontal, F.Cu at (-344.4, 429.6)
- added R133: 220, Resistor_THT:R_Axial_DIN0204_L3.6mm_D1.6mm_P7.62mm_Horizontal, F.Cu at (-344.4, 426.1)
- added R134: 220, Resistor_THT:R_Axial_DIN0204_L3.6mm_D1.6mm_P7.62mm_Horizontal, F.Cu at (-344.4, 422.5)
- added R135: 220, Resistor_THT:R_Axial_DIN0204_L3.6mm_D1.6mm_P7.62mm_Horizontal, F.Cu at (-344.4, 419.0)
- added R136: 220, Resistor_THT:R_Axial_DIN0204_L3.6mm_D1.6mm_P7.62mm_Horizontal, F.Cu at (-344.4, 415.4)
- added R137: 220, Resistor_THT:R_Axial_DIN0204_L3.6mm_D1.6mm_P7.62mm_Horizontal, F.Cu at (-355.4, 415.4)
- added R138: 220, Resistor_THT:R_Axial_DIN0204_L3.6mm_D1.6mm_P7.62mm_Horizontal, F.Cu at (-355.4, 419.0)
- added R139: 220, Resistor_THT:R_Axial_DIN0204_L3.6mm_D1.6mm_P7.62mm_Horizontal, F.Cu at (-355.4, 422.5)
- added R14: 220, Resistor_THT:R_Axial_DIN0204_L3.6mm_D1.6mm_P7.62mm_Horizontal, F.Cu at (-72.8, 429.6)
- added R140: 220, Resistor_THT:R_Axial_DIN0204_L3.6mm_D1.6mm_P7.62mm_Horizontal, F.Cu at (-355.4, 426.1)
- added R141: 220, Resistor_THT:R_Axial_DIN0204_L3.6mm_D1.6mm_P7.62mm_Horizontal, F.Cu at (-355.4, 429.6)
- added R142: 220, Resistor_THT:R_Axial_DIN0204_L3.6mm_D1.6mm_P7.62mm_Horizontal, F.Cu at (-355.4, 433.2)
- added R143: 220, Resistor_THT:R_Axial_DIN0204_L3.6mm_D1.6mm_P7.62mm_Horizontal, F.Cu at (-435.0, 408.3)
- added R144: 220, Resistor_THT:R_Axial_DIN0204_L3.6mm_D1.6mm_P7.62mm_Horizontal, F.Cu at (-445.9, 408.3)
- added R145: 220, Resistor_THT:R_Axial_DIN0204_L3.6mm_D1.6mm_P7.62mm_Horizontal, F.Cu at (-445.9, 411.9)
- added R146: 220, Resistor_THT:R_Axial_DIN0204_L3.6mm_D1.6mm_P7.62mm_Horizontal, F.Cu at (-435.0, 411.9)
- added R147: 220, Resistor_THT:R_Axial_DIN0204_L3.6mm_D1.6mm_P7.62mm_Horizontal, F.Cu at (-435.0, 433.2)
- added R148: 220, Resistor_THT:R_Axial_DIN0204_L3.6mm_D1.6mm_P7.62mm_Horizontal, F.Cu at (-435.0, 429.6)
- added R149: 220, Resistor_THT:R_Axial_DIN0204_L3.6mm_D1.6mm_P7.62mm_Horizontal, F.Cu at (-435.0, 426.1)
- added R15: 220, Resistor_THT:R_Axial_DIN0204_L3.6mm_D1.6mm_P7.62mm_Horizontal, F.Cu at (-72.8, 426.1)
- added R150: 220, Resistor_THT:R_Axial_DIN0204_L3.6mm_D1.6mm_P7.62mm_Horizontal, F.Cu at (-435.0, 422.5)
- added R151: 220, Resistor_THT:R_Axial_DIN0204_L3.6mm_D1.6mm_P7.62mm_Horizontal, F.Cu at (-435.0, 419.0)
- added R152: 220, Resistor_THT:R_Axial_DIN0204_L3.6mm_D1.6mm_P7.62mm_Horizontal, F.Cu at (-435.0, 415.4)
- added R153: 220, Resistor_THT:R_Axial_DIN0204_L3.6mm_D1.6mm_P7.62mm_Horizontal, F.Cu at (-445.9, 415.4)
- added R154: 220, Resistor_THT:R_Axial_DIN0204_L3.6mm_D1.6mm_P7.62mm_Horizontal, F.Cu at (-445.9, 419.0)
- added R155: 220, Resistor_THT:R_Axial_DIN0204_L3.6mm_D1.6mm_P7.62mm_Horizontal, F.Cu at (-445.9, 422.5)
- added R156: 220, Resistor_THT:R_Axial_DIN0204_L3.6mm_D1.6mm_P7.62mm_Horizontal, F.Cu at (-445.9, 426.1)
- added R157: 220, Resistor_THT:R_Axial_DIN0204_L3.6mm_D1.6mm_P7.62mm_Horizontal, F.Cu at (-445.9, 429.6)
- added R158: 220, Resistor_THT:R_Axial_DIN0204_L3.6mm_D1.6mm_P7.62mm_Horizontal, F.Cu at (-445.9, 433.2)
- added R159: 220, Resistor_THT:R_Axial_DIN0204_L3.6mm_D1.6mm_P7.62mm_Horizontal, F.Cu at (-190.0, 726.8)
- added R16: 220, Resistor_THT:R_Axial_DIN0204_L3.6mm_D1.6mm_P7.62mm_Horizontal, F.Cu at (-72.8, 422.5)
- added R160: 220, Resistor_THT:R_Axial_DIN0204_L3.6mm_D1.6mm_P7.62mm_Horizontal, F.Cu at (-201.0, 726.8)
- added R161: 220, Resistor_THT:R_Axial_DIN0204_L3.6mm_D1.6mm_P7.62mm_Horizontal, F.Cu at (-201.0, 730.4)
- added R162: 220, Resistor_THT:R_Axial_DIN0204_L3.6mm_D1.6mm_P7.62mm_Horizontal, F.Cu at (-190.0, 730.4)
- added R163: 220, Resistor_THT:R_Axial_DIN0204_L3.6mm_D1.6mm_P7.62mm_Horizontal, F.Cu at (-190.0, 751.7)
- added R164: 220, Resistor_THT:R_Axial_DIN0204_L3.6mm_D1.6mm_P7.62mm_Horizontal, F.Cu at (-190.0, 748.1)
- added R165: 220, Resistor_THT:R_Axial_DIN0204_L3.6mm_D1.6mm_P7.62mm_Horizontal, F.Cu at (-190.0, 744.6)
- added R166: 220, Resistor_THT:R_Axial_DIN0204_L3.6mm_D1.6mm_P7.62mm_Horizontal, F.Cu at (-190.0, 741.0)
- added R167: 220, Resistor_THT:R_Axial_DIN0204_L3.6mm_D1.6mm_P7.62mm_Horizontal, F.Cu at (-190.0, 737.5)
- added R168: 220, Resistor_THT:R_Axial_DIN0204_L3.6mm_D1.6mm_P7.62mm_Horizontal, F.Cu at (-190.0, 733.9)
- added R169: 220, Resistor_THT:R_Axial_DIN0204_L3.6mm_D1.6mm_P7.62mm_Horizontal, F.Cu at (-201.0, 733.9)
- added R17: 220, Resistor_THT:R_Axial_DIN0204_L3.6mm_D1.6mm_P7.62mm_Horizontal, F.Cu at (-72.8, 419.0)
- added R170: 220, Resistor_THT:R_Axial_DIN0204_L3.6mm_D1.6mm_P7.62mm_Horizontal, F.Cu at (-201.0, 737.5)
- added R171: 220, Resistor_THT:R_Axial_DIN0204_L3.6mm_D1.6mm_P7.62mm_Horizontal, F.Cu at (-201.0, 741.0)
- added R172: 220, Resistor_THT:R_Axial_DIN0204_L3.6mm_D1.6mm_P7.62mm_Horizontal, F.Cu at (-201.0, 744.6)
- added R173: 220, Resistor_THT:R_Axial_DIN0204_L3.6mm_D1.6mm_P7.62mm_Horizontal, F.Cu at (-201.0, 748.1)
- added R174: 220, Resistor_THT:R_Axial_DIN0204_L3.6mm_D1.6mm_P7.62mm_Horizontal, F.Cu at (-201.0, 751.7)
- added R18: 220, Resistor_THT:R_Axial_DIN0204_L3.6mm_D1.6mm_P7.62mm_Horizontal, F.Cu at (-72.8, 415.4)
- added R19: 220, Resistor_THT:R_Axial_DIN0204_L3.6mm_D1.6mm_P7.62mm_Horizontal, F.Cu at (-83.8, 415.4)
- added R20: 220, Resistor_THT:R_Axial_DIN0204_L3.6mm_D1.6mm_P7.62mm_Horizontal, F.Cu at (-83.8, 419.0)
- added R21: 220, Resistor_THT:R_Axial_DIN0204_L3.6mm_D1.6mm_P7.62mm_Horizontal, F.Cu at (-83.8, 422.5)
- added R22: 220, Resistor_THT:R_Axial_DIN0204_L3.6mm_D1.6mm_P7.62mm_Horizontal, F.Cu at (-83.8, 426.1)
- added R23: 220, Resistor_THT:R_Axial_DIN0204_L3.6mm_D1.6mm_P7.62mm_Horizontal, F.Cu at (-83.8, 429.6)
- added R24: 220, Resistor_THT:R_Axial_DIN0204_L3.6mm_D1.6mm_P7.62mm_Horizontal, F.Cu at (-83.8, 433.2)
- added R25: 220, Resistor_THT:R_Axial_DIN0204_L3.6mm_D1.6mm_P7.62mm_Horizontal, F.Cu at (146.9, 89.7)
- added R26: 220, Resistor_THT:R_Axial_DIN0204_L3.6mm_D1.6mm_P7.62mm_Horizontal, F.Cu at (135.9, 89.7)
- added R27: 220, Resistor_THT:R_Axial_DIN0204_L3.6mm_D1.6mm_P7.62mm_Horizontal, F.Cu at (135.9, 93.3)
- added R28: 220, Resistor_THT:R_Axial_DIN0204_L3.6mm_D1.6mm_P7.62mm_Horizontal, F.Cu at (146.9, 93.3)
- added R29: 220, Resistor_THT:R_Axial_DIN0204_L3.6mm_D1.6mm_P7.62mm_Horizontal, F.Cu at (146.9, 114.6)
- added R30: 220, Resistor_THT:R_Axial_DIN0204_L3.6mm_D1.6mm_P7.62mm_Horizontal, F.Cu at (146.9, 111.0)
- added R31: 220, Resistor_THT:R_Axial_DIN0204_L3.6mm_D1.6mm_P7.62mm_Horizontal, F.Cu at (146.9, 107.5)
- added R32: 220, Resistor_THT:R_Axial_DIN0204_L3.6mm_D1.6mm_P7.62mm_Horizontal, F.Cu at (146.9, 103.9)
- added R33: 220, Resistor_THT:R_Axial_DIN0204_L3.6mm_D1.6mm_P7.62mm_Horizontal, F.Cu at (146.9, 100.4)
- added R34: 220, Resistor_THT:R_Axial_DIN0204_L3.6mm_D1.6mm_P7.62mm_Horizontal, F.Cu at (146.9, 96.8)
- added R35: 220, Resistor_THT:R_Axial_DIN0204_L3.6mm_D1.6mm_P7.62mm_Horizontal, F.Cu at (135.9, 96.8)
- added R36: 220, Resistor_THT:R_Axial_DIN0204_L3.6mm_D1.6mm_P7.62mm_Horizontal, F.Cu at (135.9, 100.4)
- added R37: 220, Resistor_THT:R_Axial_DIN0204_L3.6mm_D1.6mm_P7.62mm_Horizontal, F.Cu at (135.9, 103.9)
- added R38: 220, Resistor_THT:R_Axial_DIN0204_L3.6mm_D1.6mm_P7.62mm_Horizontal, F.Cu at (135.9, 107.5)
- added R39: 220, Resistor_THT:R_Axial_DIN0204_L3.6mm_D1.6mm_P7.62mm_Horizontal, F.Cu at (135.9, 111.0)
- added R40: 220, Resistor_THT:R_Axial_DIN0204_L3.6mm_D1.6mm_P7.62mm_Horizontal, F.Cu at (135.9, 114.6)
- added R41: 220, Resistor_THT:R_Axial_DIN0204_L3.6mm_D1.6mm_P7.62mm_Horizontal, F.Cu at (149.5, 150.4)
- added R42: 220, Resistor_THT:R_Axial_DIN0204_L3.6mm_D1.6mm_P7.62mm_Horizontal, F.Cu at (138.5, 150.4)
- added R43: 220, Resistor_THT:R_Axial_DIN0204_L3.6mm_D1.6mm_P7.62mm_Horizontal, F.Cu at (138.5, 154.0)
- added R44: 220, Resistor_THT:R_Axial_DIN0204_L3.6mm_D1.6mm_P7.62mm_Horizontal, F.Cu at (149.5, 154.0)
- added R45: 220, Resistor_THT:R_Axial_DIN0204_L3.6mm_D1.6mm_P7.62mm_Horizontal, F.Cu at (149.5, 175.3)
- added R46: 220, Resistor_THT:R_Axial_DIN0204_L3.6mm_D1.6mm_P7.62mm_Horizontal, F.Cu at (149.5, 171.7)
- added R47: 220, Resistor_THT:R_Axial_DIN0204_L3.6mm_D1.6mm_P7.62mm_Horizontal, F.Cu at (149.5, 168.2)
- added R48: 220, Resistor_THT:R_Axial_DIN0204_L3.6mm_D1.6mm_P7.62mm_Horizontal, F.Cu at (149.5, 164.6)
- added R49: 220, Resistor_THT:R_Axial_DIN0204_L3.6mm_D1.6mm_P7.62mm_Horizontal, F.Cu at (149.5, 161.1)
- added R50: 220, Resistor_THT:R_Axial_DIN0204_L3.6mm_D1.6mm_P7.62mm_Horizontal, F.Cu at (149.5, 157.5)
- added R51: 220, Resistor_THT:R_Axial_DIN0204_L3.6mm_D1.6mm_P7.62mm_Horizontal, F.Cu at (138.5, 157.5)
- added R52: 220, Resistor_THT:R_Axial_DIN0204_L3.6mm_D1.6mm_P7.62mm_Horizontal, F.Cu at (138.5, 161.1)
- added R53: 220, Resistor_THT:R_Axial_DIN0204_L3.6mm_D1.6mm_P7.62mm_Horizontal, F.Cu at (138.5, 164.6)
- added R54: 220, Resistor_THT:R_Axial_DIN0204_L3.6mm_D1.6mm_P7.62mm_Horizontal, F.Cu at (138.5, 168.2)
- added R55: 220, Resistor_THT:R_Axial_DIN0204_L3.6mm_D1.6mm_P7.62mm_Horizontal, F.Cu at (138.5, 171.7)
- added R56: 220, Resistor_THT:R_Axial_DIN0204_L3.6mm_D1.6mm_P7.62mm_Horizontal, F.Cu at (138.5, 175.3)
- added R57: 220, Resistor_THT:R_Axial_DIN0204_L3.6mm_D1.6mm_P7.62mm_Horizontal, F.Cu at (-99.5, 726.8)
- added R58: 220, Resistor_THT:R_Axial_DIN0204_L3.6mm_D1.6mm_P7.62mm_Horizontal, F.Cu at (-110.4, 726.8)
- added R59: 220, Resistor_THT:R_Axial_DIN0204_L3.6mm_D1.6mm_P7.62mm_Horizontal, F.Cu at (-110.4, 730.4)
- added R60: 220, Resistor_THT:R_Axial_DIN0204_L3.6mm_D1.6mm_P7.62mm_Horizontal, F.Cu at (-99.5, 730.4)
- added R61: 220, Resistor_THT:R_Axial_DIN0204_L3.6mm_D1.6mm_P7.62mm_Horizontal, F.Cu at (-99.5, 751.7)
- added R62: 220, Resistor_THT:R_Axial_DIN0204_L3.6mm_D1.6mm_P7.62mm_Horizontal, F.Cu at (-99.5, 748.1)
- added R63: 220, Resistor_THT:R_Axial_DIN0204_L3.6mm_D1.6mm_P7.62mm_Horizontal, F.Cu at (-99.5, 744.6)
- added R64: 220, Resistor_THT:R_Axial_DIN0204_L3.6mm_D1.6mm_P7.62mm_Horizontal, F.Cu at (-99.5, 741.0)
- added R65: 220, Resistor_THT:R_Axial_DIN0204_L3.6mm_D1.6mm_P7.62mm_Horizontal, F.Cu at (-99.5, 737.5)
- added R66: 220, Resistor_THT:R_Axial_DIN0204_L3.6mm_D1.6mm_P7.62mm_Horizontal, F.Cu at (-99.5, 733.9)
- added R67: 220, Resistor_THT:R_Axial_DIN0204_L3.6mm_D1.6mm_P7.62mm_Horizontal, F.Cu at (-110.4, 733.9)
- added R68: 220, Resistor_THT:R_Axial_DIN0204_L3.6mm_D1.6mm_P7.62mm_Horizontal, F.Cu at (-110.4, 737.5)
- added R69: 220, Resistor_THT:R_Axial_DIN0204_L3.6mm_D1.6mm_P7.62mm_Horizontal, F.Cu at (-110.4, 741.0)
- added R70: 220, Resistor_THT:R_Axial_DIN0204_L3.6mm_D1.6mm_P7.62mm_Horizontal, F.Cu at (-110.4, 744.6)
- added R71: 220, Resistor_THT:R_Axial_DIN0204_L3.6mm_D1.6mm_P7.62mm_Horizontal, F.Cu at (-110.4, 748.1)
- added R72: 220, Resistor_THT:R_Axial_DIN0204_L3.6mm_D1.6mm_P7.62mm_Horizontal, F.Cu at (-110.4, 751.7)
- added R73: 220, Resistor_THT:R_Axial_DIN0204_L3.6mm_D1.6mm_P7.62mm_Horizontal, F.Cu at (-163.4, 408.3)
- added R74: 220, Resistor_THT:R_Axial_DIN0204_L3.6mm_D1.6mm_P7.62mm_Horizontal, F.Cu at (-174.3, 408.3)
- added R75: 220, Resistor_THT:R_Axial_DIN0204_L3.6mm_D1.6mm_P7.62mm_Horizontal, F.Cu at (-174.3, 411.9)
- added R76: 220, Resistor_THT:R_Axial_DIN0204_L3.6mm_D1.6mm_P7.62mm_Horizontal, F.Cu at (-163.4, 411.9)
- added R77: 220, Resistor_THT:R_Axial_DIN0204_L3.6mm_D1.6mm_P7.62mm_Horizontal, F.Cu at (-163.4, 433.2)
- added R78: 220, Resistor_THT:R_Axial_DIN0204_L3.6mm_D1.6mm_P7.62mm_Horizontal, F.Cu at (-163.4, 429.6)
- added R79: 220, Resistor_THT:R_Axial_DIN0204_L3.6mm_D1.6mm_P7.62mm_Horizontal, F.Cu at (-163.4, 426.1)
- added R80: 220, Resistor_THT:R_Axial_DIN0204_L3.6mm_D1.6mm_P7.62mm_Horizontal, F.Cu at (-163.4, 422.5)
- added R81: 220, Resistor_THT:R_Axial_DIN0204_L3.6mm_D1.6mm_P7.62mm_Horizontal, F.Cu at (-163.4, 419.0)
- added R82: 220, Resistor_THT:R_Axial_DIN0204_L3.6mm_D1.6mm_P7.62mm_Horizontal, F.Cu at (-163.4, 415.4)
- added R83: 220, Resistor_THT:R_Axial_DIN0204_L3.6mm_D1.6mm_P7.62mm_Horizontal, F.Cu at (-174.3, 415.4)
- added R84: 220, Resistor_THT:R_Axial_DIN0204_L3.6mm_D1.6mm_P7.62mm_Horizontal, F.Cu at (-174.3, 419.0)
- added R85: 220, Resistor_THT:R_Axial_DIN0204_L3.6mm_D1.6mm_P7.62mm_Horizontal, F.Cu at (-174.3, 422.5)
- added R86: 220, Resistor_THT:R_Axial_DIN0204_L3.6mm_D1.6mm_P7.62mm_Horizontal, F.Cu at (-174.3, 426.1)
- added R87: 220, Resistor_THT:R_Axial_DIN0204_L3.6mm_D1.6mm_P7.62mm_Horizontal, F.Cu at (-174.3, 429.6)
- added R88: 220, Resistor_THT:R_Axial_DIN0204_L3.6mm_D1.6mm_P7.62mm_Horizontal, F.Cu at (-174.3, 433.2)
- added R89: 220, Resistor_THT:R_Axial_DIN0204_L3.6mm_D1.6mm_P7.62mm_Horizontal, F.Cu at (-253.9, 408.3)
- added R9: 220, Resistor_THT:R_Axial_DIN0204_L3.6mm_D1.6mm_P7.62mm_Horizontal, F.Cu at (-72.8, 408.3)
- added R90: 220, Resistor_THT:R_Axial_DIN0204_L3.6mm_D1.6mm_P7.62mm_Horizontal, F.Cu at (-264.9, 408.3)
- added R91: 220, Resistor_THT:R_Axial_DIN0204_L3.6mm_D1.6mm_P7.62mm_Horizontal, F.Cu at (-264.9, 411.9)
- added R92: 220, Resistor_THT:R_Axial_DIN0204_L3.6mm_D1.6mm_P7.62mm_Horizontal, F.Cu at (-253.9, 411.9)
- added R93: 220, Resistor_THT:R_Axial_DIN0204_L3.6mm_D1.6mm_P7.62mm_Horizontal, F.Cu at (-253.9, 433.2)
- added R94: 220, Resistor_THT:R_Axial_DIN0204_L3.6mm_D1.6mm_P7.62mm_Horizontal, F.Cu at (-253.9, 429.6)
- added R95: 220, Resistor_THT:R_Axial_DIN0204_L3.6mm_D1.6mm_P7.62mm_Horizontal, F.Cu at (-253.9, 426.1)
- added R96: 220, Resistor_THT:R_Axial_DIN0204_L3.6mm_D1.6mm_P7.62mm_Horizontal, F.Cu at (-253.9, 422.5)
- added R97: 220, Resistor_THT:R_Axial_DIN0204_L3.6mm_D1.6mm_P7.62mm_Horizontal, F.Cu at (-253.9, 419.0)
- added R98: 220, Resistor_THT:R_Axial_DIN0204_L3.6mm_D1.6mm_P7.62mm_Horizontal, F.Cu at (-253.9, 415.4)
- added R99: 220, Resistor_THT:R_Axial_DIN0204_L3.6mm_D1.6mm_P7.62mm_Horizontal, F.Cu at (-264.9, 415.4)
- added U75: 74LS245, Package_DIP:DIP-20_W7.62mm, F.Cu at (-445.8, 518.3)
- moved U49 760.1 mm to (-423.3, 496.0)
- moved U48 755.5 mm to (-434.5, 496.0)
- moved U47 745.9 mm to (-423.3, 518.3)
- moved U50 745.9 mm to (-434.5, 518.3)
- moved U51 745.9 mm to (-412.0, 501.1)
- moved U52 745.9 mm to (-412.0, 523.4)
- moved R8 720.9 mm to (-435.0, 668.7)
- moved U58 695.2 mm to (-367.7, 713.6)
- moved U63 695.2 mm to (-382.0, 721.6)
- moved U64 695.2 mm to (-408.0, 721.6)
- moved U65 695.2 mm to (-434.0, 721.6)
- moved SW3 695.2 mm to (-393.1, 664.6)
- moved U62 695.2 mm to (-367.7, 733.4)
- moved C2 610.6 mm to (-405.7, 594.3)
- moved C3 610.6 mm to (-416.9, 575.2)
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Connections:
- net Net-(U1-Pad2) renamed /ALU/sheet61054F43/I0
- net Net-(U1-Pad3) renamed /ALU/sheet61054F43/I1
- net Net-(U1-Pad4) renamed /ALU/sheet61054F43/I2
- net Net-(U1-Pad5) renamed /ALU/sheet61054F43/I3
- net Net-(U1-Pad6) renamed /ALU/sheet61054F43/I4
- net Net-(U1-Pad7) renamed /ALU/sheet61054F43/I5
- net Net-(U1-Pad8) renamed /ALU/sheet61054F43/I6
- net Net-(U1-Pad9) renamed /ALU/sheet61054F43/I7
- net Net-(U2-Pad2) renamed /ALU/sheet61054F43/I8
- net Net-(U2-Pad3) renamed /ALU/sheet61054F43/I9
- net Net-(U2-Pad4) renamed /ALU/sheet61054F43/I10
- net Net-(U2-Pad5) renamed /ALU/sheet61054F43/I11
- net Net-(U2-Pad6) renamed /ALU/sheet61054F43/I12
- net Net-(U2-Pad7) renamed /ALU/sheet61054F43/I13
- net Net-(U2-Pad8) renamed /ALU/sheet61054F43/I14
- net Net-(U2-Pad9) renamed /ALU/sheet61054F43/I15
- net Net-(U29-Pad2) renamed /ProgramCounter/sheet6156E9A4/I0
- net Net-(U29-Pad3) renamed /ProgramCounter/sheet6156E9A4/I1
- net Net-(U29-Pad4) renamed /ProgramCounter/sheet6156E9A4/I2
- net Net-(U29-Pad5) renamed /ProgramCounter/sheet6156E9A4/I3
- net Net-(U29-Pad6) renamed /ProgramCounter/sheet6156E9A4/I4
- net Net-(U29-Pad7) renamed /ProgramCounter/sheet6156E9A4/I5
- net Net-(U29-Pad8) renamed /ProgramCounter/sheet6156E9A4/I6
- net Net-(U29-Pad9) renamed /ProgramCounter/sheet6156E9A4/I7
- net Net-(U30-Pad2) renamed /ProgramCounter/sheet6156E9A4/I8
- net Net-(U30-Pad3) renamed /ProgramCounter/sheet6156E9A4/I9
- net Net-(U30-Pad4) renamed /ProgramCounter/sheet6156E9A4/I10
- net Net-(U30-Pad5) renamed /ProgramCounter/sheet6156E9A4/I11
- net Net-(U30-Pad6) renamed /ProgramCounter/sheet6156E9A4/I12
- net Net-(U30-Pad7) renamed /ProgramCounter/sheet6156E9A4/I13
- net Net-(U30-Pad8) renamed /ProgramCounter/sheet6156E9A4/I14
- net Net-(U30-Pad9) renamed /ProgramCounter/sheet6156E9A4/I15
- net Net-(U36-Pad2) renamed /RAM/sheet61B5B12C/I0
- net Net-(U36-Pad3) renamed /RAM/sheet61B5B12C/I1
- net Net-(U36-Pad4) renamed /RAM/sheet61B5B12C/I2
- net Net-(U36-Pad5) renamed /RAM/sheet61B5B12C/I3
- net Net-(U36-Pad6) renamed /RAM/sheet61B5B12C/I4
- net Net-(U36-Pad7) renamed /RAM/sheet61B5B12C/I5
- net Net-(U36-Pad8) renamed /RAM/sheet61B5B12C/I6
- net Net-(U36-Pad9) renamed /RAM/sheet61B5B12C/I7
- net Net-(U40-Pad2) renamed /RAM/sheet61B5B12C/I8
- net Net-(U40-Pad3) renamed /RAM/sheet61B5B12C/I9
- net Net-(U40-Pad4) renamed /RAM/sheet61B5B12C/I10
- net Net-(U40-Pad6) renamed /RAM/sheet61B5B12C/I12
- net Net-(U40-Pad7) renamed /RAM/sheet61B5B12C/I13
- net Net-(U50-Pad2) renamed /Instruction Register/sheet621E2544/I8
- net Net-(U50-Pad3) renamed /Instruction Register/sheet621E2544/I9
- net Net-(U50-Pad4) renamed /Instruction Register/sheet621E2544/I10
- net Net-(U50-Pad5) renamed /Instruction Register/sheet621E2544/I11
- net Net-(U50-Pad6) renamed /Instruction Register/sheet621E2544/I12
- net Net-(U50-Pad7) renamed /Instruction Register/sheet621E2544/I13
- net Net-(U59-Pad2) renamed /Stack/sheet60C9B368/I0
- net Net-(U59-Pad3) renamed /Stack/sheet60C9B368/I1
- net Net-(U59-Pad4) renamed /Stack/sheet60C9B368/I2
- net Net-(U59-Pad5) renamed /Stack/sheet60C9B368/I3
- net Net-(U59-Pad6) renamed /Stack/sheet60C9B368/I4
- net Net-(U59-Pad7) renamed /Stack/sheet60C9B368/I5
- net Net-(U59-Pad8) renamed /Stack/sheet60C9B368/I6
- net Net-(U59-Pad9) renamed /Stack/sheet60C9B368/I7
- net Net-(U66-Pad2) renamed /Stack/sheet60C9B368/I8
- net Net-(U66-Pad3) renamed /Stack/sheet60C9B368/I9
- net Net-(U66-Pad4) renamed /Stack/sheet60C9B368/I10
- net Net-(U66-Pad5) renamed /Stack/sheet60C9B368/I11
- net Net-(U66-Pad6) renamed /Stack/sheet60C9B368/I12
- net Net-(U66-Pad7) renamed /Stack/sheet60C9B368/I13
- net Net-(U69-Pad2) renamed /Sheet61DF6CC6/sheet623AC6D9/I0
- net Net-(U69-Pad3) renamed /Sheet61DF6CC6/sheet623AC6D9/I1
- net Net-(U69-Pad4) renamed /Sheet61DF6CC6/sheet623AC6D9/I2
- net Net-(U69-Pad5) renamed /Sheet61DF6CC6/sheet623AC6D9/I3
- net Net-(U69-Pad6) renamed /Sheet61DF6CC6/sheet623AC6D9/I4
- net Net-(U69-Pad7) renamed /Sheet61DF6CC6/sheet623AC6D9/I5
- net Net-(U69-Pad8) renamed /Sheet61DF6CC6/sheet623AC6D9/I6
- net Net-(U69-Pad9) renamed /Sheet61DF6CC6/sheet623AC6D9/I7
- net Net-(U72-Pad2) renamed /Sheet61DF6CC6/sheet623AC6D9/I8
- net Net-(U72-Pad3) renamed /Sheet61DF6CC6/sheet623AC6D9/I9
- net Net-(U72-Pad4) renamed /Sheet61DF6CC6/sheet623AC6D9/I10
- net Net-(U72-Pad5) renamed /Sheet61DF6CC6/sheet623AC6D9/I11
- net Net-(U72-Pad6) renamed /Sheet61DF6CC6/sheet623AC6D9/I12
- net Net-(U72-Pad7) renamed /Sheet61DF6CC6/sheet623AC6D9/I13
- net Net-(U72-Pad8) renamed /Sheet61DF6CC6/sheet623AC6D9/I14
- net Net-(U72-Pad9) renamed /Sheet61DF6CC6/sheet623AC6D9/I15
- U24 pad 5: /Control Unit/CLK -> /ALU/CLK
- U25 pad 8: /Control Unit/CLK -> /ALU/CLK
- U37 pad 1: /Control Unit/CLK -> /ALU/CLK
- U38 pad 7: /Control Unit/CLK -> /ALU/CLK
- U39 pad 7: /Control Unit/CLK -> /ALU/CLK
- U41 pad 7: /Control Unit/CLK -> /ALU/CLK
- U42 pad 7: /Control Unit/CLK -> /ALU/CLK
- U48 pad 7: /Control Unit/CLK -> /ALU/CLK
- U49 pad 7: /Control Unit/CLK -> /ALU/CLK
- U51 pad 7: /Control Unit/CLK -> /ALU/CLK
- U52 pad 7: /Control Unit/CLK -> /ALU/CLK
- U60 pad 7: /Control Unit/CLK -> /ALU/CLK
- U61 pad 7: /Control Unit/CLK -> /ALU/CLK
- U62 pad 2: /Control Unit/CLK -> /ALU/CLK
- U64 pad 18: /Resgister A/~AO -> /Control Unit/~R2_AO
- U65 pad 17: /Control Unit/~IR_8O -> /Instruction Register/~I80
- U67 pad 7: /Control Unit/CLK -> /ALU/CLK
- U68 pad 7: /Control Unit/CLK -> /ALU/CLK
- U70 pad 7: /Control Unit/CLK -> /ALU/CLK
- U71 pad 7: /Control Unit/CLK -> /ALU/CLK
- U73 pad 7: /Control Unit/CLK -> /ALU/CLK
- U74 pad 7: /Control Unit/CLK -> /ALU/CLK
Routing:
- net /ALU/BUS0: track 0.00 -> 102.9 mm, vias 0 -> 2
- net /ALU/BUS1: track 0.00 -> 100.3 mm, vias 0 -> 2
- net /ALU/BUS2: track 0.00 -> 97.8 mm, vias 0 -> 2
- net /ALU/BUS3: track 0.00 -> 95.2 mm, vias 0 -> 2
- net /ALU/BUS4: track 0.00 -> 92.7 mm, vias 0 -> 2
- net /ALU/BUS5: track 0.00 -> 90.2 mm, vias 0 -> 2
- net /ALU/BUS6: track 0.00 -> 87.6 mm, vias 0 -> 2
- net /ALU/BUS7: track 0.00 -> 85.1 mm, vias 0 -> 2
- net /ALU/BUS8: track 0.00 -> 82.6 mm, vias 0 -> 2
- net /ALU/BUS9: track 0.00 -> 80.0 mm, vias 0 -> 2
- net /ALU/BUS10: track 0.00 -> 77.5 mm, vias 0 -> 2
- net /ALU/BUS11: track 0.00 -> 74.9 mm, vias 0 -> 2
- net /ALU/BUS12: track 0.00 -> 72.4 mm, vias 0 -> 2
- net /ALU/BUS13: track 0.00 -> 69.8 mm, vias 0 -> 2
- net /ALU/BUS14: track 0.00 -> 67.3 mm, vias 0 -> 2
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Other:
- copper layers 4 -> 2
