File: 16bitCpu.kicad_pcb (KiCad board)
At the start: 2 copper layers, 425 parts, among them SW1 SW_Push, SW2 SW_SPDT, SW3 SW_Push-Switch, U1 74LS245, U10 74LS86, U11 74LS245, U12 74LS173, U13 74LS173, U14 74LS245, U15 74LS173, U16 74LS173, U17 74LS245, U18 74LS173, U19 74LS173, U2 74LS245, U20 74LS245, U21 74LS173, U22 74LS173, U23 LM555xN, U24 74LS04, U25 74LS08, U26 74LS32, U27 LM555xN, U28 LM555xN, U29 74LS245, U3 74LS283, U30 74LS245, U31 74LS161, U32 74LS161, U33 74LS161, U34 74LS161, U35 74HC00, U36 74LS245, U37 74HC04, U38 74LS173, U39 74LS173, U4 74LS283, U40 74LS245, U41 74LS173, U42 74LS173, U43 AS6C6264, U44 AS6C6264, U45 AT28C64B-15PU, U46 AT28C64B-15PU, U47 74LS245, U48 74LS173, U49 74LS173, U5 74LS283, U50 74LS245, U51 74LS173, U52 74LS173, U53 74LS173, U54 74HC02, U55 74HC02, U56 74LS08, U57 74LS08, U58 7400, U59 74LS245, U6 74LS283, U60 74LS173, U61 74LS173, U62 74LS161-74xx, U63 AT28C64B-15PU, U64 AT28C64B-15PU, U65 AT28C64B-15PU, U66 74LS245, U67 74LS173, U68 74LS173, U69 74LS245, U7 74LS86, U70 74LS173, U71 74LS173, U72 74LS245, U73 74LS173, U74 74LS173, U75 74LS245, U8 74LS86, U9 74LS86

Commit message: Fixes
Parts:
- moved D117 217.3 mm to (-239.9, 556.0)
- moved D99 217.3 mm to (-231.1, 552.5)
- moved C2 217.3 mm to (-217.1, 486.3)
- moved D108 217.3 mm to (-168.1, 582.7)
- moved D109 217.3 mm to (-168.1, 575.6)
- moved D110 217.3 mm to (-168.1, 568.5)
- moved D111 217.3 mm to (-168.1, 561.4)
- moved D112 217.3 mm to (-168.1, 554.3)
- moved D121 217.3 mm to (-144.7, 290.8)
- moved D122 217.3 mm to (-138.4, 290.8)
- moved D123 217.3 mm to (-138.4, 324.0)
- moved D133 217.3 mm to (-144.7, 324.0)
- moved D137 217.3 mm to (-235.2, 290.8)
- moved D138 217.3 mm to (-228.9, 290.8)
- moved D139 217.3 mm to (-228.9, 324.0)
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Connections:
- D107 pad 2: /Control Unit/~RAM_MEMWE -> /RAM/MEMWE
- D24 pad 2: /ALU/A6 -> /ALU/A7
- D40 pad 2: /Register B/A6 -> /Register B/A7
- U65 pad 13: /Control Unit/~RAM_MEMWE -> /RAM/MEMWE

Commit message: added 3-8 decoders to cu
Parts:
- added D167: LED, LED_THT:LED_D3.0mm, F.Cu at (-43.1, -128.4)
- added D168: LED, LED_THT:LED_D3.0mm, F.Cu at (-43.1, -122.5)
- added D169: LED, LED_THT:LED_D3.0mm, F.Cu at (-43.1, -116.5)
- added D170: LED, LED_THT:LED_D3.0mm, F.Cu at (-43.1, -137.8)
- added D171: LED, LED_THT:LED_D3.0mm, F.Cu at (206.1, 519.9)
- added D172: LED, LED_THT:LED_D3.0mm, F.Cu at (199.8, 519.9)
- added D173: LED, LED_THT:LED_D3.0mm, F.Cu at (221.7, 521.1)
- added D174: LED, LED_THT:LED_D3.0mm, F.Cu at (228.0, 521.1)
- added D175: LED, LED_THT:LED_D3.0mm, F.Cu at (228.0, 554.3)
- added D176: LED, LED_THT:LED_D3.0mm, F.Cu at (228.0, 548.3)
- added D177: LED, LED_THT:LED_D3.0mm, F.Cu at (228.0, 536.4)
- added D178: LED, LED_THT:LED_D3.0mm, F.Cu at (228.0, 542.4)
- added D179: LED, LED_THT:LED_D3.0mm, F.Cu at (228.0, 527.0)
- added D180: LED, LED_THT:LED_D3.0mm, F.Cu at (199.8, 525.9)
- added D181: LED, LED_THT:LED_D3.0mm, F.Cu at (210.7, 525.9)
- added D182: LED, LED_THT:LED_D3.0mm, F.Cu at (221.7, 527.0)
- added D183: LED, LED_THT:LED_D3.0mm, F.Cu at (221.7, 542.4)
- added D184: LED, LED_THT:LED_D3.0mm, F.Cu at (221.7, 548.3)
- added D185: LED, LED_THT:LED_D3.0mm, F.Cu at (221.7, 554.3)
- added D186: LED, LED_THT:LED_D3.0mm, F.Cu at (221.7, 533.0)
- added R175: 220, Resistor_THT:R_Axial_DIN0204_L3.6mm_D1.6mm_P7.62mm_Horizontal, F.Cu at (-65.3, -122.4)
- added R176: 220, Resistor_THT:R_Axial_DIN0204_L3.6mm_D1.6mm_P7.62mm_Horizontal, F.Cu at (-65.3, -118.9)
- added R177: 220, Resistor_THT:R_Axial_DIN0204_L3.6mm_D1.6mm_P7.62mm_Horizontal, F.Cu at (-65.3, -115.3)
- added R178: 1K, Resistor_THT:R_Axial_DIN0204_L3.6mm_D1.6mm_P7.62mm_Horizontal, F.Cu at (169.8, 529.8)
- added R179: 220, Resistor_THT:R_Axial_DIN0204_L3.6mm_D1.6mm_P7.62mm_Horizontal, F.Cu at (210.5, 530.6)
- added R180: 220, Resistor_THT:R_Axial_DIN0204_L3.6mm_D1.6mm_P7.62mm_Horizontal, F.Cu at (199.6, 530.6)
- added R181: 220, Resistor_THT:R_Axial_DIN0204_L3.6mm_D1.6mm_P7.62mm_Horizontal, F.Cu at (199.6, 534.2)
- added R182: 220, Resistor_THT:R_Axial_DIN0204_L3.6mm_D1.6mm_P7.62mm_Horizontal, F.Cu at (210.5, 534.2)
- added R183: 220, Resistor_THT:R_Axial_DIN0204_L3.6mm_D1.6mm_P7.62mm_Horizontal, F.Cu at (210.5, 555.5)
- added R184: 220, Resistor_THT:R_Axial_DIN0204_L3.6mm_D1.6mm_P7.62mm_Horizontal, F.Cu at (210.5, 551.9)
- added R185: 220, Resistor_THT:R_Axial_DIN0204_L3.6mm_D1.6mm_P7.62mm_Horizontal, F.Cu at (210.5, 548.4)
- added R186: 220, Resistor_THT:R_Axial_DIN0204_L3.6mm_D1.6mm_P7.62mm_Horizontal, F.Cu at (210.5, 544.8)
- added R187: 220, Resistor_THT:R_Axial_DIN0204_L3.6mm_D1.6mm_P7.62mm_Horizontal, F.Cu at (210.5, 541.3)
- added R188: 220, Resistor_THT:R_Axial_DIN0204_L3.6mm_D1.6mm_P7.62mm_Horizontal, F.Cu at (210.5, 537.7)
- added R189: 220, Resistor_THT:R_Axial_DIN0204_L3.6mm_D1.6mm_P7.62mm_Horizontal, F.Cu at (199.6, 537.7)
- added R190: 220, Resistor_THT:R_Axial_DIN0204_L3.6mm_D1.6mm_P7.62mm_Horizontal, F.Cu at (199.6, 541.3)
- added R191: 220, Resistor_THT:R_Axial_DIN0204_L3.6mm_D1.6mm_P7.62mm_Horizontal, F.Cu at (199.6, 544.8)
- added R192: 220, Resistor_THT:R_Axial_DIN0204_L3.6mm_D1.6mm_P7.62mm_Horizontal, F.Cu at (199.6, 548.4)
- added R193: 220, Resistor_THT:R_Axial_DIN0204_L3.6mm_D1.6mm_P7.62mm_Horizontal, F.Cu at (199.6, 551.9)
- added R194: 220, Resistor_THT:R_Axial_DIN0204_L3.6mm_D1.6mm_P7.62mm_Horizontal, F.Cu at (199.6, 555.5)
- added U76: 74LS245, Package_DIP:DIP-20_W7.62mm, F.Cu at (170.0, 496.3)
- added U77: 74LS173, Package_DIP:DIP-16_W7.62mm, F.Cu at (181.2, 474.0)
- added U78: 74LS173, Package_DIP:DIP-16_W7.62mm, F.Cu at (170.0, 474.0)
- added U79: AS6C6264, Package_DIP:DIP-28_W15.24mm, F.Cu at (151.1, 486.1)
- added U80: AS6C6264, Package_DIP:DIP-28_W15.24mm, F.Cu at (151.1, 523.7)
- added U81: AT28C64B-15PU, ROM:ZIF-AT28C64B-15PU, F.Cu at (136.9, 527.1)
- added U82: AT28C64B-15PU, ROM:ZIF-AT28C64B-15PU, F.Cu at (110.9, 527.1)
- R1, R2, R3, R5, R6, R7, R8: value 1K -> 220
- R104, R105, R106, R108, R109, R49: value 220 -> 1K
- R107: value 220 -> 1M
- R4: value 1M -> 220
- SW1: value SW_Push -> SW_Push-Switch
- SW2: value SW_SPDT -> SW_Push; footprint ROM:DPDT-pushbutton -> Button_Switch_THT:SW_PUSH-12mm
- SW3: value SW_Push-Switch -> SW_SPDT; footprint Button_Switch_THT:SW_PUSH-12mm -> ROM:DPDT-pushbutton
- U10, U7: value 74LS86 -> 74LS245; footprint Package_DIP:DIP-14_W7.62mm -> Package_DIP:DIP-20_W7.62mm
- U11, U2, U29, U66, U69, U75: value 74LS245 -> 74LS173; footprint Package_DIP:DIP-20_W7.62mm -> Package_DIP:DIP-16_W7.62mm
- U13, U42, U67, U70: value 74LS173 -> 74LS245; footprint Package_DIP:DIP-16_W7.62mm -> Package_DIP:DIP-20_W7.62mm
- U15, U16, U18: value 74LS173 -> 74LS161
- U17: value 74LS245 -> 74LS161; footprint Package_DIP:DIP-20_W7.62mm -> Package_DIP:DIP-16_W7.62mm
- U19: value 74LS173 -> 7400; footprint Package_DIP:DIP-16_W7.62mm -> Package_DIP:DIP-14_W7.62mm
- U20: value 74LS245 -> 74LS161-74xx; footprint Package_DIP:DIP-20_W7.62mm -> Package_DIP:DIP-16_W7.62mm
- U21, U22: value 74LS173 -> AT28C64B-15PU; footprint Package_DIP:DIP-16_W7.62mm -> ROM:ZIF-AT28C64B-15PU
- U23: value LM555xN -> AT28C64B-15PU; footprint Package_DIP:DIP-8_W7.62mm -> ROM:ZIF-AT28C64B-15PU
- U24: value 74LS04 -> 74LS245; footprint Package_DIP:DIP-14_W7.62mm -> Package_DIP:DIP-20_W7.62mm
- U25: value 74LS08 -> 74LS173; footprint Package_DIP:DIP-14_W7.62mm -> Package_DIP:DIP-16_W7.62mm
- U26: value 74LS32 -> 74LS173; footprint Package_DIP:DIP-14_W7.62mm -> Package_DIP:DIP-16_W7.62mm
- U27: value LM555xN -> 74LS245; footprint Package_DIP:DIP-8_W7.62mm -> Package_DIP:DIP-20_W7.62mm
- U28: value LM555xN -> 74LS173; footprint Package_DIP:DIP-8_W7.62mm -> Package_DIP:DIP-16_W7.62mm
- U3, U5, U6: value 74LS283 -> 74LS173
- U31, U32, U34: value 74LS161 -> 74LS173
- U33: value 74LS161 -> 74LS245; footprint Package_DIP:DIP-16_W7.62mm -> Package_DIP:DIP-20_W7.62mm
- U35: value 74HC00 -> 74LS173; footprint Package_DIP:DIP-14_W7.62mm -> Package_DIP:DIP-16_W7.62mm
- U36, U40: value 74LS245 -> LM555xN; footprint Package_DIP:DIP-20_W7.62mm -> Package_DIP:DIP-8_W7.62mm
- U37: value 74HC04 -> 74LS04
- U38: value 74LS173 -> 74LS08; footprint Package_DIP:DIP-16_W7.62mm -> Package_DIP:DIP-14_W7.62mm
- U39: value 74LS173 -> 74LS32; footprint Package_DIP:DIP-16_W7.62mm -> Package_DIP:DIP-14_W7.62mm
- U4: value 74LS283 -> 74LS245; footprint Package_DIP:DIP-16_W7.62mm -> Package_DIP:DIP-20_W7.62mm
- U41: value 74LS173 -> LM555xN; footprint Package_DIP:DIP-16_W7.62mm -> Package_DIP:DIP-8_W7.62mm
- U43: value AS6C6264 -> 74LS00; footprint Package_DIP:DIP-28_W15.24mm -> Package_DIP:DIP-14_W7.62mm
- U44: value AS6C6264 -> 74LS86; footprint Package_DIP:DIP-28_W15.24mm -> Package_DIP:DIP-14_W7.62mm
- U45, U46: value AT28C64B-15PU -> 74LS86; footprint ROM:ZIF-AT28C64B-15PU -> Package_DIP:DIP-14_W7.62mm
- U47, U50: value 74LS245 -> 74LS00; footprint Package_DIP:DIP-20_W7.62mm -> Package_DIP:DIP-14_W7.62mm
- U48: value 74LS173 -> 74LS86; footprint Package_DIP:DIP-16_W7.62mm -> Package_DIP:DIP-14_W7.62mm
- U49: value 74LS173 -> 74HC02; footprint Package_DIP:DIP-16_W7.62mm -> Package_DIP:DIP-14_W7.62mm
- U51: value 74LS173 -> 74LS00; footprint Package_DIP:DIP-16_W7.62mm -> Package_DIP:DIP-14_W7.62mm
- U52, U61: value 74LS173 -> 74LS283
- U53: value 74LS173 -> 74LS85
- U54: value 74HC02 -> 74LS283; footprint Package_DIP:DIP-14_W7.62mm -> Package_DIP:DIP-16_W7.62mm
- U55: value 74HC02 -> 74LS245; footprint Package_DIP:DIP-14_W7.62mm -> Package_DIP:DIP-20_W7.62mm
- U56: value 74LS08 -> 74LS85; footprint Package_DIP:DIP-14_W7.62mm -> Package_DIP:DIP-16_W7.62mm
- U57: value 74LS08 -> 74LS245; footprint Package_DIP:DIP-14_W7.62mm -> Package_DIP:DIP-20_W7.62mm
- U58: value 7400 -> 74LS283; footprint Package_DIP:DIP-14_W7.62mm -> Package_DIP:DIP-16_W7.62mm
- U59: value 74LS245 -> 74LS85; footprint Package_DIP:DIP-20_W7.62mm -> Package_DIP:DIP-16_W7.62mm
- U62: value 74LS161-74xx -> 74LS245; footprint Package_DIP:DIP-16_W7.62mm -> Package_DIP:DIP-20_W7.62mm
- U63: value AT28C64B-15PU -> 74LS85; footprint ROM:ZIF-AT28C64B-15PU -> Package_DIP:DIP-16_W7.62mm
- U64: value AT28C64B-15PU -> 74LS245; footprint ROM:ZIF-AT28C64B-15PU -> Package_DIP:DIP-20_W7.62mm
- U65: value AT28C64B-15PU -> 74LS173; footprint ROM:ZIF-AT28C64B-15PU -> Package_DIP:DIP-16_W7.62mm
- U71: value 74LS173 -> 74HC00; footprint Package_DIP:DIP-16_W7.62mm -> Package_DIP:DIP-14_W7.62mm
- U73: value 74LS173 -> 74HC04; footprint Package_DIP:DIP-16_W7.62mm -> Package_DIP:DIP-14_W7.62mm
- U8, U9: value 74LS86 -> 74LS173; footprint Package_DIP:DIP-14_W7.62mm -> Package_DIP:DIP-16_W7.62mm
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Connections:
- D1 pad 2: /ALU/sheet61054F43/I0 -> /ALU/A0
- D10 pad 2: /ALU/sheet61054F43/I9 -> /ALU/A9
- D100 pad 2: /Register B/~AI -> /Sheet61DF6CC6/sheet623AC6D9/I13
- D101 pad 2: /Register B/~AO -> /Sheet61DF6CC6/sheet623AC6D9/I14
- D102 pad 2: /Resgister A/~AI -> /Sheet61DF6CC6/sheet623AC6D9/I15
- D103 pad 2: /Control Unit/~R2_AO -> /ALU/CF
- D104 pad 2: /RAM/~AI -> /ALU/ZF
- D105 pad 2: /RAM/~AO -> /ALU/ALTBF
- D106 pad 2: /RAM/~MEMOE -> /ALU/AGTBF
- D107 pad 2: /RAM/MEMWE -> /ALU/sheet61054F43/I0
- D108 pad 2: /Instruction Register/~II -> /ALU/sheet61054F43/I1
- D109 pad 2: /Instruction Register/~I0 -> /ALU/sheet61054F43/I2
- D11 pad 2: /ALU/sheet61054F43/I10 -> /ALU/A10
- D110 pad 2: /Instruction Register/~I80 -> /ALU/sheet61054F43/I3
- D111 pad 2: /ProgramCounter/~J -> /ALU/sheet61054F43/I4
- D112 pad 2: /ProgramCounter/CE -> /ALU/sheet61054F43/I5
- D113 pad 2: /ProgramCounter/~CO -> /ALU/sheet61054F43/I6
- D114 pad 2: /Control Unit/RESET_COUNTER -> /ALU/sheet61054F43/I7
- D115 pad 2: /Control Unit/~SI -> /ALU/sheet61054F43/I8
- D116 pad 2: /Control Unit/~SO -> /ALU/sheet61054F43/I9
- D117 pad 2: /Control Unit/~XI -> /ALU/sheet61054F43/I10
- D118 pad 2: /Control Unit/~XO -> /ALU/sheet61054F43/I11
- D119 pad 2: /Stack/sheet60C9B368/I0 -> /ALU/sheet61054F43/I12
- D12 pad 2: /ALU/sheet61054F43/I11 -> /ALU/A11
- D120 pad 2: /Stack/sheet60C9B368/I1 -> /ALU/sheet61054F43/I13
- D121 pad 2: /Stack/sheet60C9B368/I2 -> /ALU/sheet61054F43/I14
- D122 pad 2: /Stack/sheet60C9B368/I3 -> /ALU/sheet61054F43/I15
- D123 pad 2: /Stack/sheet60C9B368/I4 -> /ALU/sheet67DDEE7E/I0
- D124 pad 2: /Stack/sheet60C9B368/I5 -> /ALU/sheet67DDEE7E/I1
- D125 pad 2: /Stack/sheet60C9B368/I6 -> /ALU/sheet67DDEE7E/I2
- D126 pad 2: /Stack/sheet60C9B368/I7 -> /ALU/sheet67DDEE7E/I3
- D127 pad 2: /Stack/sheet60C9B368/I8 -> /ALU/sheet67DDEE7E/I4
- D128 pad 2: /Stack/sheet60C9B368/I9 -> /ALU/sheet67DDEE7E/I5
- D129 pad 2: /Stack/sheet60C9B368/I10 -> /ALU/sheet67DDEE7E/I6
- D13 pad 2: /ALU/sheet61054F43/I12 -> /ALU/A12
- D130 pad 2: /Stack/sheet60C9B368/I11 -> /ALU/sheet67DDEE7E/I7
- D131 pad 2: /Stack/sheet60C9B368/I12 -> /ALU/sheet67DDEE7E/I8
- D132 pad 2: /Stack/sheet60C9B368/I13 -> /ALU/sheet67DDEE7E/I9
- D133 pad 2: GND -> /ALU/sheet67DDEE7E/I10
- D134 pad 2: GND -> /ALU/sheet67DDEE7E/I11
- D135 pad 2: /Sheet61DF6CC6/sheet623AC6D9/I0 -> /ALU/sheet67DDEE7E/I12
- D136 pad 2: /Sheet61DF6CC6/sheet623AC6D9/I1 -> /ALU/sheet67DDEE7E/I13
- D137 pad 2: /Sheet61DF6CC6/sheet623AC6D9/I2 -> /ALU/sheet67DDEE7E/I14
- D138 pad 2: /Sheet61DF6CC6/sheet623AC6D9/I3 -> /ALU/sheet67DDEE7E/I15
- D139 pad 2: /Sheet61DF6CC6/sheet623AC6D9/I4 -> /Control Unit/I0
- D14 pad 2: /ALU/sheet61054F43/I13 -> /ALU/A13
- D140 pad 2: /Sheet61DF6CC6/sheet623AC6D9/I5 -> /Control Unit/I1
- D141 pad 2: /Sheet61DF6CC6/sheet623AC6D9/I6 -> /Control Unit/I2
- D142 pad 2: /Sheet61DF6CC6/sheet623AC6D9/I7 -> /Control Unit/I3
- D143 pad 2: /Sheet61DF6CC6/sheet623AC6D9/I8 -> /Control Unit/I4
- D144 pad 2: /Sheet61DF6CC6/sheet623AC6D9/I9 -> /Control Unit/I5
- D145 pad 2: /Sheet61DF6CC6/sheet623AC6D9/I10 -> /Control Unit/I6
- D146 pad 2: /Sheet61DF6CC6/sheet623AC6D9/I11 -> /Control Unit/I7
- D147 pad 2: /Sheet61DF6CC6/sheet623AC6D9/I12 -> /Instruction Register/sheet621E2544/I8
- D148 pad 2: /Sheet61DF6CC6/sheet623AC6D9/I13 -> /Instruction Register/sheet621E2544/I9
- D149 pad 2: /Sheet61DF6CC6/sheet623AC6D9/I14 -> /Instruction Register/sheet621E2544/I10
- D15 pad 2: /ALU/sheet61054F43/I14 -> /ALU/A14
- D150 pad 2: /Sheet61DF6CC6/sheet623AC6D9/I15 -> /Instruction Register/sheet621E2544/I11
- D151 pad 2: /ALU/BUS15 -> /Instruction Register/sheet621E2544/I12
- D152 pad 2: /ALU/BUS14 -> /Instruction Register/sheet621E2544/I13
- D153 pad 2: /ALU/BUS13 -> /Instruction Register/sheet621E2544/I10
- D154 pad 2: /ALU/BUS12 -> /Instruction Register/sheet621E2544/I11
- D155 pad 2: /ALU/BUS11 -> /ALU/BUS0
- D156 pad 2: /ALU/BUS10 -> /ALU/BUS1
- D157 pad 2: /ALU/BUS9 -> /ALU/BUS2
- D158 pad 2: /ALU/BUS8 -> /ALU/BUS3
- D159 pad 2: /ALU/BUS7 -> /ALU/BUS4
- D16 pad 2: /ALU/sheet61054F43/I15 -> /ALU/A15
- D160 pad 2: /ALU/BUS6 -> /ALU/BUS5
- D161 pad 2: /ALU/BUS5 -> /ALU/BUS6
- D162 pad 2: /ALU/BUS4 -> /ALU/BUS7
- D163 pad 2: /ALU/BUS3 -> /ALU/BUS8
- D164 pad 2: /ALU/BUS2 -> /ALU/BUS9
- D165 pad 2: /ALU/BUS1 -> /ALU/BUS10
- D166 pad 2: /ALU/BUS0 -> /ALU/BUS11
- D17 pad 2: /ALU/A0 -> /Register B/A0
- D18 pad 2: /ALU/A1 -> /Register B/A1
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Routing:
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
Commit message: using new ROM in CU and more jumps
Parts:
- removed C6: 0.01uF, Capacitor_THT:CP_Axial_L10.0mm_D4.5mm_P15.00mm_Horizontal
- removed R194: 220, Resistor_THT:R_Axial_DIN0204_L3.6mm_D1.6mm_P7.62mm_Horizontal
- removed the U20 at (-3.56, 339.5)
- removed the U53 at (-13.5, -203.2)
- removed the U54 at (-13.5, -180.9)
- removed the U55 at (-47.3, -186.0)
- removed the U56 at (-24.8, -180.9)
- removed the U61 at (-47.3, -208.3)
- removed the U72 at (170.0, 533.8)
- added U23: 74LS138, Package_DIP:DIP-16_W7.62mm, F.Cu at (45.2, 326.8)
- added U57: 74LS245, Package_DIP:DIP-20_W7.62mm, F.Cu at (4.43, 227.1)
- added U59: 74LS245, Package_DIP:DIP-20_W7.62mm, F.Cu at (-6.82, 227.1)
- added U66: 74LS173, Package_DIP:DIP-16_W7.62mm, F.Cu at (99.9, 64.7)
- added U68: 74LS173, Package_DIP:DIP-16_W7.62mm, F.Cu at (111.2, 87.0)
- added U69: 74LS173, Package_DIP:DIP-16_W7.62mm, F.Cu at (99.9, 87.0)
- added U76: 74LS173, Package_DIP:DIP-16_W7.62mm, F.Cu at (-68.6, 284.2)
- added U83: 74HC04, Package_DIP:DIP-14_W7.62mm, F.Cu at (-57.3, 307.0)
- R178: value 1K -> 220
- U20: renamed from U23; value AT28C64B-15PU -> 74LS161-74xx; footprint ROM:ZIF-AT28C64B-15PU -> Package_DIP:DIP-16_W7.62mm
- U21, U22: value AT28C64B-15PU -> AT28C256
- U24: value 74LS245 -> 74LS138; footprint Package_DIP:DIP-20_W7.62mm -> Package_DIP:DIP-16_W7.62mm
- U25: value 74LS173 -> 74LS138
- U26, U29, U32, U35, U74: value 74LS173 -> 74LS245; footprint Package_DIP:DIP-16_W7.62mm -> Package_DIP:DIP-20_W7.62mm
- U27, U30, U33, U67: value 74LS245 -> 74LS173; footprint Package_DIP:DIP-20_W7.62mm -> Package_DIP:DIP-16_W7.62mm
- U36: value LM555xN -> 74LS173; footprint Package_DIP:DIP-8_W7.62mm -> Package_DIP:DIP-16_W7.62mm
- U37: value 74LS04 -> 74LS173; footprint Package_DIP:DIP-14_W7.62mm -> Package_DIP:DIP-16_W7.62mm
- U38: value 74LS08 -> LM555xN; footprint Package_DIP:DIP-14_W7.62mm -> Package_DIP:DIP-8_W7.62mm
- U39: value 74LS32 -> 74LS04
- U40: value LM555xN -> 74LS08; footprint Package_DIP:DIP-8_W7.62mm -> Package_DIP:DIP-14_W7.62mm
- U41: value LM555xN -> 74LS32; footprint Package_DIP:DIP-8_W7.62mm -> Package_DIP:DIP-14_W7.62mm
- U42: value 74LS245 -> LM555xN; footprint Package_DIP:DIP-20_W7.62mm -> Package_DIP:DIP-8_W7.62mm
- U43: value 74LS00 -> LM555xN; footprint Package_DIP:DIP-14_W7.62mm -> Package_DIP:DIP-8_W7.62mm
- U44: value 74LS86 -> 74LS245; footprint Package_DIP:DIP-14_W7.62mm -> Package_DIP:DIP-20_W7.62mm
- U45: value 74LS86 -> 74LS00
- U47, U50: value 74LS00 -> 74LS86
- U49: value 74HC02 -> 74LS00
- U51: value 74LS00 -> 74HC02
- U52: value 74LS283 -> 74LS00; footprint Package_DIP:DIP-16_W7.62mm -> Package_DIP:DIP-14_W7.62mm
- U53: renamed from U57; value 74LS245 -> 74LS00; footprint Package_DIP:DIP-20_W7.62mm -> Package_DIP:DIP-14_W7.62mm
- U56: renamed from U60; value 74LS173 -> 74LS283
- U58: renamed from U62; value 74LS245 -> 74LS85; footprint Package_DIP:DIP-20_W7.62mm -> Package_DIP:DIP-16_W7.62mm
- U60: renamed from U64; value 74LS245 -> 74LS283; footprint Package_DIP:DIP-20_W7.62mm -> Package_DIP:DIP-16_W7.62mm
- U61: renamed from U65; value 74LS173 -> 74LS85
- U63: value 74LS85 -> 74LS283
- U64: renamed from U68; value 74LS173 -> 74LS245; footprint Package_DIP:DIP-16_W7.62mm -> Package_DIP:DIP-20_W7.62mm
- U65: renamed from U69; value 74LS173 -> 74LS85
- U71: value 74HC00 -> 74LS245; footprint Package_DIP:DIP-14_W7.62mm -> Package_DIP:DIP-20_W7.62mm
- U72: renamed from U76; value 74LS245 -> 74LS173; footprint Package_DIP:DIP-20_W7.62mm -> Package_DIP:DIP-16_W7.62mm
- U73: value 74HC04 -> 74LS173; footprint Package_DIP:DIP-14_W7.62mm -> Package_DIP:DIP-16_W7.62mm
- U77: value 74LS173 -> 74HC04; footprint Package_DIP:DIP-16_W7.62mm -> Package_DIP:DIP-14_W7.62mm
- U78: value 74LS173 -> 74HC00; footprint Package_DIP:DIP-16_W7.62mm -> Package_DIP:DIP-14_W7.62mm
- U79, U80: value AS6C6264 -> AT28C256; footprint Package_DIP:DIP-28_W15.24mm -> ROM:ZIF-AT28C64B-15PU
- U81, U82: value AT28C64B-15PU -> AS6C62256A; footprint ROM:ZIF-AT28C64B-15PU -> Package_DIP:DIP-28_W15.24mm
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- renumbered U58 to U54, U59 to U55, U66 to U62
Connections:
- D103 pad 2: /ALU/CF -> Net-(D103-Pad2)
- D104 pad 2: /ALU/ZF -> Net-(D104-Pad2)
- D105 pad 2: /ALU/ALTBF -> Net-(D105-Pad2)
- D106 pad 2: /ALU/AGTBF -> Net-(D106-Pad2)
- D153 pad 2: /Instruction Register/sheet621E2544/I10 -> /Instruction Register/sheet621E2544/I14
- D154 pad 2: /Instruction Register/sheet621E2544/I11 -> /Instruction Register/sheet621E2544/I15
- D185 pad 2: GND -> /RAM/sheet61B5B12C/I14
- D186 pad 2: GND -> /RAM/sheet61B5B12C/I15
- D51 pad 2: /Control Unit/~ALU_EO -> /RAM/MEMWE
- D52 pad 2: /Resgister A/~AI -> /ProgramCounter/CE
- D54 pad 2: /Register B/~AI -> /Register B/~AO
- D55 pad 2: /Register B/~AO -> /RAM/~AO
- D56 pad 2: /RAM/~AI -> /ProgramCounter/~CO
- D57 pad 2: /RAM/~AO -> /Instruction Register/~I80
- D58 pad 2: /RAM/~MEMOE -> /Control Unit/~XO
- D59 pad 2: /RAM/MEMWE -> /Control Unit/~SO
- D60 pad 2: /Instruction Register/~II -> /RAM/~MEMOE
- D61 pad 2: /Instruction Register/~I0 -> /Control Unit/~SO
- D62 pad 2: /Instruction Register/~I80 -> /Control Unit/~ALU_EO
- D63 pad 2: /ProgramCounter/~J -> /Control Unit/~ALU_NAND_O
- D64 pad 2: /ProgramCounter/CE -> /Resgister A/~AI
- D65 pad 2: /ProgramCounter/~CO -> /Register B/~AI
- D66 pad 2: /Control Unit/RESET_COUNTER -> /RAM/~AI
- D67 pad 2: /Control Unit/~SI -> /ProgramCounter/~J
- D68 pad 2: /Control Unit/~SO -> /Instruction Register/~II
- D70 pad 2: /Control Unit/~XO -> /Control Unit/~SI
- D85 pad 2: GND -> /Stack/sheet60C9B368/I14
- D86 pad 2: GND -> /Stack/sheet60C9B368/I15
- R178 pad 1: Net-(C6-Pad2) -> Net-(D171-Pad1)
- R179 pad 1: Net-(D171-Pad1) -> Net-(D172-Pad1)
- R180 pad 1: Net-(D172-Pad1) -> Net-(D173-Pad1)
- R181 pad 1: Net-(D173-Pad1) -> Net-(D174-Pad1)
- R182 pad 1: Net-(D174-Pad1) -> Net-(D175-Pad1)
- R183 pad 1: Net-(D175-Pad1) -> Net-(D176-Pad1)
- R184 pad 1: Net-(D176-Pad1) -> Net-(D177-Pad1)
- R185 pad 1: Net-(D177-Pad1) -> Net-(D178-Pad1)
- R186 pad 1: Net-(D178-Pad1) -> Net-(D179-Pad1)
- R187 pad 1: Net-(D179-Pad1) -> Net-(D180-Pad1)
- R188 pad 1: Net-(D180-Pad1) -> Net-(D181-Pad1)
- R189 pad 1: Net-(D181-Pad1) -> Net-(D182-Pad1)
- R190 pad 1: Net-(D182-Pad1) -> Net-(D183-Pad1)
- R191 pad 1: Net-(D183-Pad1) -> Net-(D184-Pad1)
- R192 pad 1: Net-(D184-Pad1) -> Net-(D185-Pad1)
- R193 pad 1: Net-(D185-Pad1) -> Net-(D186-Pad1)
- U20 pad 1: (no net) -> Net-(U19-Pad6)
- U20 pad 10: /Control Unit/I0 -> +5V
- U20 pad 11: /RAM/~AO -> Net-(U20-Pad11)
- U20 pad 12: /RAM/~MEMOE -> Net-(U20-Pad12)
- U20 pad 13: /RAM/MEMWE -> Net-(U20-Pad13)
- U20 pad 14: GND -> Net-(U20-Pad14)
- U20 pad 15: /Instruction Register/~II -> Net-(U20-Pad15)
- U20 pad 16: /Instruction Register/~I0 -> +5V
- U20 pad 2: /ALU/CF -> /ALU/CLK
- U20 pad 3: /Control Unit/I7 -> Net-(U20-Pad3)
- U20 pad 4: /Control Unit/I6 -> Net-(U20-Pad4)
- U20 pad 5: /Control Unit/I5 -> Net-(U20-Pad5)
- U20 pad 6: /Control Unit/I4 -> Net-(U20-Pad6)
- U20 pad 7: /Control Unit/I3 -> +5V
- U20 pad 8: /Control Unit/I2 -> GND
- U20 pad 9: /Control Unit/I1 -> +5V
- U21 pad 1: (no net) -> /Control Unit/AGTBF
- U21 pad 11: /ProgramCounter/~CO -> Net-(U21-Pad11)
- U21 pad 12: /Control Unit/RESET_COUNTER -> Net-(U21-Pad12)
- U21 pad 13: /Control Unit/~SI -> Net-(U21-Pad13)
- U21 pad 15: /Control Unit/~SO -> Net-(U21-Pad15)
- U21 pad 16: /Control Unit/~XI -> Net-(U21-Pad16)
- U21 pad 17: /Control Unit/~XO -> Net-(U21-Pad17)
- U21 pad 18: Net-(U21-Pad18) -> /Control Unit/~ALU_FI
- U21 pad 19: Net-(U21-Pad19) -> /Control Unit/ALU_SU
- U21 pad 20: Net-(U21-Pad20) -> GND
- U21 pad 22: Net-(U21-Pad22) -> GND
- U21 pad 26: (no net) -> /Control Unit/ALTBF
- U22 pad 1: (no net) -> /Control Unit/AGTBF
- U22 pad 11: /Control Unit/~ALU_FI -> /RAM/MEMWE
- U22 pad 12: /Control Unit/ALU_SU -> /ProgramCounter/CE
- U22 pad 13: /Control Unit/~ALU_EO -> Net-(U22-Pad13)
- U22 pad 15: /Resgister A/~AI -> Net-(U22-Pad15)
- U22 pad 16: /Resgister A/~AO -> Net-(U22-Pad16)
- U22 pad 17: /Register B/~AI -> Net-(U22-Pad17)
- U22 pad 18: /Register B/~AO -> Net-(U22-Pad18)
- U22 pad 19: /RAM/~AI -> /Control Unit/RESET_COUNTER
- U22 pad 20: Net-(U22-Pad20) -> GND
- U22 pad 22: Net-(U22-Pad22) -> GND
- U22 pad 26: (no net) -> /Control Unit/ALTBF
- U24 pad 1: +5V -> Net-(U21-Pad15)
- U24 pad 10: GND -> Net-(U24-Pad10)
- U24 pad 11: /ALU/BUS7 -> /Control Unit/~ALU_NAND_O
- U24 pad 12: /ALU/BUS6 -> /Control Unit/~ALU_EO
- U24 pad 13: /ALU/BUS5 -> /Control Unit/~SO
- U24 pad 14: /ALU/BUS4 -> /RAM/~MEMOE
- U24 pad 15: /ALU/BUS3 -> Net-(U24-Pad15)
- U24 pad 16: /ALU/BUS2 -> +5V
- U24 pad 2: /Stack/sheet60C9B368/I0 -> Net-(U21-Pad16)
- U24 pad 3: /Stack/sheet60C9B368/I1 -> Net-(U21-Pad17)
- U24 pad 4: /Stack/sheet60C9B368/I2 -> GND
- U24 pad 5: /Stack/sheet60C9B368/I3 -> GND
- U24 pad 6: /Stack/sheet60C9B368/I4 -> +5V
- U24 pad 7: /Stack/sheet60C9B368/I5 -> Net-(U24-Pad7)
- U24 pad 8: /Stack/sheet60C9B368/I6 -> GND
- U24 pad 9: /Stack/sheet60C9B368/I7 -> Net-(U24-Pad9)
- U25 pad 1: GND -> Net-(U22-Pad16)
- U25 pad 10: /Control Unit/~SI -> /Instruction Register/~II
- U25 pad 11: /ALU/BUS3 -> /ProgramCounter/~J
- U25 pad 12: /ALU/BUS2 -> /RAM/~AI
- U25 pad 13: /ALU/BUS1 -> /Register B/~AI
- U25 pad 14: /ALU/BUS0 -> /Resgister A/~AI
- U25 pad 15: /Stack/CLR -> Net-(U25-Pad15)
- U25 pad 2: GND -> Net-(U22-Pad17)
- U25 pad 3: /Stack/sheet60C9B368/I0 -> Net-(U22-Pad18)
- U25 pad 4: /Stack/sheet60C9B368/I1 -> GND
- U25 pad 5: /Stack/sheet60C9B368/I2 -> GND
- U25 pad 6: /Stack/sheet60C9B368/I3 -> +5V
- U25 pad 7: /ALU/CLK -> /Control Unit/~SI
- U25 pad 9: /Control Unit/~SI -> /Control Unit/~XI
- U26 pad 1: GND -> +5V
- U26 pad 10: /Control Unit/~SI -> GND
- U26 pad 15: /Stack/CLR -> /ALU/BUS3
- U26 pad 16: +5V -> /ALU/BUS2
- U26 pad 2: GND -> /Stack/sheet60C9B368/I0
- U26 pad 3: /Stack/sheet60C9B368/I4 -> /Stack/sheet60C9B368/I1
- U26 pad 4: /Stack/sheet60C9B368/I5 -> /Stack/sheet60C9B368/I2
- U26 pad 5: /Stack/sheet60C9B368/I6 -> /Stack/sheet60C9B368/I3
- U26 pad 6: /Stack/sheet60C9B368/I7 -> /Stack/sheet60C9B368/I4
- U26 pad 7: /ALU/CLK -> /Stack/sheet60C9B368/I5
- U26 pad 8: GND -> /Stack/sheet60C9B368/I6
- U26 pad 9: /Control Unit/~SI -> /Stack/sheet60C9B368/I7
- U27 pad 1: +5V -> GND
- U27 pad 10: GND -> /Control Unit/~SI
- U27 pad 11: /ALU/BUS15 -> /ALU/BUS3
- U27 pad 12: /ALU/BUS14 -> /ALU/BUS2
- U27 pad 13: /ALU/BUS13 -> /ALU/BUS1
- U27 pad 14: /ALU/BUS12 -> /ALU/BUS0
- U27 pad 15: /ALU/BUS11 -> /Stack/CLR
- U27 pad 16: /ALU/BUS10 -> +5V
- U27 pad 2: /Stack/sheet60C9B368/I8 -> GND
- U27 pad 3: /Stack/sheet60C9B368/I9 -> /Stack/sheet60C9B368/I0
- U27 pad 4: /Stack/sheet60C9B368/I10 -> /Stack/sheet60C9B368/I1
- U27 pad 5: /Stack/sheet60C9B368/I11 -> /Stack/sheet60C9B368/I2
- U27 pad 6: /Stack/sheet60C9B368/I12 -> /Stack/sheet60C9B368/I3
- U27 pad 7: /Stack/sheet60C9B368/I13 -> /ALU/CLK
- U27 pad 8: Net-(U27-Pad8) -> GND
- U27 pad 9: Net-(U27-Pad9) -> /Control Unit/~SI
- U28 pad 11: /ALU/BUS11 -> /ALU/BUS7
- U28 pad 12: /ALU/BUS10 -> /ALU/BUS6
- U28 pad 13: /ALU/BUS9 -> /ALU/BUS5
- U28 pad 14: /ALU/BUS8 -> /ALU/BUS4
- U28 pad 3: /Stack/sheet60C9B368/I8 -> /Stack/sheet60C9B368/I4
- U28 pad 4: /Stack/sheet60C9B368/I9 -> /Stack/sheet60C9B368/I5
- U28 pad 5: /Stack/sheet60C9B368/I10 -> /Stack/sheet60C9B368/I6
- U28 pad 6: /Stack/sheet60C9B368/I11 -> /Stack/sheet60C9B368/I7
- U29 pad 1: GND -> +5V
- U29 pad 10: /Control Unit/~SI -> GND
- U29 pad 15: /Stack/CLR -> /ALU/BUS11
- U29 pad 16: +5V -> /ALU/BUS10
- U29 pad 2: GND -> /Stack/sheet60C9B368/I8
- U29 pad 3: /Stack/sheet60C9B368/I12 -> /Stack/sheet60C9B368/I9
- U29 pad 4: /Stack/sheet60C9B368/I13 -> /Stack/sheet60C9B368/I10
- U29 pad 5: GND -> /Stack/sheet60C9B368/I11
- U29 pad 6: GND -> /Stack/sheet60C9B368/I12
- U29 pad 7: /ALU/CLK -> /Stack/sheet60C9B368/I13
- U29 pad 8: GND -> /Stack/sheet60C9B368/I14
- U29 pad 9: /Control Unit/~SI -> /Stack/sheet60C9B368/I15
- U30 pad 1: +5V -> GND
- U30 pad 10: GND -> /Control Unit/~SI
- U30 pad 11: /ALU/BUS7 -> /ALU/BUS11
- U30 pad 12: /ALU/BUS6 -> /ALU/BUS10
- U30 pad 13: /ALU/BUS5 -> /ALU/BUS9
- U30 pad 14: /ALU/BUS4 -> /ALU/BUS8
- U30 pad 15: /ALU/BUS3 -> /Stack/CLR
- U30 pad 16: /ALU/BUS2 -> +5V
- U30 pad 2: /Sheet61DF6CC6/sheet623AC6D9/I0 -> GND
- U30 pad 3: /Sheet61DF6CC6/sheet623AC6D9/I1 -> /Stack/sheet60C9B368/I8
- U30 pad 4: /Sheet61DF6CC6/sheet623AC6D9/I2 -> /Stack/sheet60C9B368/I9
- U30 pad 5: /Sheet61DF6CC6/sheet623AC6D9/I3 -> /Stack/sheet60C9B368/I10
- U30 pad 6: /Sheet61DF6CC6/sheet623AC6D9/I4 -> /Stack/sheet60C9B368/I11
- U30 pad 7: /Sheet61DF6CC6/sheet623AC6D9/I5 -> /ALU/CLK
- U30 pad 8: /Sheet61DF6CC6/sheet623AC6D9/I6 -> GND
- U30 pad 9: /Sheet61DF6CC6/sheet623AC6D9/I7 -> /Control Unit/~SI
- U31 pad 10: /Control Unit/~XI -> /Control Unit/~SI
- U31 pad 11: /ALU/BUS3 -> /ALU/BUS15
- U31 pad 12: /ALU/BUS2 -> /ALU/BUS14
- U31 pad 13: /ALU/BUS1 -> /ALU/BUS13
- U31 pad 14: /ALU/BUS0 -> /ALU/BUS12
- U31 pad 15: /Sheet61DF6CC6/CLR -> /Stack/CLR
- U31 pad 3: /Sheet61DF6CC6/sheet623AC6D9/I0 -> /Stack/sheet60C9B368/I12
- U31 pad 4: /Sheet61DF6CC6/sheet623AC6D9/I1 -> /Stack/sheet60C9B368/I13
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
Commit message: Added power connector
Parts:
- removed D63: LED, LED_THT:LED_D3.0mm
- removed R64: 220, Resistor_THT:R_Axial_DIN0204_L3.6mm_D1.6mm_P7.62mm_Horizontal
- added C10: 0.1uF, Capacitor_THT:CP_Axial_L10.0mm_D4.5mm_P15.00mm_Horizontal, F.Cu at (177.8, 61.5)
- added C11: 0.1uF, Capacitor_THT:CP_Axial_L10.0mm_D4.5mm_P15.00mm_Horizontal, F.Cu at (177.8, 68.4)
- added C12: 0.1uF, Capacitor_THT:CP_Axial_L10.0mm_D4.5mm_P15.00mm_Horizontal, F.Cu at (137.8, -51.5)
- added C13: 0.1uF, Capacitor_THT:CP_Axial_L10.0mm_D4.5mm_P15.00mm_Horizontal, F.Cu at (137.8, -44.5)
- added C14: 0.1uF, Capacitor_THT:CP_Axial_L10.0mm_D4.5mm_P15.00mm_Horizontal, F.Cu at (64.8, -51.5)
- added C15: 0.1uF, Capacitor_THT:CP_Axial_L10.0mm_D4.5mm_P15.00mm_Horizontal, F.Cu at (64.8, -44.5)
- added C16: 0.1uF, Capacitor_THT:CP_Axial_L10.0mm_D4.5mm_P15.00mm_Horizontal, F.Cu at (-27.8, 44.8)
- added C17: 0.1uF, Capacitor_THT:CP_Axial_L10.0mm_D4.5mm_P15.00mm_Horizontal, F.Cu at (-27.8, 76.7)
- added C18: 0.1uF, Capacitor_THT:CP_Axial_L10.0mm_D4.5mm_P15.00mm_Horizontal, F.Cu at (76.0, 19.4)
- added C19: 0.1uF, Capacitor_THT:CP_Axial_L10.0mm_D4.5mm_P15.00mm_Horizontal, F.Cu at (76.0, 26.3)
- added C20: 0.1uF, Capacitor_THT:CP_Axial_L10.0mm_D4.5mm_P15.00mm_Horizontal, F.Cu at (98.5, 19.4)
- added C21: 0.1uF, Capacitor_THT:CP_Axial_L10.0mm_D4.5mm_P15.00mm_Horizontal, F.Cu at (98.5, 26.3)
- added C22: 0.1uF, Capacitor_THT:CP_Axial_L10.0mm_D4.5mm_P15.00mm_Horizontal, F.Cu at (-26.4, -48.6)
- added C23: 0.1uF, Capacitor_THT:CP_Axial_L10.0mm_D4.5mm_P15.00mm_Horizontal, F.Cu at (-45.3, -48.6)
- added C24: 0.1uF, Capacitor_THT:CP_Axial_L10.0mm_D4.5mm_P15.00mm_Horizontal, F.Cu at (-56.6, 123.8)
- added C25: 0.1uF, Capacitor_THT:CP_Axial_L10.0mm_D4.5mm_P15.00mm_Horizontal, F.Cu at (-56.6, 130.8)
- added C26: 0.1uF, Capacitor_THT:CP_Axial_L10.0mm_D4.5mm_P15.00mm_Horizontal, F.Cu at (-56.6, 137.7)
- added C27: 0.1uF, Capacitor_THT:CP_Axial_L10.0mm_D4.5mm_P15.00mm_Horizontal, F.Cu at (14.3, 129.8)
- added C28: 0.1uF, Capacitor_THT:CP_Axial_L10.0mm_D4.5mm_P15.00mm_Horizontal, F.Cu at (64.8, 130.8)
- added C29: 0.1uF, Capacitor_THT:CP_Axial_L10.0mm_D4.5mm_P15.00mm_Horizontal, F.Cu at (128.1, 136.2)
- added C30: 0.1uF, Capacitor_THT:CP_Axial_L10.0mm_D4.5mm_P15.00mm_Horizontal, F.Cu at (64.8, 137.7)
- added C31: 0.1uF, Capacitor_THT:CP_Axial_L10.0mm_D4.5mm_P15.00mm_Horizontal, F.Cu at (90.8, 137.7)
- added C6: 0.1uF, Capacitor_THT:CP_Axial_L10.0mm_D4.5mm_P15.00mm_Horizontal, F.Cu at (210.8, -51.5)
- added C7: 0.1uF, Capacitor_THT:CP_Axial_L10.0mm_D4.5mm_P15.00mm_Horizontal, F.Cu at (210.8, -44.5)
- added C8: 0.1uF, Capacitor_THT:CP_Axial_L10.0mm_D4.5mm_P15.00mm_Horizontal, F.Cu at (186.2, 182.8)
- added C9: 0.1uF, Capacitor_THT:CP_Axial_L10.0mm_D4.5mm_P15.00mm_Horizontal, F.Cu at (186.2, 189.7)
- added J1: ATX24RH, ROM:ATX24_RIGHT_ANGLE, F.Cu at (-31.8, -90.3)
- added SW4: SW_SPDT-Switch, ROM:SW_MINI-SPDT-SW, F.Cu at (-51.1, -106.0)
- SW3: footprint ROM:DPDT-pushbutton -> ROM:SW_MINI-SPDT-SW
- U19: value 7400 -> LMC555xN; footprint Package_DIP:DIP-14_W7.62mm -> Package_DIP:DIP-8_W7.62mm
- U20: value 74LS161-74xx -> LMC555xN; footprint Package_DIP:DIP-16_W7.62mm -> Package_DIP:DIP-8_W7.62mm
- U21: value AT28C256 -> LMC555xN; footprint ROM:ZIF-AT28C64B-15PU -> Package_DIP:DIP-8_W7.62mm
- U22: value AT28C256 -> 7400; footprint ROM:ZIF-AT28C64B-15PU -> Package_DIP:DIP-14_W7.62mm
- U23: value 74LS138 -> 74LS161-74xx
- U24, U25: value 74LS138 -> AT28C256; footprint Package_DIP:DIP-16_W7.62mm -> ROM:ZIF-AT28C64B-15PU
- U38, U42, U43: value LM555xN -> 74LS138; footprint Package_DIP:DIP-8_W7.62mm -> Package_DIP:DIP-16_W7.62mm
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Connections:
- net /Instruction Register/sheet621E2544/I10 renamed /Instruction-Register/sheet621E2544/I10
- net /Instruction Register/sheet621E2544/I11 renamed /Instruction-Register/sheet621E2544/I11
- net /Instruction Register/sheet621E2544/I12 renamed /Instruction-Register/sheet621E2544/I12
- net /Instruction Register/sheet621E2544/I13 renamed /Instruction-Register/sheet621E2544/I13
- net /Instruction Register/sheet621E2544/I14 renamed /Instruction-Register/sheet621E2544/I14
- net /Instruction Register/sheet621E2544/I15 renamed /Instruction-Register/sheet621E2544/I15
- net /Instruction Register/sheet621E2544/I8 renamed /Instruction-Register/sheet621E2544/I8
- net /Instruction Register/sheet621E2544/I9 renamed /Instruction-Register/sheet621E2544/I9
- net /Register B/A0 renamed /Register-B/A0
- net /Register B/A1 renamed /Register-B/A1
- net /Register B/A10 renamed /Register-B/A10
- net /Register B/A11 renamed /Register-B/A11
- net /Register B/A12 renamed /Register-B/A12
- net /Register B/A13 renamed /Register-B/A13
- net /Register B/A14 renamed /Register-B/A14
- net /Register B/A15 renamed /Register-B/A15
- net /Register B/A2 renamed /Register-B/A2
- net /Register B/A3 renamed /Register-B/A3
- net /Register B/A4 renamed /Register-B/A4
- net /Register B/A5 renamed /Register-B/A5
- net /Register B/A6 renamed /Register-B/A6
- net /Register B/A7 renamed /Register-B/A7
- net /Register B/A8 renamed /Register-B/A8
- net /Register B/A9 renamed /Register-B/A9
- D139 pad 2: /Control Unit/I0 -> /Control-Unit/I0
- D140 pad 2: /Control Unit/I1 -> /Control-Unit/I1
- D141 pad 2: /Control Unit/I2 -> /Control-Unit/I2
- D142 pad 2: /Control Unit/I3 -> /Control-Unit/I3
- D143 pad 2: /Control Unit/I4 -> /Control-Unit/I4
- D144 pad 2: /Control Unit/I5 -> /Control-Unit/I5
- D145 pad 2: /Control Unit/I6 -> /Control-Unit/I6
- D146 pad 2: /Control Unit/I7 -> /Control-Unit/I7
- D49 pad 2: /Control Unit/~ALU_FI -> /Control-Unit/~ALU_FI
- D50 pad 2: /Control Unit/ALU_SU -> /Control-Unit/ALU_SU
- D53 pad 2: /Resgister A/~AO -> /Resgister-A/~AO
- D54 pad 2: /Register B/~AO -> /Register-B/~AO
- D57 pad 2: /Instruction Register/~I80 -> /Instruction-Register/~I80
- D58 pad 2: /Control Unit/~XO -> /Control-Unit/~XO
- D59 pad 2: /Control Unit/~SO -> /Control-Unit/~SO
- D61 pad 2: /Control Unit/~SO -> /Control-Unit/~ALU_EO
- D62 pad 2: /Control Unit/~ALU_EO -> /Control-Unit/~ALU_NAND_O
- D64 pad 2: /Resgister A/~AI -> /Resgister-A/~AI
- D65 pad 2: /Register B/~AI -> /Register-B/~AI
- D68 pad 2: /Instruction Register/~II -> /Instruction-Register/~II
- D69 pad 2: /Control Unit/~XI -> /Control-Unit/~XI
- D70 pad 2: /Control Unit/~SI -> /Control-Unit/~SI
- U1 pad 19: /Resgister A/~AO -> /Resgister-A/~AO
- U10 pad 19: /Register B/~AO -> /Register-B/~AO
- U11 pad 10: /Register B/~AI -> /Register-B/~AI
- U11 pad 15: /Register B/CLR -> /ALU/CLR
- U11 pad 9: /Register B/~AI -> /Register-B/~AI
- U12 pad 10: /Register B/~AI -> /Register-B/~AI
- U12 pad 15: /Register B/CLR -> /ALU/CLR
- U12 pad 9: /Register B/~AI -> /Register-B/~AI
- U15 pad 1: /ProgramCounter/~CLR -> /ALU/CLR
- U16 pad 1: /ProgramCounter/~CLR -> /ALU/CLR
- U17 pad 1: /ProgramCounter/~CLR -> /ALU/CLR
- U18 pad 1: /ProgramCounter/~CLR -> /ALU/CLR
- U19 pad 1: /Control Unit/~CLR -> GND
- U19 pad 2: /Control Unit/RESET_COUNTER -> Net-(C2-Pad1)
- U19 pad 4: Net-(U19-Pad3) -> +5V
- U19 pad 5: Net-(U19-Pad3) -> Net-(C1-Pad1)
- U19 pad 6: Net-(U19-Pad6) -> Net-(C2-Pad1)
- U19 pad 7: GND -> Net-(R104-Pad2)
- U19 pad 8: /Control Unit/CLR -> +5V
- U2 pad 10: /Resgister A/~AI -> /Resgister-A/~AI
- U2 pad 15: /Resgister A/CLR -> /ALU/CLR
- U2 pad 9: /Resgister A/~AI -> /Resgister-A/~AI
- U20 pad 1: Net-(U19-Pad6) -> GND
- U20 pad 2: /ALU/CLK -> Net-(R106-Pad2)
- U20 pad 4: Net-(U20-Pad4) -> +5V
- U20 pad 5: Net-(U20-Pad5) -> Net-(C3-Pad1)
- U20 pad 6: Net-(U20-Pad6) -> Net-(C4-Pad1)
- U20 pad 7: +5V -> Net-(C4-Pad1)
- U20 pad 8: GND -> +5V
- U21 pad 1: /Control Unit/AGTBF -> GND
- U21 pad 2: /ALU/CF -> Net-(R108-Pad2)
- U21 pad 3: /Control Unit/I7 -> Net-(U21-Pad3)
- U21 pad 4: /Control Unit/I6 -> Net-(R109-Pad2)
- U21 pad 5: /Control Unit/I5 -> Net-(C5-Pad1)
- U21 pad 6: /Control Unit/I4 -> GND
- U21 pad 7: /Control Unit/I3 -> Net-(U21-Pad7)
- U21 pad 8: /Control Unit/I2 -> +5V
- U22 pad 1: /Control Unit/AGTBF -> /Control-Unit/~CLR
- U22 pad 10: /Control Unit/I0 -> /Control-Unit/~CLR
- U22 pad 11: /RAM/MEMWE -> /Control-Unit/~CLR
- U22 pad 12: /ProgramCounter/CE -> Net-(R49-Pad1)
- U22 pad 13: Net-(U22-Pad13) -> Net-(R49-Pad1)
- U22 pad 14: GND -> +5V
- U22 pad 2: /ALU/CF -> /Control-Unit/RESET_COUNTER
- U22 pad 3: /Control Unit/I7 -> Net-(U22-Pad3)
- U22 pad 4: /Control Unit/I6 -> Net-(U22-Pad3)
- U22 pad 5: /Control Unit/I5 -> Net-(U22-Pad3)
- U22 pad 6: /Control Unit/I4 -> Net-(U22-Pad6)
- U22 pad 7: /Control Unit/I3 -> GND
- U22 pad 8: /Control Unit/I2 -> /ALU/CLR
- U22 pad 9: /Control Unit/I1 -> /Control-Unit/~CLR
- U23 pad 1: Net-(U21-Pad11) -> Net-(U22-Pad6)
- U23 pad 10: /Instruction Register/~I80 -> +5V
- U23 pad 11: /ProgramCounter/~CO -> Net-(U23-Pad11)
- U23 pad 12: /RAM/~AO -> Net-(U23-Pad12)
- U23 pad 13: /Register B/~AO -> Net-(U23-Pad13)
- U23 pad 14: /Resgister A/~AO -> Net-(U23-Pad14)
- U23 pad 2: Net-(U21-Pad12) -> /ALU/CLK
- U23 pad 3: Net-(U21-Pad13) -> Net-(U23-Pad3)
- U23 pad 4: GND -> Net-(U23-Pad4)
- U23 pad 5: GND -> Net-(U23-Pad5)
- U23 pad 6: +5V -> Net-(U23-Pad6)
- U23 pad 7: /Control Unit/~SO -> +5V
- U23 pad 9: /Control Unit/~XO -> +5V
- U24 pad 1: Net-(U21-Pad15) -> /ALU/AGTBF
- U24 pad 10: Net-(U24-Pad10) -> /Control-Unit/I0
- U24 pad 11: /Control Unit/~ALU_NAND_O -> Net-(U24-Pad11)
- U24 pad 12: /Control Unit/~ALU_EO -> Net-(U24-Pad12)
- U24 pad 13: /Control Unit/~SO -> Net-(U24-Pad13)
- U24 pad 14: /RAM/~MEMOE -> GND
- U24 pad 16: +5V -> Net-(U24-Pad16)
- U24 pad 2: Net-(U21-Pad16) -> /ALU/CF
- U24 pad 3: Net-(U21-Pad17) -> /Control-Unit/I7
- U24 pad 4: GND -> /Control-Unit/I6
- U24 pad 5: GND -> /Control-Unit/I5
- U24 pad 6: +5V -> /Control-Unit/I4
- U24 pad 7: Net-(U24-Pad7) -> /Control-Unit/I3
- U24 pad 8: GND -> /Control-Unit/I2
- U24 pad 9: Net-(U24-Pad9) -> /Control-Unit/I1
- U25 pad 1: Net-(U22-Pad16) -> /ALU/AGTBF
- U25 pad 10: /Instruction Register/~II -> /Control-Unit/I0
- U25 pad 11: /ProgramCounter/~J -> /RAM/MEMWE
- U25 pad 12: /RAM/~AI -> /ProgramCounter/CE
- U25 pad 13: /Register B/~AI -> Net-(U25-Pad13)
- U25 pad 14: /Resgister A/~AI -> GND
- U25 pad 16: +5V -> Net-(U25-Pad16)
- U25 pad 2: Net-(U22-Pad17) -> /ALU/CF
- U25 pad 3: Net-(U22-Pad18) -> /Control-Unit/I7
- U25 pad 4: GND -> /Control-Unit/I6
- U25 pad 5: GND -> /Control-Unit/I5
- U25 pad 6: +5V -> /Control-Unit/I4
- U25 pad 7: /Control Unit/~SI -> /Control-Unit/I3
- U25 pad 8: GND -> /Control-Unit/I2
- U25 pad 9: /Control Unit/~XI -> /Control-Unit/I1
- U26 pad 19: /Control Unit/~SO -> /Control-Unit/~SO
- U27 pad 10: /Control Unit/~SI -> /Control-Unit/~SI
- U27 pad 15: /Stack/CLR -> /ALU/CLR
- U27 pad 9: /Control Unit/~SI -> /Control-Unit/~SI
- U28 pad 10: /Control Unit/~SI -> /Control-Unit/~SI
- U28 pad 15: /Stack/CLR -> /ALU/CLR
- U28 pad 9: /Control Unit/~SI -> /Control-Unit/~SI
- U29 pad 19: /Control Unit/~SO -> /Control-Unit/~SO
- U3 pad 10: /Resgister A/~AI -> /Resgister-A/~AI
- U3 pad 15: /Resgister A/CLR -> /ALU/CLR
- U3 pad 9: /Resgister A/~AI -> /Resgister-A/~AI
- U30 pad 10: /Control Unit/~SI -> /Control-Unit/~SI
- U30 pad 15: /Stack/CLR -> /ALU/CLR
- U30 pad 9: /Control Unit/~SI -> /Control-Unit/~SI
- U31 pad 10: /Control Unit/~SI -> /Control-Unit/~SI
- U31 pad 15: /Stack/CLR -> /ALU/CLR
- U31 pad 9: /Control Unit/~SI -> /Control-Unit/~SI
- U32 pad 19: /Control Unit/~XO -> /Control-Unit/~XO
- U33 pad 10: /Control Unit/~XI -> /Control-Unit/~XI
- U33 pad 15: /Sheet61DF6CC6/CLR -> /ALU/CLR
- U33 pad 9: /Control Unit/~XI -> /Control-Unit/~XI
- U34 pad 10: /Control Unit/~XI -> /Control-Unit/~XI
- U34 pad 15: /Sheet61DF6CC6/CLR -> /ALU/CLR
- U34 pad 9: /Control Unit/~XI -> /Control-Unit/~XI
- U35 pad 19: /Control Unit/~XO -> /Control-Unit/~XO
- U36 pad 10: /Control Unit/~XI -> /Control-Unit/~XI
- U36 pad 15: /Sheet61DF6CC6/CLR -> /ALU/CLR
- U36 pad 9: /Control Unit/~XI -> /Control-Unit/~XI
- U37 pad 10: /Control Unit/~XI -> /Control-Unit/~XI
- U37 pad 15: /Sheet61DF6CC6/CLR -> /ALU/CLR
- U37 pad 9: /Control Unit/~XI -> /Control-Unit/~XI
- U38 pad 1: GND -> Net-(U24-Pad11)
- U38 pad 2: Net-(C2-Pad1) -> Net-(U24-Pad12)
- U38 pad 3: Net-(U38-Pad3) -> Net-(U24-Pad13)
- U38 pad 4: +5V -> GND
- U38 pad 5: Net-(C1-Pad1) -> GND
- U38 pad 6: Net-(C2-Pad1) -> +5V
- U38 pad 7: Net-(R104-Pad2) -> /Control-Unit/~SO
- U38 pad 8: +5V -> GND
- U39 pad 1: Net-(U39-Pad1) -> Net-(U21-Pad3)
- U4 pad 19: /Resgister A/~AO -> /Resgister-A/~AO
- U40 pad 1: Net-(U38-Pad3) -> Net-(U19-Pad3)
- U40 pad 2: Net-(U39-Pad1) -> Net-(U21-Pad3)
- U40 pad 5: Net-(U40-Pad5) -> Net-(U20-Pad3)
- U42 pad 1: GND -> Net-(U24-Pad15)
- U42 pad 2: Net-(R106-Pad2) -> Net-(U24-Pad16)
- U42 pad 3: Net-(U40-Pad5) -> Net-(U24-Pad17)
- U42 pad 4: +5V -> GND
- U42 pad 5: Net-(C3-Pad1) -> GND
- U42 pad 6: Net-(C4-Pad1) -> +5V
- U42 pad 7: Net-(C4-Pad1) -> Net-(U42-Pad7)
- U42 pad 8: +5V -> GND
- U43 pad 1: GND -> Net-(U25-Pad16)
- U43 pad 2: Net-(R108-Pad2) -> Net-(U25-Pad17)
- U43 pad 3: Net-(U39-Pad1) -> Net-(U25-Pad18)
- U43 pad 4: Net-(R109-Pad2) -> GND
- U43 pad 5: Net-(C5-Pad1) -> GND
- U43 pad 6: GND -> +5V
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