File: 16bitCpu.kicad_pcb (KiCad board)
At the start: 2 copper layers, 497 parts, among them J1 ATX24RH, SW1 SW_Push-Switch, SW2 SW_Push, SW3 SW_SPDT, SW4 SW_SPDT-Switch, U1 74LS245, U10 74LS245, U11 74LS173, U12 74LS173, U13 74LS245, U14 74LS245, U15 74LS161, U16 74LS161, U17 74LS161, U18 74LS161, U19 LMC555xN, U2 74LS173, U20 LMC555xN, U21 LMC555xN, U22 7400, U23 74LS161-74xx, U24 AT28C256, U25 AT28C256, U26 74LS245, U27 74LS173, U28 74LS173, U29 74LS245, U3 74LS173, U30 74LS173, U31 74LS173, U32 74LS245, U33 74LS173, U34 74LS173, U35 74LS245, U36 74LS173, U37 74LS173, U38 74LS138, U39 74LS04, U4 74LS245, U40 74LS08, U41 74LS32, U42 74LS138, U43 74LS138, U44 74LS245, U45 74LS00, U46 74LS86, U47 74LS86, U48 74LS86, U49 74LS00, U5 74LS173, U50 74LS86, U51 74HC02, U52 74LS00, U53 74LS00, U54 74LS283, U55 74LS85, U56 74LS283, U57 74LS245, U58 74LS85, U59 74LS245, U6 74LS173, U60 74LS283, U61 74LS85, U62 74LS173, U63 74LS283, U64 74LS245, U65 74LS85, U66 74LS173, U67 74LS173, U68 74LS173, U69 74LS173, U7 74LS245, U70 74LS245, U71 74LS245, U72 74LS173, U73 74LS173, U74 74LS245, U75 74LS173, U76 74LS173, U77 74HC04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

Commit message: added display
Parts:
- added D187: LED, LED_THT:LED_D3.0mm, F.Cu at (124.1, 187.0)
- added D188: LED, LED_THT:LED_D3.0mm, F.Cu at (124.1, 193.0)
- added D63: LED, LED_THT:LED_D3.0mm, F.Cu at (337.1, 244.7)
- added R194: 220, Resistor_THT:R_Axial_DIN0204_L3.6mm_D1.6mm_P7.62mm_Horizontal, F.Cu at (68.3, 159.5)
- added R195: 220, Resistor_THT:R_Axial_DIN0204_L3.6mm_D1.6mm_P7.62mm_Horizontal, F.Cu at (57.3, 159.5)
- added R64: 220, Resistor_THT:R_Axial_DIN0204_L3.6mm_D1.6mm_P7.62mm_Horizontal, F.Cu at (314.9, 245.9)
- added RV2: 10K, ROM:Potentiometer-5.5mm, F.Cu at (-82.1, 78.6)
- added U84: RC1602A, Display:WC1602A, F.Cu at (-75.7, 85.0)
- C1, C3, C5: value 0.01uF -> 0.1uF
- C11, C13, C15: value 0.1uF -> 0.01uF
- C12: value 0.1uF -> 1uF
- C2: value 1uF -> 0.1uF
- R104, R105, R106, R108, R109, R49: value 1K -> 220
- R107: value 1M -> 220
- R171, R81, R82, R83, R85, R86: value 220 -> 1K
- R84: value 220 -> 1M
- SW1: value SW_Push-Switch -> SW_Push
- SW2: value SW_Push -> SW_SPDT; footprint Button_Switch_THT:SW_PUSH-12mm -> ROM:SW_MINI-SPDT-SW
- SW3: value SW_SPDT -> SW_Push-Switch; footprint ROM:SW_MINI-SPDT-SW -> Button_Switch_THT:SW_PUSH-12mm
- U19: value LMC555xN -> 74LS245; footprint Package_DIP:DIP-8_W7.62mm -> Package_DIP:DIP-20_W7.62mm
- U20, U21: value LMC555xN -> 74LS173; footprint Package_DIP:DIP-8_W7.62mm -> Package_DIP:DIP-16_W7.62mm
- U22: value 7400 -> 74LS245; footprint Package_DIP:DIP-14_W7.62mm -> Package_DIP:DIP-20_W7.62mm
- U23: value 74LS161-74xx -> 74LS173
- U24: value AT28C256 -> 74LS173; footprint ROM:ZIF-AT28C64B-15PU -> Package_DIP:DIP-16_W7.62mm
- U25: value AT28C256 -> 74LS245; footprint ROM:ZIF-AT28C64B-15PU -> Package_DIP:DIP-20_W7.62mm
- U26, U29, U59: value 74LS245 -> 74LS173; footprint Package_DIP:DIP-20_W7.62mm -> Package_DIP:DIP-16_W7.62mm
- U28, U37, U67: value 74LS173 -> 74LS245; footprint Package_DIP:DIP-16_W7.62mm -> Package_DIP:DIP-20_W7.62mm
- U31, U36: value 74LS173 -> LMC555xN; footprint Package_DIP:DIP-16_W7.62mm -> Package_DIP:DIP-8_W7.62mm
- U32: value 74LS245 -> 74LS04; footprint Package_DIP:DIP-20_W7.62mm -> Package_DIP:DIP-14_W7.62mm
- U33: value 74LS173 -> 74LS08; footprint Package_DIP:DIP-16_W7.62mm -> Package_DIP:DIP-14_W7.62mm
- U34: value 74LS173 -> 74LS32; footprint Package_DIP:DIP-16_W7.62mm -> Package_DIP:DIP-14_W7.62mm
- U35: value 74LS245 -> LMC555xN; footprint Package_DIP:DIP-20_W7.62mm -> Package_DIP:DIP-8_W7.62mm
- U38, U42: value 74LS138 -> 74LS00; footprint Package_DIP:DIP-16_W7.62mm -> Package_DIP:DIP-14_W7.62mm
- U39: value 74LS04 -> 74LS86
- U40: value 74LS08 -> 74LS86
- U41: value 74LS32 -> 74LS86
- U43: value 74LS138 -> 74LS86; footprint Package_DIP:DIP-16_W7.62mm -> Package_DIP:DIP-14_W7.62mm
- U44: value 74LS245 -> 74HC02; footprint Package_DIP:DIP-20_W7.62mm -> Package_DIP:DIP-14_W7.62mm
- U46: value 74LS86 -> 74LS00
- U47: value 74LS86 -> 74LS283; footprint Package_DIP:DIP-14_W7.62mm -> Package_DIP:DIP-16_W7.62mm
- U48: value 74LS86 -> 74LS85; footprint Package_DIP:DIP-14_W7.62mm -> Package_DIP:DIP-16_W7.62mm
- U49, U53: value 74LS00 -> 74LS283; footprint Package_DIP:DIP-14_W7.62mm -> Package_DIP:DIP-16_W7.62mm
- U50: value 74LS86 -> 74LS245; footprint Package_DIP:DIP-14_W7.62mm -> Package_DIP:DIP-20_W7.62mm
- U51: value 74HC02 -> 74LS85; footprint Package_DIP:DIP-14_W7.62mm -> Package_DIP:DIP-16_W7.62mm
- U52: value 74LS00 -> 74LS245; footprint Package_DIP:DIP-14_W7.62mm -> Package_DIP:DIP-20_W7.62mm
- U54: value 74LS283 -> 74LS85
- U55, U61, U65: value 74LS85 -> 74LS173
- U60: value 74LS283 -> 74LS173
- U63: value 74LS283 -> 74LS245; footprint Package_DIP:DIP-16_W7.62mm -> Package_DIP:DIP-20_W7.62mm
- U70: value 74LS245 -> 74HC04; footprint Package_DIP:DIP-20_W7.62mm -> Package_DIP:DIP-14_W7.62mm
- U71: value 74LS245 -> 74HC00; footprint Package_DIP:DIP-20_W7.62mm -> Package_DIP:DIP-14_W7.62mm
- U72, U73: value 74LS173 -> AT28C256; footprint Package_DIP:DIP-16_W7.62mm -> ROM:ZIF-AT28C64B-15PU
- U74: value 74LS245 -> AS6C62256A; footprint Package_DIP:DIP-20_W7.62mm -> Package_DIP:DIP-28_W15.24mm
- U75: value 74LS173 -> AS6C62256A; footprint Package_DIP:DIP-16_W7.62mm -> Package_DIP:DIP-28_W15.24mm
- U76: value 74LS173 -> 74HC04; footprint Package_DIP:DIP-16_W7.62mm -> Package_DIP:DIP-14_W7.62mm
- U77: value 74HC04 -> 7400
- U78: value 74HC00 -> 74LS161-74xx; footprint Package_DIP:DIP-14_W7.62mm -> Package_DIP:DIP-16_W7.62mm
- U81, U82: value AS6C62256A -> 74LS138; footprint Package_DIP:DIP-28_W15.24mm -> Package_DIP:DIP-16_W7.62mm
- U83: value 74HC04 -> 74LS138; footprint Package_DIP:DIP-14_W7.62mm -> Package_DIP:DIP-16_W7.62mm
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Connections:
- C1 pad 1: Net-(C1-Pad1) -> +5V
- C11 pad 1: +5V -> Net-(C11-Pad1)
- C12 pad 1: +5V -> Net-(C12-Pad1)
- C13 pad 1: +5V -> Net-(C13-Pad1)
- C14 pad 1: +5V -> Net-(C14-Pad1)
- C15 pad 1: +5V -> Net-(C15-Pad1)
- C2 pad 1: Net-(C2-Pad1) -> +5V
- C3 pad 1: Net-(C3-Pad1) -> +5V
- C4 pad 1: Net-(C4-Pad1) -> +5V
- C5 pad 1: Net-(C5-Pad1) -> +5V
- D100 pad 2: /Sheet61DF6CC6/sheet623AC6D9/I13 -> /ALU/sheet61054F43/I15
- D101 pad 2: /Sheet61DF6CC6/sheet623AC6D9/I14 -> /ALU/sheet67DDEE7E/I0
- D102 pad 2: /Sheet61DF6CC6/sheet623AC6D9/I15 -> /ALU/sheet67DDEE7E/I1
- D103 pad 2: Net-(D103-Pad2) -> /ALU/sheet67DDEE7E/I2
- D104 pad 2: Net-(D104-Pad2) -> /ALU/sheet67DDEE7E/I3
- D105 pad 2: Net-(D105-Pad2) -> /ALU/sheet67DDEE7E/I4
- D106 pad 2: Net-(D106-Pad2) -> /ALU/sheet67DDEE7E/I5
- D107 pad 2: /ALU/sheet61054F43/I0 -> /ALU/sheet67DDEE7E/I6
- D108 pad 2: /ALU/sheet61054F43/I1 -> /ALU/sheet67DDEE7E/I7
- D109 pad 2: /ALU/sheet61054F43/I2 -> /ALU/sheet67DDEE7E/I8
- D110 pad 2: /ALU/sheet61054F43/I3 -> /ALU/sheet67DDEE7E/I9
- D111 pad 2: /ALU/sheet61054F43/I4 -> /ALU/sheet67DDEE7E/I10
- D112 pad 2: /ALU/sheet61054F43/I5 -> /ALU/sheet67DDEE7E/I11
- D113 pad 2: /ALU/sheet61054F43/I6 -> /ALU/sheet67DDEE7E/I12
- D114 pad 2: /ALU/sheet61054F43/I7 -> /ALU/sheet67DDEE7E/I13
- D115 pad 2: /ALU/sheet61054F43/I8 -> /ALU/sheet67DDEE7E/I14
- D116 pad 2: /ALU/sheet61054F43/I9 -> /ALU/sheet67DDEE7E/I15
- D117 pad 2: /ALU/sheet61054F43/I10 -> /Control-Unit/I0
- D118 pad 2: /ALU/sheet61054F43/I11 -> /Control-Unit/I1
- D119 pad 2: /ALU/sheet61054F43/I12 -> /Control-Unit/I2
- D120 pad 2: /ALU/sheet61054F43/I13 -> /Control-Unit/I3
- D121 pad 2: /ALU/sheet61054F43/I14 -> /Control-Unit/I4
- D122 pad 2: /ALU/sheet61054F43/I15 -> /Control-Unit/I5
- D123 pad 2: /ALU/sheet67DDEE7E/I0 -> /Control-Unit/I6
- D124 pad 2: /ALU/sheet67DDEE7E/I1 -> /Control-Unit/I7
- D125 pad 2: /ALU/sheet67DDEE7E/I2 -> /Instruction-Register/sheet621E2544/I8
- D126 pad 2: /ALU/sheet67DDEE7E/I3 -> /Instruction-Register/sheet621E2544/I9
- D127 pad 2: /ALU/sheet67DDEE7E/I4 -> /Instruction-Register/sheet621E2544/I10
- D128 pad 2: /ALU/sheet67DDEE7E/I5 -> /Instruction-Register/sheet621E2544/I11
- D129 pad 2: /ALU/sheet67DDEE7E/I6 -> /Instruction-Register/sheet621E2544/I12
- D130 pad 2: /ALU/sheet67DDEE7E/I7 -> /Instruction-Register/sheet621E2544/I13
- D131 pad 2: /ALU/sheet67DDEE7E/I8 -> /Instruction-Register/sheet621E2544/I14
- D132 pad 2: /ALU/sheet67DDEE7E/I9 -> /Instruction-Register/sheet621E2544/I15
- D133 pad 2: /ALU/sheet67DDEE7E/I10 -> /ALU/BUS0
- D134 pad 2: /ALU/sheet67DDEE7E/I11 -> /ALU/BUS1
- D135 pad 2: /ALU/sheet67DDEE7E/I12 -> /ALU/BUS2
- D136 pad 2: /ALU/sheet67DDEE7E/I13 -> /ALU/BUS3
- D137 pad 2: /ALU/sheet67DDEE7E/I14 -> /ALU/BUS4
- D138 pad 2: /ALU/sheet67DDEE7E/I15 -> /ALU/BUS5
- D139 pad 2: /Control-Unit/I0 -> /ALU/BUS6
- D140 pad 2: /Control-Unit/I1 -> /ALU/BUS7
- D141 pad 2: /Control-Unit/I2 -> /ALU/BUS8
- D142 pad 2: /Control-Unit/I3 -> /ALU/BUS9
- D143 pad 2: /Control-Unit/I4 -> /ALU/BUS10
- D144 pad 2: /Control-Unit/I5 -> /ALU/BUS11
- D145 pad 2: /Control-Unit/I6 -> /ALU/BUS12
- D146 pad 2: /Control-Unit/I7 -> /ALU/BUS13
- D147 pad 2: /Instruction-Register/sheet621E2544/I8 -> /ALU/BUS14
- D148 pad 2: /Instruction-Register/sheet621E2544/I9 -> /ALU/BUS15
- D149 pad 2: /Instruction-Register/sheet621E2544/I10 -> /RAM/sheet61B5B12C/I0
- D150 pad 2: /Instruction-Register/sheet621E2544/I11 -> /RAM/sheet61B5B12C/I1
- D151 pad 2: /Instruction-Register/sheet621E2544/I12 -> /RAM/sheet61B5B12C/I2
- D152 pad 2: /Instruction-Register/sheet621E2544/I13 -> /RAM/sheet61B5B12C/I3
- D153 pad 2: /Instruction-Register/sheet621E2544/I14 -> /RAM/sheet61B5B12C/I4
- D154 pad 2: /Instruction-Register/sheet621E2544/I15 -> /RAM/sheet61B5B12C/I5
- D155 pad 2: /ALU/BUS0 -> /RAM/sheet61B5B12C/I6
- D156 pad 2: /ALU/BUS1 -> /RAM/sheet61B5B12C/I7
- D157 pad 2: /ALU/BUS2 -> /RAM/sheet61B5B12C/I8
- D158 pad 2: /ALU/BUS3 -> /RAM/sheet61B5B12C/I9
- D159 pad 2: /ALU/BUS4 -> /RAM/sheet61B5B12C/I10
- D160 pad 2: /ALU/BUS5 -> /RAM/sheet61B5B12C/I11
- D161 pad 2: /ALU/BUS6 -> /RAM/sheet61B5B12C/I12
- D162 pad 2: /ALU/BUS7 -> /RAM/sheet61B5B12C/I13
- D163 pad 2: /ALU/BUS8 -> /RAM/sheet61B5B12C/I14
- D164 pad 2: /ALU/BUS9 -> /RAM/sheet61B5B12C/I15
- D165 pad 2: /ALU/BUS10 -> /RAM/MEMWE
- D166 pad 2: /ALU/BUS11 -> /ProgramCounter/CE
- D167 pad 2: /ALU/BUS12 -> /Control-Unit/~ALU_FI
- D168 pad 2: /ALU/BUS13 -> /Control-Unit/ALU_SU
- D169 pad 2: /ALU/BUS14 -> /Control-Unit/DSP_RS
- D170 pad 2: /ALU/BUS15 -> /Control-Unit/DSP_R\W
- D171 pad 2: /RAM/sheet61B5B12C/I0 -> /Control-Unit/DSP_E
- D172 pad 2: /RAM/sheet61B5B12C/I1 -> /Resgister-A/~AO
- D173 pad 2: /RAM/sheet61B5B12C/I2 -> /Register-B/~AO
- D174 pad 2: /RAM/sheet61B5B12C/I3 -> /RAM/~AO
- D175 pad 2: /RAM/sheet61B5B12C/I4 -> /ProgramCounter/~CO
- D176 pad 2: /RAM/sheet61B5B12C/I5 -> /Instruction-Register/~I80
- D177 pad 2: /RAM/sheet61B5B12C/I6 -> /Control-Unit/~XO
- D178 pad 2: /RAM/sheet61B5B12C/I7 -> /Control-Unit/~SO
- D179 pad 2: /RAM/sheet61B5B12C/I8 -> /RAM/~MEMOE
- D180 pad 2: /RAM/sheet61B5B12C/I9 -> /Control-Unit/~ALU_EO
- D181 pad 2: /RAM/sheet61B5B12C/I10 -> /Control-Unit/~ALU_NAND_O
- D182 pad 2: /RAM/sheet61B5B12C/I11 -> /Resgister-A/~AI
- D183 pad 2: /RAM/sheet61B5B12C/I12 -> /Register-B/~AI
- D184 pad 2: /RAM/sheet61B5B12C/I13 -> /RAM/~AI
- D185 pad 2: /RAM/sheet61B5B12C/I14 -> /ProgramCounter/~J
- D186 pad 2: /RAM/sheet61B5B12C/I15 -> /Instruction-Register/~II
- D49 pad 2: /Control-Unit/~ALU_FI -> /Stack/sheet60C9B368/I0
- D50 pad 2: /Control-Unit/ALU_SU -> /Stack/sheet60C9B368/I1
- D51 pad 2: /RAM/MEMWE -> /Stack/sheet60C9B368/I2
- D52 pad 2: /ProgramCounter/CE -> /Stack/sheet60C9B368/I3
- D53 pad 2: /Resgister-A/~AO -> /Stack/sheet60C9B368/I4
- D54 pad 2: /Register-B/~AO -> /Stack/sheet60C9B368/I5
- D55 pad 2: /RAM/~AO -> /Stack/sheet60C9B368/I6
- D56 pad 2: /ProgramCounter/~CO -> /Stack/sheet60C9B368/I7
- D57 pad 2: /Instruction-Register/~I80 -> /Stack/sheet60C9B368/I8
- D58 pad 2: /Control-Unit/~XO -> /Stack/sheet60C9B368/I9
- D59 pad 2: /Control-Unit/~SO -> /Stack/sheet60C9B368/I10
- D60 pad 2: /RAM/~MEMOE -> /Stack/sheet60C9B368/I11
- D61 pad 2: /Control-Unit/~ALU_EO -> /Stack/sheet60C9B368/I12
- D62 pad 2: /Control-Unit/~ALU_NAND_O -> /Stack/sheet60C9B368/I13
- D64 pad 2: /Resgister-A/~AI -> /Stack/sheet60C9B368/I15
- D65 pad 2: /Register-B/~AI -> /Sheet61DF6CC6/sheet623AC6D9/I0
- D66 pad 2: /RAM/~AI -> /Sheet61DF6CC6/sheet623AC6D9/I1
- D67 pad 2: /ProgramCounter/~J -> /Sheet61DF6CC6/sheet623AC6D9/I2
- D68 pad 2: /Instruction-Register/~II -> /Sheet61DF6CC6/sheet623AC6D9/I3
- D69 pad 2: /Control-Unit/~XI -> /Sheet61DF6CC6/sheet623AC6D9/I4
- D70 pad 2: /Control-Unit/~SI -> /Sheet61DF6CC6/sheet623AC6D9/I5
- D71 pad 2: /Stack/sheet60C9B368/I0 -> /Sheet61DF6CC6/sheet623AC6D9/I6
- D72 pad 2: /Stack/sheet60C9B368/I1 -> /Sheet61DF6CC6/sheet623AC6D9/I7
- D73 pad 2: /Stack/sheet60C9B368/I2 -> /Sheet61DF6CC6/sheet623AC6D9/I8
- D74 pad 2: /Stack/sheet60C9B368/I3 -> /Sheet61DF6CC6/sheet623AC6D9/I9
- D75 pad 2: /Stack/sheet60C9B368/I4 -> /Sheet61DF6CC6/sheet623AC6D9/I10
- D76 pad 2: /Stack/sheet60C9B368/I5 -> /Sheet61DF6CC6/sheet623AC6D9/I11
- D77 pad 2: /Stack/sheet60C9B368/I6 -> /Sheet61DF6CC6/sheet623AC6D9/I12
- D78 pad 2: /Stack/sheet60C9B368/I7 -> /Sheet61DF6CC6/sheet623AC6D9/I13
- D79 pad 2: /Stack/sheet60C9B368/I8 -> /Sheet61DF6CC6/sheet623AC6D9/I14
- D80 pad 2: /Stack/sheet60C9B368/I9 -> /Sheet61DF6CC6/sheet623AC6D9/I15
- D81 pad 2: /Stack/sheet60C9B368/I10 -> Net-(D81-Pad2)
- D82 pad 2: /Stack/sheet60C9B368/I11 -> Net-(D82-Pad2)
- D83 pad 2: /Stack/sheet60C9B368/I12 -> Net-(D83-Pad2)
- D84 pad 2: /Stack/sheet60C9B368/I13 -> Net-(D84-Pad2)
- D85 pad 2: /Stack/sheet60C9B368/I14 -> /ALU/sheet61054F43/I0
- D86 pad 2: /Stack/sheet60C9B368/I15 -> /ALU/sheet61054F43/I1
- D87 pad 2: /Sheet61DF6CC6/sheet623AC6D9/I0 -> /ALU/sheet61054F43/I2
- D88 pad 2: /Sheet61DF6CC6/sheet623AC6D9/I1 -> /ALU/sheet61054F43/I3
- D89 pad 2: /Sheet61DF6CC6/sheet623AC6D9/I2 -> /ALU/sheet61054F43/I4
- D90 pad 2: /Sheet61DF6CC6/sheet623AC6D9/I3 -> /ALU/sheet61054F43/I5
- D91 pad 2: /Sheet61DF6CC6/sheet623AC6D9/I4 -> /ALU/sheet61054F43/I6
- D92 pad 2: /Sheet61DF6CC6/sheet623AC6D9/I5 -> /ALU/sheet61054F43/I7
- D93 pad 2: /Sheet61DF6CC6/sheet623AC6D9/I6 -> /ALU/sheet61054F43/I8
- D94 pad 2: /Sheet61DF6CC6/sheet623AC6D9/I7 -> /ALU/sheet61054F43/I9
- D95 pad 2: /Sheet61DF6CC6/sheet623AC6D9/I8 -> /ALU/sheet61054F43/I10
- D96 pad 2: /Sheet61DF6CC6/sheet623AC6D9/I9 -> /ALU/sheet61054F43/I11
- D97 pad 2: /Sheet61DF6CC6/sheet623AC6D9/I10 -> /ALU/sheet61054F43/I12
- D98 pad 2: /Sheet61DF6CC6/sheet623AC6D9/I11 -> /ALU/sheet61054F43/I13
- D99 pad 2: /Sheet61DF6CC6/sheet623AC6D9/I12 -> /ALU/sheet61054F43/I14
- R100 pad 1: Net-(D99-Pad1) -> Net-(D94-Pad1)
- R101 pad 1: Net-(D100-Pad1) -> Net-(D95-Pad1)
- R102 pad 1: Net-(D101-Pad1) -> Net-(D96-Pad1)
- R103 pad 1: Net-(D102-Pad1) -> Net-(D97-Pad1)
- R104 pad 1: +5V -> Net-(D98-Pad1)
- R104 pad 2: Net-(R104-Pad2) -> GND
- R105 pad 1: Net-(R104-Pad2) -> Net-(D99-Pad1)
- R105 pad 2: Net-(R105-Pad2) -> GND
- R106 pad 1: +5V -> Net-(D100-Pad1)
- R106 pad 2: Net-(R106-Pad2) -> GND
- R107 pad 1: +5V -> Net-(D101-Pad1)
- R107 pad 2: Net-(C4-Pad1) -> GND
- R108 pad 1: +5V -> Net-(D102-Pad1)
- R108 pad 2: Net-(R108-Pad2) -> GND
- R109 pad 1: +5V -> Net-(D103-Pad1)
- R109 pad 2: Net-(R109-Pad2) -> GND
- R110 pad 1: Net-(D103-Pad1) -> Net-(D104-Pad1)
- R111 pad 1: Net-(D104-Pad1) -> Net-(D105-Pad1)
- R112 pad 1: Net-(D105-Pad1) -> Net-(D106-Pad1)
- R113 pad 1: Net-(D106-Pad1) -> Net-(D107-Pad1)
- R114 pad 1: Net-(D107-Pad1) -> Net-(D108-Pad1)
- R115 pad 1: Net-(D108-Pad1) -> Net-(D109-Pad1)
- R116 pad 1: Net-(D109-Pad1) -> Net-(D110-Pad1)
- R117 pad 1: Net-(D110-Pad1) -> Net-(D111-Pad1)
- R118 pad 1: Net-(D111-Pad1) -> Net-(D112-Pad1)
- R119 pad 1: Net-(D112-Pad1) -> Net-(D113-Pad1)
- R120 pad 1: Net-(D113-Pad1) -> Net-(D114-Pad1)
- R121 pad 1: Net-(D114-Pad1) -> Net-(D115-Pad1)
- R122 pad 1: Net-(D115-Pad1) -> Net-(D116-Pad1)
- R123 pad 1: Net-(D116-Pad1) -> Net-(D117-Pad1)
- R124 pad 1: Net-(D117-Pad1) -> Net-(D118-Pad1)
- R125 pad 1: Net-(D118-Pad1) -> Net-(D119-Pad1)
- R126 pad 1: Net-(D119-Pad1) -> Net-(D120-Pad1)
- R127 pad 1: Net-(D120-Pad1) -> Net-(D121-Pad1)
- R128 pad 1: Net-(D121-Pad1) -> Net-(D122-Pad1)
- R129 pad 1: Net-(D122-Pad1) -> Net-(D123-Pad1)
- R130 pad 1: Net-(D123-Pad1) -> Net-(D124-Pad1)
- R131 pad 1: Net-(D124-Pad1) -> Net-(D125-Pad1)
- R132 pad 1: Net-(D125-Pad1) -> Net-(D126-Pad1)
- R133 pad 1: Net-(D126-Pad1) -> Net-(D127-Pad1)
- R134 pad 1: Net-(D127-Pad1) -> Net-(D128-Pad1)
- R135 pad 1: Net-(D128-Pad1) -> Net-(D129-Pad1)
- R136 pad 1: Net-(D129-Pad1) -> Net-(D130-Pad1)
- R137 pad 1: Net-(D130-Pad1) -> Net-(D131-Pad1)
- R138 pad 1: Net-(D131-Pad1) -> Net-(D132-Pad1)
- R139 pad 1: Net-(D132-Pad1) -> Net-(D133-Pad1)
- R140 pad 1: Net-(D133-Pad1) -> Net-(D134-Pad1)
- R141 pad 1: Net-(D134-Pad1) -> Net-(D135-Pad1)
- R142 pad 1: Net-(D135-Pad1) -> Net-(D136-Pad1)
- R143 pad 1: Net-(D136-Pad1) -> Net-(D137-Pad1)
- R144 pad 1: Net-(D137-Pad1) -> Net-(D138-Pad1)
- R145 pad 1: Net-(D138-Pad1) -> Net-(D139-Pad1)
- R146 pad 1: Net-(D139-Pad1) -> Net-(D140-Pad1)
- R147 pad 1: Net-(D140-Pad1) -> Net-(D141-Pad1)
- R148 pad 1: Net-(D141-Pad1) -> Net-(D142-Pad1)
- R149 pad 1: Net-(D142-Pad1) -> Net-(D143-Pad1)
- R150 pad 1: Net-(D143-Pad1) -> Net-(D144-Pad1)
- R151 pad 1: Net-(D144-Pad1) -> Net-(D145-Pad1)
- R152 pad 1: Net-(D145-Pad1) -> Net-(D146-Pad1)
- R153 pad 1: Net-(D146-Pad1) -> Net-(D147-Pad1)
- R154 pad 1: Net-(D147-Pad1) -> Net-(D148-Pad1)
- R155 pad 1: Net-(D148-Pad1) -> Net-(D149-Pad1)
- R156 pad 1: Net-(D149-Pad1) -> Net-(D150-Pad1)
- R157 pad 1: Net-(D150-Pad1) -> Net-(D151-Pad1)
- R158 pad 1: Net-(D151-Pad1) -> Net-(D152-Pad1)
- R159 pad 1: Net-(D152-Pad1) -> Net-(D153-Pad1)
- R160 pad 1: Net-(D153-Pad1) -> Net-(D154-Pad1)
- R161 pad 1: Net-(D154-Pad1) -> Net-(D155-Pad1)
- R162 pad 1: Net-(D155-Pad1) -> Net-(D156-Pad1)
- R163 pad 1: Net-(D156-Pad1) -> Net-(D157-Pad1)
- R164 pad 1: Net-(D157-Pad1) -> Net-(D158-Pad1)
- R165 pad 1: Net-(D158-Pad1) -> Net-(D159-Pad1)
- R166 pad 1: Net-(D159-Pad1) -> Net-(D160-Pad1)
- R167 pad 1: Net-(D160-Pad1) -> Net-(D161-Pad1)
- R168 pad 1: Net-(D161-Pad1) -> Net-(D162-Pad1)
- R169 pad 1: Net-(D162-Pad1) -> Net-(D163-Pad1)
- R170 pad 1: Net-(D163-Pad1) -> Net-(D164-Pad1)
- R171 pad 1: Net-(D164-Pad1) -> Net-(R171-Pad1)
- R49 pad 1: Net-(R49-Pad1) -> Net-(D49-Pad1)
- R50 pad 1: Net-(D49-Pad1) -> Net-(D50-Pad1)
- R51 pad 1: Net-(D50-Pad1) -> Net-(D51-Pad1)
- R52 pad 1: Net-(D51-Pad1) -> Net-(D52-Pad1)
- R53 pad 1: Net-(D52-Pad1) -> Net-(D53-Pad1)
- R54 pad 1: Net-(D53-Pad1) -> Net-(D54-Pad1)
- R55 pad 1: Net-(D54-Pad1) -> Net-(D55-Pad1)
- R56 pad 1: Net-(D55-Pad1) -> Net-(D56-Pad1)
- R57 pad 1: Net-(D56-Pad1) -> Net-(D57-Pad1)
- R58 pad 1: Net-(D57-Pad1) -> Net-(D58-Pad1)
- R59 pad 1: Net-(D58-Pad1) -> Net-(D59-Pad1)
- R60 pad 1: Net-(D59-Pad1) -> Net-(D60-Pad1)
- R61 pad 1: Net-(D60-Pad1) -> Net-(D61-Pad1)
- R62 pad 1: Net-(D61-Pad1) -> Net-(D62-Pad1)
- R63 pad 1: Net-(D62-Pad1) -> Net-(D63-Pad1)
- R65 pad 1: Net-(D64-Pad1) -> Net-(D65-Pad1)
- R66 pad 1: Net-(D65-Pad1) -> Net-(D66-Pad1)
- R67 pad 1: Net-(D66-Pad1) -> Net-(D67-Pad1)
- R68 pad 1: Net-(D67-Pad1) -> Net-(D68-Pad1)
- R69 pad 1: Net-(D68-Pad1) -> Net-(D69-Pad1)
- R70 pad 1: Net-(D69-Pad1) -> Net-(D70-Pad1)
- R71 pad 1: Net-(D70-Pad1) -> Net-(D71-Pad1)
- R72 pad 1: Net-(D71-Pad1) -> Net-(D72-Pad1)
- R73 pad 1: Net-(D72-Pad1) -> Net-(D73-Pad1)
- R74 pad 1: Net-(D73-Pad1) -> Net-(D74-Pad1)
- R75 pad 1: Net-(D74-Pad1) -> Net-(D75-Pad1)
- R76 pad 1: Net-(D75-Pad1) -> Net-(D76-Pad1)
- R77 pad 1: Net-(D76-Pad1) -> Net-(D77-Pad1)
- R78 pad 1: Net-(D77-Pad1) -> Net-(D78-Pad1)
- R79 pad 1: Net-(D78-Pad1) -> Net-(D79-Pad1)
- R80 pad 1: Net-(D79-Pad1) -> Net-(D80-Pad1)
- R81 pad 1: Net-(D80-Pad1) -> +5V
- R81 pad 2: GND -> Net-(R81-Pad2)
- R82 pad 1: Net-(D81-Pad1) -> Net-(R81-Pad2)
- R82 pad 2: GND -> Net-(R82-Pad2)
- R83 pad 1: Net-(D82-Pad1) -> +5V
- R83 pad 2: GND -> Net-(R83-Pad2)
- R84 pad 1: Net-(D83-Pad1) -> +5V
- R84 pad 2: GND -> Net-(C14-Pad1)
- R85 pad 1: Net-(D84-Pad1) -> +5V
- R85 pad 2: GND -> Net-(R85-Pad2)
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
Commit message: images and pcb
Parts:
- removed U84: RC1602A, Display:WC1602A
- added D189: LED, LED_THT:LED_D3.0mm, F.Cu at (132.1, 128.9)
- added DS1: WC1602A, Display:WC1602A, F.Cu at (51.7, 47.3)
- added R196: 220, Resistor_THT:R_Axial_DIN0204_L3.6mm_D1.6mm_P7.62mm_Horizontal, F.Cu at (65.4, 99.0)
- moved D117 664.9 mm to (-40.7, 443.8)
- moved D118 664.9 mm to (-47.0, 443.8)
- moved D119 664.9 mm to (-25.1, 444.9)
- moved D120 664.9 mm to (-18.8, 444.9)
- moved D121 664.9 mm to (-18.8, 478.1)
- moved D122 664.9 mm to (-18.8, 472.2)
- moved D123 664.9 mm to (-18.8, 460.3)
- moved D124 664.9 mm to (-18.8, 466.2)
- moved D125 664.9 mm to (-18.8, 450.9)
- moved D126 664.9 mm to (-47.0, 449.7)
- moved D127 664.9 mm to (-36.0, 449.7)
- moved D128 664.9 mm to (-25.1, 450.9)
- moved D129 664.9 mm to (-25.1, 466.2)
- moved D130 664.9 mm to (-25.1, 472.2)
- moved D131 664.9 mm to (-25.1, 478.1)
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
Commit message: clean up
Parts:
- added U84: 74LS138, Package_DIP:DIP-16_W7.62mm, F.Cu at (90.6, 380.1)
- added U85: 74LS138, Package_DIP:DIP-16_W7.62mm, F.Cu at (79.4, 380.1)
- U29, U59, U65, U66, U69: value 74LS173 -> 74LS245; footprint Package_DIP:DIP-16_W7.62mm -> Package_DIP:DIP-20_W7.62mm
- U31: value LMC555xN -> 74LS173; footprint Package_DIP:DIP-8_W7.62mm -> Package_DIP:DIP-16_W7.62mm
- U32: value 74LS04 -> 74LS245; footprint Package_DIP:DIP-14_W7.62mm -> Package_DIP:DIP-20_W7.62mm
- U33: value 74LS08 -> LMC555xN; footprint Package_DIP:DIP-14_W7.62mm -> Package_DIP:DIP-8_W7.62mm
- U34: value 74LS32 -> 74LS04
- U35: value LMC555xN -> 74LS08; footprint Package_DIP:DIP-8_W7.62mm -> Package_DIP:DIP-14_W7.62mm
- U36: value LMC555xN -> 74LS32; footprint Package_DIP:DIP-8_W7.62mm -> Package_DIP:DIP-14_W7.62mm
- U37: value 74LS245 -> LMC555xN; footprint Package_DIP:DIP-20_W7.62mm -> Package_DIP:DIP-8_W7.62mm
- U38: value 74LS00 -> LMC555xN; footprint Package_DIP:DIP-14_W7.62mm -> Package_DIP:DIP-8_W7.62mm
- U39: value 74LS86 -> 74LS245; footprint Package_DIP:DIP-14_W7.62mm -> Package_DIP:DIP-20_W7.62mm
- U40: value 74LS86 -> 74LS00
- U42, U45: value 74LS00 -> 74LS86
- U44: value 74HC02 -> 74LS00
- U46: value 74LS00 -> 74HC02
- U47: value 74LS283 -> 74LS00; footprint Package_DIP:DIP-16_W7.62mm -> Package_DIP:DIP-14_W7.62mm
- U48: value 74LS85 -> 74LS00; footprint Package_DIP:DIP-16_W7.62mm -> Package_DIP:DIP-14_W7.62mm
- U50: value 74LS245 -> 74LS85; footprint Package_DIP:DIP-20_W7.62mm -> Package_DIP:DIP-16_W7.62mm
- U51, U58: value 74LS85 -> 74LS283
- U53, U56: value 74LS283 -> 74LS85
- U54: value 74LS85 -> 74LS245; footprint Package_DIP:DIP-16_W7.62mm -> Package_DIP:DIP-20_W7.62mm
- U55: value 74LS173 -> 74LS283
- U57, U63, U64, U67: value 74LS245 -> 74LS173; footprint Package_DIP:DIP-20_W7.62mm -> Package_DIP:DIP-16_W7.62mm
- U60: value 74LS173 -> 74LS85
- U70: value 74HC04 -> 74LS173; footprint Package_DIP:DIP-14_W7.62mm -> Package_DIP:DIP-16_W7.62mm
- U71: value 74HC00 -> 74LS173; footprint Package_DIP:DIP-14_W7.62mm -> Package_DIP:DIP-16_W7.62mm
- U72: value AT28C256 -> 74HC04; footprint ROM:ZIF-AT28C64B-15PU -> Package_DIP:DIP-14_W7.62mm
- U73: value AT28C256 -> 74HC00; footprint ROM:ZIF-AT28C64B-15PU -> Package_DIP:DIP-14_W7.62mm
- U74, U75: value AS6C62256A -> AT28C256; footprint Package_DIP:DIP-28_W15.24mm -> ROM:ZIF-AT28C64B-15PU
- U76: value 74HC04 -> AS6C62256A; footprint Package_DIP:DIP-14_W7.62mm -> Package_DIP:DIP-28_W15.24mm
- U77: value 7400 -> AS6C62256A; footprint Package_DIP:DIP-14_W7.62mm -> Package_DIP:DIP-28_W15.24mm
- U78: value 74LS161-74xx -> 74HC04; footprint Package_DIP:DIP-16_W7.62mm -> Package_DIP:DIP-14_W7.62mm
- U79: value AT28C256 -> 7400; footprint ROM:ZIF-AT28C64B-15PU -> Package_DIP:DIP-14_W7.62mm
- U80: value AT28C256 -> 74LS161-74xx; footprint ROM:ZIF-AT28C64B-15PU -> Package_DIP:DIP-16_W7.62mm
- U81, U82: value 74LS138 -> AT28C256; footprint Package_DIP:DIP-16_W7.62mm -> ROM:ZIF-AT28C64B-15PU
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Connections:
- D165 pad 2: /RAM/MEMWE -> /Control-Unit/RESET_COUNTER
- D166 pad 2: /ProgramCounter/CE -> /RAM/MEMWE
- D167 pad 2: /Control-Unit/~ALU_FI -> /ProgramCounter/CE
- D168 pad 2: /Control-Unit/ALU_SU -> /Control-Unit/~ALU_FI
- D169 pad 2: /Control-Unit/DSP_RS -> /Control-Unit/ALU_SU
- D170 pad 2: /Control-Unit/DSP_R\W -> /Control-Unit/DSP_RS
- D171 pad 2: /Control-Unit/DSP_E -> /Control-Unit/DSP_R\W
- D172 pad 2: /Resgister-A/~AO -> /Control-Unit/DSP_E
- D173 pad 2: /Register-B/~AO -> /Register-A/~AO
- D174 pad 2: /RAM/~AO -> /Register-B/~AO
- D175 pad 2: /ProgramCounter/~CO -> /RAM/~AO
- D176 pad 2: /Instruction-Register/~I80 -> /ProgramCounter/~CO
- D177 pad 2: /Control-Unit/~XO -> /Instruction-Register/~I80
- D178 pad 2: /Control-Unit/~SO -> /Control-Unit/~XO
- D179 pad 2: /RAM/~MEMOE -> /Control-Unit/~SO
- D180 pad 2: /Control-Unit/~ALU_EO -> /RAM/~MEMOE
- D181 pad 2: /Control-Unit/~ALU_NAND_O -> /Control-Unit/~ALU_EO
- D182 pad 2: /Resgister-A/~AI -> /Control-Unit/~ALU_NAND_O
- D183 pad 2: /Register-B/~AI -> /Register-A/~AI
- D184 pad 2: /RAM/~AI -> /Register-B/~AI
- D185 pad 2: /ProgramCounter/~J -> /RAM/~AI
- D186 pad 2: /Instruction-Register/~II -> /ProgramCounter/~J
- D187 pad 2: /Control-Unit/~XI -> /Instruction-Register/~II
- D188 pad 2: /Control-Unit/~SI -> /Control-Unit/~XI
- D189 pad 2: /Control-Unit/RESET_COUNTER -> /Control-Unit/~SI
- D81 pad 2: Net-(D81-Pad2) -> /ALU/AGTBF
- D82 pad 2: Net-(D82-Pad2) -> /ALU/ALTBF
- D83 pad 2: Net-(D83-Pad2) -> /ALU/ZF
- D84 pad 2: Net-(D84-Pad2) -> /ALU/CF
- U1 pad 19: /Resgister-A/~AO -> /Register-A/~AO
- U2 pad 10: /Resgister-A/~AI -> /Register-A/~AI
- U2 pad 9: /Resgister-A/~AI -> /Register-A/~AI
- U29 pad 1: GND -> +5V
- U29 pad 10: /Control-Unit/~XI -> GND
- U29 pad 11: /ALU/BUS11 -> /ALU/BUS7
- U29 pad 12: /ALU/BUS10 -> /ALU/BUS6
- U29 pad 13: /ALU/BUS9 -> /ALU/BUS5
- U29 pad 14: /ALU/BUS8 -> /ALU/BUS4
- U29 pad 15: /ALU/CLR -> /ALU/BUS3
- U29 pad 16: +5V -> /ALU/BUS2
- U29 pad 2: GND -> /Sheet61DF6CC6/sheet623AC6D9/I8
- U29 pad 3: /Sheet61DF6CC6/sheet623AC6D9/I8 -> /Sheet61DF6CC6/sheet623AC6D9/I9
- U29 pad 4: /Sheet61DF6CC6/sheet623AC6D9/I9 -> /Sheet61DF6CC6/sheet623AC6D9/I10
- U29 pad 5: /Sheet61DF6CC6/sheet623AC6D9/I10 -> /Sheet61DF6CC6/sheet623AC6D9/I11
- U29 pad 6: /Sheet61DF6CC6/sheet623AC6D9/I11 -> /Sheet61DF6CC6/sheet623AC6D9/I12
- U29 pad 7: /ALU/CLK -> /Sheet61DF6CC6/sheet623AC6D9/I13
- U29 pad 8: GND -> /Sheet61DF6CC6/sheet623AC6D9/I14
- U29 pad 9: /Control-Unit/~XI -> /Sheet61DF6CC6/sheet623AC6D9/I15
- U3 pad 10: /Resgister-A/~AI -> /Register-A/~AI
- U3 pad 9: /Resgister-A/~AI -> /Register-A/~AI
- U30 pad 11: /ALU/BUS15 -> /ALU/BUS11
- U30 pad 12: /ALU/BUS14 -> /ALU/BUS10
- U30 pad 13: /ALU/BUS13 -> /ALU/BUS9
- U30 pad 14: /ALU/BUS12 -> /ALU/BUS8
- U30 pad 3: /Sheet61DF6CC6/sheet623AC6D9/I12 -> /Sheet61DF6CC6/sheet623AC6D9/I8
- U30 pad 4: /Sheet61DF6CC6/sheet623AC6D9/I13 -> /Sheet61DF6CC6/sheet623AC6D9/I9
- U30 pad 5: /Sheet61DF6CC6/sheet623AC6D9/I14 -> /Sheet61DF6CC6/sheet623AC6D9/I10
- U30 pad 6: /Sheet61DF6CC6/sheet623AC6D9/I15 -> /Sheet61DF6CC6/sheet623AC6D9/I11
- U31 pad 2: Net-(C12-Pad1) -> GND
- U31 pad 3: Net-(U31-Pad3) -> /Sheet61DF6CC6/sheet623AC6D9/I12
- U31 pad 4: +5V -> /Sheet61DF6CC6/sheet623AC6D9/I13
- U31 pad 5: Net-(C11-Pad1) -> /Sheet61DF6CC6/sheet623AC6D9/I14
- U31 pad 6: Net-(C12-Pad1) -> /Sheet61DF6CC6/sheet623AC6D9/I15
- U31 pad 7: Net-(R81-Pad2) -> /ALU/CLK
- U31 pad 8: +5V -> GND
- U32 pad 1: Net-(U32-Pad1) -> +5V
- U32 pad 10: (no net) -> GND
- U32 pad 11: (no net) -> /ALU/BUS15
- U32 pad 12: (no net) -> /ALU/BUS14
- U32 pad 13: (no net) -> /ALU/BUS13
- U32 pad 14: +5V -> /ALU/BUS12
- U32 pad 2: Net-(U32-Pad2) -> /Sheet61DF6CC6/sheet623AC6D9/I0
- U32 pad 3: /clock/HLT -> /Sheet61DF6CC6/sheet623AC6D9/I1
- U32 pad 4: Net-(U32-Pad4) -> /Sheet61DF6CC6/sheet623AC6D9/I2
- U32 pad 5: /ALU/CLK -> /Sheet61DF6CC6/sheet623AC6D9/I3
- U32 pad 6: /clock/~CLK -> /Sheet61DF6CC6/sheet623AC6D9/I4
- U32 pad 7: GND -> /Sheet61DF6CC6/sheet623AC6D9/I5
- U32 pad 8: (no net) -> /Sheet61DF6CC6/sheet623AC6D9/I6
- U32 pad 9: (no net) -> /Sheet61DF6CC6/sheet623AC6D9/I7
- U33 pad 1: Net-(U31-Pad3) -> GND
- U33 pad 2: Net-(U32-Pad1) -> Net-(C12-Pad1)
- U33 pad 4: Net-(U32-Pad2) -> +5V
- U33 pad 5: Net-(U33-Pad5) -> Net-(C11-Pad1)
- U33 pad 6: Net-(U33-Pad6) -> Net-(C12-Pad1)
- U33 pad 7: GND -> Net-(R81-Pad2)
- U33 pad 8: /ALU/CLK -> +5V
- U34 pad 1: Net-(U33-Pad3) -> Net-(U34-Pad1)
- U34 pad 2: Net-(U33-Pad6) -> Net-(U34-Pad2)
- U34 pad 3: Net-(U33-Pad9) -> (no net)
- U34 pad 5: (no net) -> /ALU/CLK
- U34 pad 6: (no net) -> /clock/~CLK
- U35 pad 1: GND -> Net-(U33-Pad3)
- U35 pad 2: Net-(R83-Pad2) -> Net-(U34-Pad1)
- U35 pad 3: Net-(U33-Pad5) -> Net-(U35-Pad3)
- U35 pad 4: +5V -> Net-(U34-Pad2)
- U35 pad 5: Net-(C13-Pad1) -> Net-(U35-Pad5)
- U35 pad 6: Net-(C14-Pad1) -> Net-(U35-Pad6)
- U35 pad 7: Net-(C14-Pad1) -> GND
- U35 pad 8: +5V -> /ALU/CLK
- U36 pad 1: GND -> Net-(U35-Pad3)
- U36 pad 2: Net-(R85-Pad2) -> Net-(U35-Pad6)
- U36 pad 3: Net-(U32-Pad1) -> Net-(U35-Pad9)
- U36 pad 4: Net-(R86-Pad2) -> (no net)
- U36 pad 5: Net-(C15-Pad1) -> (no net)
- U36 pad 6: GND -> (no net)
- U36 pad 7: Net-(U36-Pad7) -> GND
- U36 pad 8: +5V -> (no net)
- U37 pad 1: +5V -> GND
- U37 pad 2: /ALU/sheet67DDEE7E/I8 -> Net-(R83-Pad2)
- U37 pad 3: /ALU/sheet67DDEE7E/I9 -> Net-(U35-Pad5)
- U37 pad 4: /ALU/sheet67DDEE7E/I10 -> +5V
- U37 pad 5: /ALU/sheet67DDEE7E/I11 -> Net-(C13-Pad1)
- U37 pad 6: /ALU/sheet67DDEE7E/I12 -> Net-(C14-Pad1)
- U37 pad 7: /ALU/sheet67DDEE7E/I13 -> Net-(C14-Pad1)
- U37 pad 8: /ALU/sheet67DDEE7E/I14 -> +5V
- U38 pad 1: /ALU/A8 -> GND
- U38 pad 2: Net-(U38-Pad2) -> Net-(R85-Pad2)
- U38 pad 3: /ALU/sheet67DDEE7E/I8 -> Net-(U34-Pad1)
- U38 pad 4: /ALU/A9 -> Net-(R86-Pad2)
- U38 pad 5: Net-(U38-Pad5) -> Net-(C15-Pad1)
- U38 pad 6: /ALU/sheet67DDEE7E/I9 -> GND
- U38 pad 7: +5V -> Net-(U38-Pad7)
- U38 pad 8: /ALU/sheet67DDEE7E/I10 -> +5V
- U39 pad 1: /Register-B/A12 -> +5V
- U39 pad 10: /Control-Unit/ALU_SU -> GND
- U39 pad 11: Net-(U39-Pad11) -> /ALU/BUS15
- U39 pad 12: /Register-B/A15 -> /ALU/BUS14
- U39 pad 13: /Control-Unit/ALU_SU -> /ALU/BUS13
- U39 pad 14: +5V -> /ALU/BUS12
- U39 pad 2: /Control-Unit/ALU_SU -> /ALU/sheet67DDEE7E/I8
- U39 pad 3: Net-(U39-Pad3) -> /ALU/sheet67DDEE7E/I9
- U39 pad 4: /Register-B/A13 -> /ALU/sheet67DDEE7E/I10
- U39 pad 5: /Control-Unit/ALU_SU -> /ALU/sheet67DDEE7E/I11
- U39 pad 6: Net-(U39-Pad6) -> /ALU/sheet67DDEE7E/I12
- U39 pad 7: GND -> /ALU/sheet67DDEE7E/I13
- U39 pad 8: Net-(U39-Pad8) -> /ALU/sheet67DDEE7E/I14
- U39 pad 9: /Register-B/A14 -> /ALU/sheet67DDEE7E/I15
- U4 pad 19: /Resgister-A/~AO -> /Register-A/~AO
- U40 pad 1: /Register-B/A8 -> /ALU/A8
- U40 pad 10: /Control-Unit/ALU_SU -> Net-(U40-Pad10)
- U40 pad 11: Net-(U38-Pad13) -> /ALU/sheet67DDEE7E/I11
- U40 pad 12: /Register-B/A11 -> /ALU/A11
- U40 pad 13: /Control-Unit/ALU_SU -> Net-(U40-Pad13)
- U40 pad 14: +5V -> GND
- U40 pad 2: /Control-Unit/ALU_SU -> Net-(U40-Pad2)
- U40 pad 3: Net-(U38-Pad2) -> /ALU/sheet67DDEE7E/I8
- U40 pad 4: /Register-B/A9 -> /ALU/A9
- U40 pad 5: /Control-Unit/ALU_SU -> Net-(U40-Pad5)
- U40 pad 6: Net-(U38-Pad5) -> /ALU/sheet67DDEE7E/I9
- U40 pad 7: GND -> +5V
- U40 pad 8: Net-(U38-Pad10) -> /ALU/sheet67DDEE7E/I10
- U40 pad 9: /Register-B/A10 -> /ALU/A10
- U41 pad 1: /Register-B/A4 -> /Register-B/A12
- U41 pad 12: /Register-B/A7 -> /Register-B/A15
- U41 pad 4: /Register-B/A5 -> /Register-B/A13
- U41 pad 6: /ALU/A3 -> Net-(U41-Pad6)
- U41 pad 9: /Register-B/A6 -> /Register-B/A14
- U42 pad 1: /ALU/A12 -> /Register-B/A8
- U42 pad 10: Net-(U39-Pad8) -> /Control-Unit/ALU_SU
- U42 pad 11: /ALU/sheet67DDEE7E/I15 -> Net-(U40-Pad13)
- U42 pad 12: /ALU/A15 -> /Register-B/A11
- U42 pad 13: Net-(U39-Pad11) -> /Control-Unit/ALU_SU
- U42 pad 14: GND -> +5V
- U42 pad 2: Net-(U39-Pad3) -> /Control-Unit/ALU_SU
- U42 pad 3: /ALU/sheet67DDEE7E/I12 -> Net-(U40-Pad2)
- U42 pad 4: /ALU/A13 -> /Register-B/A9
- U42 pad 5: Net-(U39-Pad6) -> /Control-Unit/ALU_SU
- U42 pad 6: /ALU/sheet67DDEE7E/I13 -> Net-(U40-Pad5)
- U42 pad 7: +5V -> GND
- U42 pad 8: /ALU/sheet67DDEE7E/I14 -> Net-(U40-Pad10)
- U42 pad 9: /ALU/A14 -> /Register-B/A10
- U43 pad 1: /Register-B/A0 -> /Register-B/A4
- U43 pad 12: /Register-B/A3 -> /Register-B/A7
- U43 pad 3: /ALU/A1 -> Net-(U43-Pad3)
- U43 pad 4: /Register-B/A1 -> /Register-B/A5
- U43 pad 6: Net-(U43-Pad6) -> /ALU/A3
- U43 pad 9: /Register-B/A2 -> /Register-B/A6
- U44 pad 1: (no net) -> /ALU/A12
- U44 pad 10: (no net) -> Net-(U41-Pad8)
- U44 pad 11: (no net) -> /ALU/sheet67DDEE7E/I15
- U44 pad 12: (no net) -> /ALU/A15
- U44 pad 13: (no net) -> Net-(U41-Pad11)
- U44 pad 14: +5V -> GND
- U44 pad 2: (no net) -> Net-(U41-Pad3)
- U44 pad 3: (no net) -> /ALU/sheet67DDEE7E/I12
- U44 pad 4: (no net) -> /ALU/A13
- U44 pad 5: (no net) -> Net-(U41-Pad6)
- U44 pad 6: (no net) -> /ALU/sheet67DDEE7E/I13
- U44 pad 7: GND -> +5V
- U44 pad 8: (no net) -> /ALU/sheet67DDEE7E/I14
- U44 pad 9: (no net) -> /ALU/A14
- U45 pad 1: /ALU/A0 -> /Register-B/A0
- U45 pad 10: Net-(U43-Pad8) -> /Control-Unit/ALU_SU
- U45 pad 11: /ALU/sheet67DDEE7E/I3 -> Net-(U45-Pad11)
- U45 pad 12: /ALU/A3 -> /Register-B/A3
- U45 pad 13: Net-(U43-Pad11) -> /Control-Unit/ALU_SU
- U45 pad 14: GND -> +5V
- U45 pad 2: /ALU/A1 -> /Control-Unit/ALU_SU
- U45 pad 3: /ALU/sheet67DDEE7E/I0 -> /ALU/A1
- U45 pad 4: /ALU/A1 -> /Register-B/A1
- U45 pad 5: Net-(U43-Pad6) -> /Control-Unit/ALU_SU
- U45 pad 6: /ALU/sheet67DDEE7E/I1 -> Net-(U45-Pad6)
- U45 pad 7: +5V -> GND
- U45 pad 8: /ALU/sheet67DDEE7E/I2 -> Net-(U45-Pad8)
- U45 pad 9: /ALU/A2 -> /Register-B/A2
- U46 pad 1: /ALU/A4 -> (no net)
- U46 pad 10: Net-(U41-Pad8) -> (no net)
- U46 pad 11: /ALU/sheet67DDEE7E/I7 -> (no net)
- U46 pad 12: /ALU/A7 -> (no net)
- U46 pad 13: Net-(U41-Pad11) -> (no net)
- U46 pad 14: GND -> +5V
- U46 pad 2: Net-(U41-Pad3) -> (no net)
- U46 pad 3: /ALU/sheet67DDEE7E/I4 -> (no net)
- U46 pad 4: /ALU/A5 -> (no net)
- U46 pad 5: /ALU/A3 -> (no net)
- U46 pad 6: /ALU/sheet67DDEE7E/I5 -> (no net)
- U46 pad 7: +5V -> GND
- U46 pad 8: /ALU/sheet67DDEE7E/I6 -> (no net)
- U46 pad 9: /ALU/A6 -> (no net)
- U47 pad 1: /ALU/sheet61054F43/I1 -> /ALU/A0
- U47 pad 10: /ALU/sheet61054F43/I3 -> Net-(U45-Pad8)
- U47 pad 11: Net-(U43-Pad11) -> /ALU/sheet67DDEE7E/I3
- U47 pad 13: /ALU/sheet61054F43/I2 -> Net-(U45-Pad11)
- U47 pad 14: /ALU/A2 -> GND
- U47 pad 2: Net-(U43-Pad6) -> /ALU/A1
- U47 pad 3: /ALU/A1 -> /ALU/sheet67DDEE7E/I0
- U47 pad 4: /ALU/sheet61054F43/I0 -> /ALU/A1
- U47 pad 5: /ALU/A0 -> Net-(U45-Pad6)
- U47 pad 6: /ALU/A1 -> /ALU/sheet67DDEE7E/I1
- U47 pad 7: /Control-Unit/ALU_SU -> +5V
- U47 pad 8: GND -> /ALU/sheet67DDEE7E/I2
- U47 pad 9: Net-(U47-Pad9) -> /ALU/A2
- U48 pad 1: Net-(U43-Pad11) -> /ALU/A4
- U48 pad 10: /ALU/A3 -> Net-(U43-Pad8)
- U48 pad 11: Net-(U43-Pad6) -> /ALU/sheet67DDEE7E/I7
- U48 pad 12: /ALU/A2 -> /ALU/A7
- U48 pad 13: /ALU/A1 -> Net-(U43-Pad11)
- U48 pad 14: Net-(U43-Pad8) -> GND
- U48 pad 2: Net-(U48-Pad2) -> Net-(U43-Pad3)
- U48 pad 3: Net-(U48-Pad3) -> /ALU/sheet67DDEE7E/I4
- U48 pad 4: Net-(U48-Pad4) -> /ALU/A5
- U48 pad 5: Net-(U48-Pad5) -> /ALU/A3
- U48 pad 6: Net-(U48-Pad6) -> /ALU/sheet67DDEE7E/I5
- U48 pad 7: Net-(U48-Pad7) -> +5V
- U48 pad 8: GND -> /ALU/sheet67DDEE7E/I6
- U48 pad 9: /ALU/A1 -> /ALU/A6
- U49 pad 1: /ALU/sheet61054F43/I5 -> /ALU/sheet61054F43/I1
- U49 pad 10: /ALU/sheet61054F43/I7 -> /ALU/sheet61054F43/I3
- U49 pad 11: Net-(U41-Pad11) -> Net-(U45-Pad11)
- U49 pad 12: /ALU/A7 -> /ALU/A3
- U49 pad 13: /ALU/sheet61054F43/I6 -> /ALU/sheet61054F43/I2
- U49 pad 14: /ALU/A6 -> /ALU/A2
- U49 pad 15: Net-(U41-Pad8) -> Net-(U45-Pad8)
- U49 pad 2: /ALU/A3 -> Net-(U45-Pad6)
- U49 pad 3: /ALU/A5 -> /ALU/A1
- U49 pad 4: /ALU/sheet61054F43/I4 -> /ALU/sheet61054F43/I0
- U49 pad 5: /ALU/A4 -> /ALU/A0
- U49 pad 6: Net-(U41-Pad3) -> /ALU/A1
- U49 pad 7: Net-(U47-Pad9) -> /Control-Unit/ALU_SU
- U5 pad 10: /Resgister-A/~AI -> /Register-A/~AI
- U5 pad 9: /Resgister-A/~AI -> /Register-A/~AI
- U50 pad 1: +5V -> Net-(U45-Pad11)
- U50 pad 10: GND -> /ALU/A3
- U50 pad 11: /ALU/BUS7 -> Net-(U45-Pad6)
- U50 pad 12: /ALU/BUS6 -> /ALU/A2
- U50 pad 13: /ALU/BUS5 -> /ALU/A1
- U50 pad 14: /ALU/BUS4 -> Net-(U45-Pad8)
- U50 pad 15: /ALU/BUS3 -> /ALU/A0
- U50 pad 16: /ALU/BUS2 -> +5V
- U50 pad 2: /ALU/sheet61054F43/I0 -> Net-(U50-Pad2)
- U50 pad 3: /ALU/sheet61054F43/I1 -> Net-(U50-Pad3)
- U50 pad 4: /ALU/sheet61054F43/I2 -> Net-(U50-Pad4)
- U50 pad 5: /ALU/sheet61054F43/I3 -> Net-(U50-Pad5)
- U50 pad 6: /ALU/sheet61054F43/I4 -> Net-(U50-Pad6)
- U50 pad 7: /ALU/sheet61054F43/I5 -> Net-(U50-Pad7)
- U50 pad 8: /ALU/sheet61054F43/I6 -> GND
- U50 pad 9: /ALU/sheet61054F43/I7 -> /ALU/A1
- U51 pad 1: Net-(U41-Pad11) -> /ALU/sheet61054F43/I5
- U51 pad 10: /ALU/A4 -> /ALU/sheet61054F43/I7
- U51 pad 11: /ALU/A3 -> Net-(U43-Pad11)
- U51 pad 12: /ALU/A5 -> /ALU/A7
- U51 pad 13: /ALU/A6 -> /ALU/sheet61054F43/I6
- U51 pad 14: Net-(U41-Pad8) -> /ALU/A6
- U51 pad 15: /ALU/A7 -> Net-(U43-Pad8)
- U51 pad 2: Net-(U48-Pad7) -> /ALU/A3
- U51 pad 3: Net-(U48-Pad5) -> /ALU/A5
- U51 pad 4: Net-(U48-Pad6) -> /ALU/sheet61054F43/I4
- U51 pad 5: Net-(U51-Pad5) -> /ALU/A4
- U51 pad 6: Net-(U51-Pad6) -> Net-(U43-Pad3)
- U51 pad 7: Net-(U51-Pad7) -> Net-(U49-Pad9)
- U51 pad 9: Net-(U41-Pad3) -> Net-(U51-Pad9)
- U52 pad 11: /ALU/BUS15 -> /ALU/BUS7
- U52 pad 12: /ALU/BUS14 -> /ALU/BUS6
- U52 pad 13: /ALU/BUS13 -> /ALU/BUS5
- U52 pad 14: /ALU/BUS12 -> /ALU/BUS4
- U52 pad 15: /ALU/BUS11 -> /ALU/BUS3
- U52 pad 16: /ALU/BUS10 -> /ALU/BUS2
- U52 pad 17: /ALU/BUS9 -> /ALU/BUS1
- U52 pad 18: /ALU/BUS8 -> /ALU/BUS0
- U52 pad 2: /ALU/sheet61054F43/I8 -> /ALU/sheet61054F43/I0
- U52 pad 3: /ALU/sheet61054F43/I9 -> /ALU/sheet61054F43/I1
- U52 pad 4: /ALU/sheet61054F43/I10 -> /ALU/sheet61054F43/I2
- U52 pad 5: /ALU/sheet61054F43/I11 -> /ALU/sheet61054F43/I3
- U52 pad 6: /ALU/sheet61054F43/I12 -> /ALU/sheet61054F43/I4
- U52 pad 7: /ALU/sheet61054F43/I13 -> /ALU/sheet61054F43/I5
- U52 pad 8: /ALU/sheet61054F43/I14 -> /ALU/sheet61054F43/I6
- U52 pad 9: /ALU/sheet61054F43/I15 -> /ALU/sheet61054F43/I7
- U53 pad 1: /ALU/sheet61054F43/I9 -> Net-(U43-Pad11)
- U53 pad 10: /ALU/sheet61054F43/I11 -> /ALU/A4
- U53 pad 11: Net-(U38-Pad13) -> /ALU/A3
- U53 pad 12: /ALU/A11 -> /ALU/A5
- U53 pad 13: /ALU/sheet61054F43/I10 -> /ALU/A6
- U53 pad 14: /ALU/A10 -> Net-(U43-Pad8)
- U53 pad 15: Net-(U38-Pad10) -> /ALU/A7
- U53 pad 2: Net-(U38-Pad5) -> Net-(U50-Pad7)
- U53 pad 3: /ALU/A9 -> Net-(U50-Pad5)
- U53 pad 4: /ALU/sheet61054F43/I8 -> Net-(U50-Pad6)
- U53 pad 5: /ALU/A8 -> Net-(U53-Pad5)
- U53 pad 6: Net-(U38-Pad2) -> Net-(U53-Pad6)
- U53 pad 7: Net-(U49-Pad9) -> Net-(U53-Pad7)
- U53 pad 9: Net-(U53-Pad9) -> Net-(U43-Pad3)
- U54 pad 1: Net-(U38-Pad13) -> +5V
- U54 pad 10: /ALU/A8 -> GND
- U54 pad 11: Net-(U38-Pad5) -> /ALU/BUS15
- U54 pad 12: /ALU/A9 -> /ALU/BUS14
- U54 pad 13: /ALU/A10 -> /ALU/BUS13
- U54 pad 14: Net-(U38-Pad10) -> /ALU/BUS12
- U54 pad 15: /ALU/A11 -> /ALU/BUS11
- U54 pad 16: +5V -> /ALU/BUS10
- U54 pad 2: Net-(U51-Pad7) -> /ALU/sheet61054F43/I8
- U54 pad 3: Net-(U51-Pad6) -> /ALU/sheet61054F43/I9
- U54 pad 4: Net-(U51-Pad5) -> /ALU/sheet61054F43/I10
- U54 pad 5: Net-(U54-Pad5) -> /ALU/sheet61054F43/I11
- U54 pad 6: Net-(U54-Pad6) -> /ALU/sheet61054F43/I12
- U54 pad 7: Net-(U54-Pad7) -> /ALU/sheet61054F43/I13
- U54 pad 8: GND -> /ALU/sheet61054F43/I14
- U54 pad 9: Net-(U38-Pad2) -> /ALU/sheet61054F43/I15
- U55 pad 1: GND -> /ALU/sheet61054F43/I9
- U55 pad 10: /Control-Unit/~ALU_FI -> /ALU/sheet61054F43/I11
- U55 pad 11: Net-(D81-Pad2) -> Net-(U40-Pad13)
- U55 pad 12: Net-(D82-Pad2) -> /ALU/A11
- U55 pad 13: Net-(D83-Pad2) -> /ALU/sheet61054F43/I10
- U55 pad 14: Net-(D84-Pad2) -> /ALU/A10
- U55 pad 15: /ALU/CLR -> Net-(U40-Pad10)
- U55 pad 2: GND -> Net-(U40-Pad5)
- U55 pad 3: /ALU/AGTBF -> /ALU/A9
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
Commit message: test
Parts:
- moved C24 1152.9 mm to (1046.6, 134.8)
- moved C25 1152.9 mm to (1046.6, 141.7)
- moved C26 1152.9 mm to (1046.6, 148.6)
- moved C27 1152.9 mm to (1117.4, 140.8)
- moved U66 1152.9 mm to (1117.3, 206.1)
- moved U67 1152.9 mm to (1128.5, 188.9)
- moved U68 1152.9 mm to (1128.5, 211.2)
- moved U69 1152.9 mm to (1117.3, 168.6)
- moved U70 1152.9 mm to (1128.5, 146.3)
- moved U71 1152.9 mm to (1117.3, 146.3)
- moved U72 1152.9 mm to (1072.4, 134.3)
- moved U73 1152.9 mm to (1098.5, 138.6)
- moved U74 1152.9 mm to (1084.2, 199.4)
- moved U75 1152.9 mm to (1058.2, 199.4)
- moved U76 1152.9 mm to (1098.4, 158.4)
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Routing:
- net /Control-Unit/I7: track 0.00 -> 110.9 mm
- net /Control-Unit/I6: track 0.00 -> 99.9 mm
- net GND: track 0.00 -> 95.2 mm
- net /Control-Unit/I5: track 0.00 -> 93.3 mm
- net /Control-Unit/I0: track 0.00 -> 84.4 mm
- net /Control-Unit/I1: track 0.00 -> 79.0 mm
- net /Control-Unit/I4: track 0.00 -> 75.9 mm
- net /Control-Unit/I2: track 0.00 -> 75.8 mm
- net /Control-Unit/I3: track 0.00 -> 71.4 mm
- net /ALU/BUS0: track 0.00 -> 21.6 mm, vias 0 -> 1
- net /Instruction-Register/sheet621E2544/I12: track 0.00 -> 20.7 mm
- net /ALU/BUS1: track 0.00 -> 20.3 mm, vias 0 -> 1
- net /Instruction-Register/sheet621E2544/I8: track 0.00 -> 20.0 mm
- net /ALU/BUS2: track 0.00 -> 19.1 mm, vias 0 -> 1
- net /Instruction-Register/sheet621E2544/I9: track 0.00 -> 18.4 mm
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