File: ProgramCounter.sch (KiCad schematic (older format))
At the start: 6 parts

Commit message: Added footprints
Parts:
- U45, U46, U47, U48: renamed from U?; footprint (none) -> Package_DIP:DIP-16_W7.62mm
- gave numbers to parts that had none: 2
Changed lines of the file:
@@
 AR Path="/603B766D/5F6D5FCC" Ref="#PWR?"  Part="1"
 AR Path="/5F74778C/5F6D5FCC" Ref="#PWR?"  Part="1"
-AR Path="/5F6ACD14/5F6D5FCC" Ref="#PWR0167"  Part="1"
-F 0 "#PWR0167" H 4750 4200 50  0001 C CNN
+AR Path="/5F6ACD14/5F6D5FCC" Ref="#PWR0122"  Part="1"
+F 0 "#PWR0122" H 4750 4200 50  0001 C CNN
 F 1 "GND" H 4755 4277 50  0000 C CNN
 F 2 "" H 4750 4450 50  0001 C CNN
@@
 AR Path="/603B766D/5F6D5FE4" Ref="#PWR?"  Part="1"
 AR Path="/5F74778C/5F6D5FE4" Ref="#PWR?"  Part="1"
-AR Path="/5F6ACD14/5F6D5FE4" Ref="#PWR0168"  Part="1"
-F 0 "#PWR0168" H 3150 3400 50  0001 C CNN
+AR Path="/5F6ACD14/5F6D5FE4" Ref="#PWR0118"  Part="1"
+F 0 "#PWR0118" H 3150 3400 50  0001 C CNN
 F 1 "GND" H 3155 3477 50  0000 C CNN
 F 2 "" H 3150 3650 50  0001 C CNN
@@
 AR Path="/603B766D/5F6D5FF6" Ref="#PWR?"  Part="1"
 AR Path="/5F74778C/5F6D5FF6" Ref="#PWR?"  Part="1"
-AR Path="/5F6ACD14/5F6D5FF6" Ref="#PWR0169"  Part="1"
-F 0 "#PWR0169" H 3150 4300 50  0001 C CNN
+AR Path="/5F6ACD14/5F6D5FF6" Ref="#PWR0120"  Part="1"
+F 0 "#PWR0120" H 3150 4300 50  0001 C CNN
 F 1 "+5V" H 3165 4623 50  0000 C CNN
 F 2 "" H 3150 4450 50  0001 C CNN
@@
 AR Path="/603B766D/5F6D6094" Ref="U?"  Part="1"
 AR Path="/5F74778C/5F6D6094" Ref="U?"  Part="1"
-AR Path="/5F6ACD14/5F6D6094" Ref="U?"  Part="1"
-F 0 "U?" V 2396 2806 50  0000 R CNN
+AR Path="/5F6ACD14/5F6D6094" Ref="U43"  Part="1"
+F 0 "U43" V 2396 2806 50  0000 R CNN
 F 1 "74LS245" V 2305 2806 50  0000 R CNN
 F 2 "Package_DIP:DIP-20_W7.62mm" H 2350 3650 50  0001 C CNN
@@
 AR Path="/603B766D/5F6D60A0" Ref="#PWR?"  Part="1"
 AR Path="/5F74778C/5F6D60A0" Ref="#PWR?"  Part="1"
-AR Path="/5F6ACD14/5F6D60A0" Ref="#PWR0170"  Part="1"
-F 0 "#PWR0170" H 4750 4200 50  0001 C CNN
+AR Path="/5F6ACD14/5F6D60A0" Ref="#PWR0123"  Part="1"
+F 0 "#PWR0123" H 4750 4200 50  0001 C CNN
 F 1 "GND" H 4755 4277 50  0000 C CNN
 F 2 "" H 4750 4450 50  0001 C CNN
@@
 AR Path="/603B766D/5F6D60B8" Ref="#PWR?"  Part="1"
 AR Path="/5F74778C/5F6D60B8" Ref="#PWR?"  Part="1"
-AR Path="/5F6ACD14/5F6D60B8" Ref="#PWR0171"  Part="1"
-F 0 "#PWR0171" H 3150 3400 50  0001 C CNN
+AR Path="/5F6ACD14/5F6D60B8" Ref="#PWR0119"  Part="1"
+F 0 "#PWR0119" H 3150 3400 50  0001 C CNN
 F 1 "GND" H 3155 3477 50  0000 C CNN
 F 2 "" H 3150 3650 50  0001 C CNN
@@
 AR Path="/603B766D/5F6D60C4" Ref="#PWR?"  Part="1"
 AR Path="/5F74778C/5F6D60C4" Ref="#PWR?"  Part="1"
-AR Path="/5F6ACD14/5F6D60C4" Ref="#PWR0172"  Part="1"
-F 0 "#PWR0172" H 1550 3500 50  0001 C CNN
+AR Path="/5F6ACD14/5F6D60C4" Ref="#PWR0116"  Part="1"
+F 0 "#PWR0116" H 1550 3500 50  0001 C CNN
 F 1 "+5V" H 1565 3823 50  0000 C CNN
 F 2 "" H 1550 3650 50  0001 C CNN
@@
 AR Path="/603B766D/5F6D60D0" Ref="#PWR?"  Part="1"
 AR Path="/5F74778C/5F6D60D0" Ref="#PWR?"  Part="1"
-AR Path="/5F6ACD14/5F6D60D0" Ref="#PWR0173"  Part="1"
-F 0 "#PWR0173" H 3150 4300 50  0001 C CNN
+AR Path="/5F6ACD14/5F6D60D0" Ref="#PWR0121"  Part="1"
+F 0 "#PWR0121" H 3150 4300 50  0001 C CNN
 F 1 "+5V" H 3165 4623 50  0000 C CNN
 F 2 "" H 3150 4450 50  0001 C CNN
@@
 AR Path="/603B766D/5F6D6117" Ref="U?"  Part="1"
 AR Path="/5F74778C/5F6D6117" Ref="U?"  Part="1"
-AR Path="/5F6ACD14/5F6D6117" Ref="U?"  Part="1"
-F 0 "U?" V 3996 3606 50  0000 R CNN
+AR Path="/5F6ACD14/5F6D6117" Ref="U44"  Part="1"
+F 0 "U44" V 3996 3606 50  0000 R CNN
 F 1 "74LS245" V 3905 3606 50  0000 R CNN
 F 2 "Package_DIP:DIP-20_W7.62mm" H 3950 4450 50  0001 C CNN
@@
 AR Path="/603B766D/5F6D6186" Ref="#PWR?"  Part="1"
 AR Path="/5F74778C/5F6D6186" Ref="#PWR?"  Part="1"
-AR Path="/5F6ACD14/5F6D6186" Ref="#PWR0174"  Part="1"
-F 0 "#PWR0174" H 1550 3500 50  0001 C CNN
+AR Path="/5F6ACD14/5F6D6186" Ref="#PWR0117"  Part="1"
+F 0 "#PWR0117" H 1550 3500 50  0001 C CNN
 F 1 "+5V" H 1565 3823 50  0000 C CNN
 F 2 "" H 1550 3650 50  0001 C CNN
@@
 	1550 4650 1550 3650
 $Comp
-L 74xx:74LS161 U?
+L 74xx:74LS161 U45
 U 1 1 5F779E04
 P 6100 4450
-F 0 "U?" V 6054 5294 50  0000 L CNN
+F 0 "U45" V 6054 5294 50  0000 L CNN
 F 1 "74LS161" V 6145 5294 50  0000 L CNN
-F 2 "" H 6100 4450 50  0001 C CNN
+F 2 "Package_DIP:DIP-16_W7.62mm" H 6100 4450 50  0001 C CNN
 F 3 "http://www.ti.com/lit/gpn/sn74LS161" H 6100 4450 50  0001 C CNN
 	1    6100 4450
@@
 $EndComp
 $Comp
-L 74xx:74LS161 U?
+L 74xx:74LS161 U47
 U 1 1 5F77F8AA
 P 9900 4450
-F 0 "U?" V 9854 5294 50  0000 L CNN
+F 0 "U47" V 9854 5294 50  0000 L CNN
 F 1 "74LS161" V 9945 5294 50  0000 L CNN
-F 2 "" H 9900 4450 50  0001 C CNN
+F 2 "Package_DIP:DIP-16_W7.62mm" H 9900 4450 50  0001 C CNN
 F 3 "http://www.ti.com/lit/gpn/sn74LS161" H 9900 4450 50  0001 C CNN
 	1    9900 4450
@@
 $EndComp
 $Comp
-L 74xx:74LS161 U?
+L 74xx:74LS161 U48
 U 1 1 5F780CA7
 P 11750 4450
-F 0 "U?" V 11704 5294 50  0000 L CNN
+F 0 "U48" V 11704 5294 50  0000 L CNN
 F 1 "74LS161" V 11795 5294 50  0000 L CNN
-F 2 "" H 11750 4450 50  0001 C CNN
+F 2 "Package_DIP:DIP-16_W7.62mm" H 11750 4450 50  0001 C CNN
 F 3 "http://www.ti.com/lit/gpn/sn74LS161" H 11750 4450 50  0001 C CNN
 	1    11750 4450
@@
 	8050 4950 8050 5200
 $Comp
-L 74xx:74LS161 U?
+L 74xx:74LS161 U46
 U 1 1 5F77E072
 P 8050 4450
-F 0 "U?" V 8004 5294 50  0000 L CNN
+F 0 "U46" V 8004 5294 50  0000 L CNN
 F 1 "74LS161" V 8095 5294 50  0000 L CNN
-F 2 "" H 8050 4450 50  0001 C CNN
+F 2 "Package_DIP:DIP-16_W7.62mm" H 8050 4450 50  0001 C CNN
 F 3 "http://www.ti.com/lit/gpn/sn74LS161" H 8050 4450 50  0001 C CNN
 	1    8050 4450
@@
 	6900 4450 6900 4250
 $Comp
-L power:+5V #PWR0175
+L power:+5V #PWR0125
 U 1 1 5F9A8E46
 P 6900 4250
-F 0 "#PWR0175" H 6900 4100 50  0001 C CNN
+F 0 "#PWR0125" H 6900 4100 50  0001 C CNN
 F 1 "+5V" H 6915 4423 50  0000 C CNN
 F 2 "" H 6900 4250 50  0001 C CNN
@@
 $EndComp
 $Comp
-L power:+5V #PWR0176
+L power:+5V #PWR0127
 U 1 1 5F9B1DDA
 P 8850 4400
-F 0 "#PWR0176" H 8850 4250 50  0001 C CNN
+F 0 "#PWR0127" H 8850 4250 50  0001 C CNN
 F 1 "+5V" H 8865 4573 50  0000 C CNN
 F 2 "" H 8850 4400 50  0001 C CNN
@@
 	8850 4400 8850 4450
 $Comp
-L power:+5V #PWR0177
+L power:+5V #PWR0129
 U 1 1 5F9BCAE2
 P 10700 4450
-F 0 "#PWR0177" H 10700 4300 50  0001 C CNN
+F 0 "#PWR0129" H 10700 4300 50  0001 C CNN
 F 1 "+5V" H 10715 4623 50  0000 C CNN
 F 2 "" H 10700 4450 50  0001 C CNN
@@
 $EndComp
 $Comp
-L power:+5V #PWR0178
+L power:+5V #PWR0131
 U 1 1 5F9BD87F
 P 12550 4450
-F 0 "#PWR0178" H 12550 4300 50  0001 C CNN
+F 0 "#PWR0131" H 12550 4300 50  0001 C CNN
 F 1 "+5V" H 12565 4623 50  0000 C CNN
 F 2 "" H 12550 4450 50  0001 C CNN
@@
 $EndComp
 $Comp
-L power:GND #PWR0179
+L power:GND #PWR0124
 U 1 1 5F9BEDE2
 P 5300 4450
-F 0 "#PWR0179" H 5300 4200 50  0001 C CNN
+F 0 "#PWR0124" H 5300 4200 50  0001 C CNN
 F 1 "GND" H 5305 4277 50  0000 C CNN
 F 2 "" H 5300 4450 50  0001 C CNN
@@
 $EndComp
 $Comp
-L power:GND #PWR0180
+L power:GND #PWR0126
 U 1 1 5F9C426E
 P 7250 4450
-F 0 "#PWR0180" H 7250 4200 50  0001 C CNN
+F 0 "#PWR0126" H 7250 4200 50  0001 C CNN
 F 1 "GND" H 7255 4277 50  0000 C CNN
 F 2 "" H 7250 4450 50  0001 C CNN
@@
 $EndComp
 $Comp
-L power:GND #PWR0181
+L power:GND #PWR0128
 U 1 1 5F9CE333
 P 9100 4450
-F 0 "#PWR0181" H 9100 4200 50  0001 C CNN
+F 0 "#PWR0128" H 9100 4200 50  0001 C CNN
 F 1 "GND" H 9105 4277 50  0000 C CNN
 F 2 "" H 9100 4450 50  0001 C CNN
@@
 $EndComp
 $Comp
-L power:GND #PWR0182
+L power:GND #PWR0130
 U 1 1 5F9D8AA1
 P 10950 4450
-F 0 "#PWR0182" H 10950 4200 50  0001 C CNN
+F 0 "#PWR0130" H 10950 4200 50  0001 C CNN
 F 1 "GND" H 10955 4277 50  0000 C CNN
 F 2 "" H 10950 4450 50  0001 C CNN

Commit message: Fixed power for multi part comps
Parts:
- renumbered U43 to U29, U44 to U30, U45 to U31, U46 to U32, U47 to U33, U48 to U34
Changed lines of the file:
@@
 AR Path="/603B766D/5F6D5FCC" Ref="#PWR?"  Part="1"
 AR Path="/5F74778C/5F6D5FCC" Ref="#PWR?"  Part="1"
-AR Path="/5F6ACD14/5F6D5FCC" Ref="#PWR0122"  Part="1"
-F 0 "#PWR0122" H 4750 4200 50  0001 C CNN
+AR Path="/5F6ACD14/5F6D5FCC" Ref="#PWR091"  Part="1"
+F 0 "#PWR091" H 4750 4200 50  0001 C CNN
 F 1 "GND" H 4755 4277 50  0000 C CNN
 F 2 "" H 4750 4450 50  0001 C CNN
@@
 AR Path="/603B766D/5F6D5FE4" Ref="#PWR?"  Part="1"
 AR Path="/5F74778C/5F6D5FE4" Ref="#PWR?"  Part="1"
-AR Path="/5F6ACD14/5F6D5FE4" Ref="#PWR0118"  Part="1"
-F 0 "#PWR0118" H 3150 3400 50  0001 C CNN
+AR Path="/5F6ACD14/5F6D5FE4" Ref="#PWR087"  Part="1"
+F 0 "#PWR087" H 3150 3400 50  0001 C CNN
 F 1 "GND" H 3155 3477 50  0000 C CNN
 F 2 "" H 3150 3650 50  0001 C CNN
@@
 AR Path="/603B766D/5F6D5FF6" Ref="#PWR?"  Part="1"
 AR Path="/5F74778C/5F6D5FF6" Ref="#PWR?"  Part="1"
-AR Path="/5F6ACD14/5F6D5FF6" Ref="#PWR0120"  Part="1"
-F 0 "#PWR0120" H 3150 4300 50  0001 C CNN
+AR Path="/5F6ACD14/5F6D5FF6" Ref="#PWR089"  Part="1"
+F 0 "#PWR089" H 3150 4300 50  0001 C CNN
 F 1 "+5V" H 3165 4623 50  0000 C CNN
 F 2 "" H 3150 4450 50  0001 C CNN
@@
 AR Path="/603B766D/5F6D6094" Ref="U?"  Part="1"
 AR Path="/5F74778C/5F6D6094" Ref="U?"  Part="1"
-AR Path="/5F6ACD14/5F6D6094" Ref="U43"  Part="1"
-F 0 "U43" V 2396 2806 50  0000 R CNN
+AR Path="/5F6ACD14/5F6D6094" Ref="U29"  Part="1"
+F 0 "U29" V 2396 2806 50  0000 R CNN
 F 1 "74LS245" V 2305 2806 50  0000 R CNN
 F 2 "Package_DIP:DIP-20_W7.62mm" H 2350 3650 50  0001 C CNN
@@
 AR Path="/603B766D/5F6D60A0" Ref="#PWR?"  Part="1"
 AR Path="/5F74778C/5F6D60A0" Ref="#PWR?"  Part="1"
-AR Path="/5F6ACD14/5F6D60A0" Ref="#PWR0123"  Part="1"
-F 0 "#PWR0123" H 4750 4200 50  0001 C CNN
+AR Path="/5F6ACD14/5F6D60A0" Ref="#PWR092"  Part="1"
+F 0 "#PWR092" H 4750 4200 50  0001 C CNN
 F 1 "GND" H 4755 4277 50  0000 C CNN
 F 2 "" H 4750 4450 50  0001 C CNN
@@
 AR Path="/603B766D/5F6D60B8" Ref="#PWR?"  Part="1"
 AR Path="/5F74778C/5F6D60B8" Ref="#PWR?"  Part="1"
-AR Path="/5F6ACD14/5F6D60B8" Ref="#PWR0119"  Part="1"
-F 0 "#PWR0119" H 3150 3400 50  0001 C CNN
+AR Path="/5F6ACD14/5F6D60B8" Ref="#PWR088"  Part="1"
+F 0 "#PWR088" H 3150 3400 50  0001 C CNN
 F 1 "GND" H 3155 3477 50  0000 C CNN
 F 2 "" H 3150 3650 50  0001 C CNN
@@
 AR Path="/603B766D/5F6D60C4" Ref="#PWR?"  Part="1"
 AR Path="/5F74778C/5F6D60C4" Ref="#PWR?"  Part="1"
-AR Path="/5F6ACD14/5F6D60C4" Ref="#PWR0116"  Part="1"
-F 0 "#PWR0116" H 1550 3500 50  0001 C CNN
+AR Path="/5F6ACD14/5F6D60C4" Ref="#PWR085"  Part="1"
+F 0 "#PWR085" H 1550 3500 50  0001 C CNN
 F 1 "+5V" H 1565 3823 50  0000 C CNN
 F 2 "" H 1550 3650 50  0001 C CNN
@@
 AR Path="/603B766D/5F6D60D0" Ref="#PWR?"  Part="1"
 AR Path="/5F74778C/5F6D60D0" Ref="#PWR?"  Part="1"
-AR Path="/5F6ACD14/5F6D60D0" Ref="#PWR0121"  Part="1"
-F 0 "#PWR0121" H 3150 4300 50  0001 C CNN
+AR Path="/5F6ACD14/5F6D60D0" Ref="#PWR090"  Part="1"
+F 0 "#PWR090" H 3150 4300 50  0001 C CNN
 F 1 "+5V" H 3165 4623 50  0000 C CNN
 F 2 "" H 3150 4450 50  0001 C CNN
@@
 AR Path="/603B766D/5F6D6117" Ref="U?"  Part="1"
 AR Path="/5F74778C/5F6D6117" Ref="U?"  Part="1"
-AR Path="/5F6ACD14/5F6D6117" Ref="U44"  Part="1"
-F 0 "U44" V 3996 3606 50  0000 R CNN
+AR Path="/5F6ACD14/5F6D6117" Ref="U30"  Part="1"
+F 0 "U30" V 3996 3606 50  0000 R CNN
 F 1 "74LS245" V 3905 3606 50  0000 R CNN
 F 2 "Package_DIP:DIP-20_W7.62mm" H 3950 4450 50  0001 C CNN
@@
 AR Path="/603B766D/5F6D6186" Ref="#PWR?"  Part="1"
 AR Path="/5F74778C/5F6D6186" Ref="#PWR?"  Part="1"
-AR Path="/5F6ACD14/5F6D6186" Ref="#PWR0117"  Part="1"
-F 0 "#PWR0117" H 1550 3500 50  0001 C CNN
+AR Path="/5F6ACD14/5F6D6186" Ref="#PWR086"  Part="1"
+F 0 "#PWR086" H 1550 3500 50  0001 C CNN
 F 1 "+5V" H 1565 3823 50  0000 C CNN
 F 2 "" H 1550 3650 50  0001 C CNN
@@
 	1550 4650 1550 3650
 $Comp
-L 74xx:74LS161 U45
+L 74xx:74LS161 U31
 U 1 1 5F779E04
 P 6100 4450
-F 0 "U45" V 6054 5294 50  0000 L CNN
+F 0 "U31" V 6054 5294 50  0000 L CNN
 F 1 "74LS161" V 6145 5294 50  0000 L CNN
 F 2 "Package_DIP:DIP-16_W7.62mm" H 6100 4450 50  0001 C CNN
@@
 $EndComp
 $Comp
-L 74xx:74LS161 U47
+L 74xx:74LS161 U33
 U 1 1 5F77F8AA
 P 9900 4450
-F 0 "U47" V 9854 5294 50  0000 L CNN
+F 0 "U33" V 9854 5294 50  0000 L CNN
 F 1 "74LS161" V 9945 5294 50  0000 L CNN
 F 2 "Package_DIP:DIP-16_W7.62mm" H 9900 4450 50  0001 C CNN
@@
 $EndComp
 $Comp
-L 74xx:74LS161 U48
+L 74xx:74LS161 U34
 U 1 1 5F780CA7
 P 11750 4450
-F 0 "U48" V 11704 5294 50  0000 L CNN
+F 0 "U34" V 11704 5294 50  0000 L CNN
 F 1 "74LS161" V 11795 5294 50  0000 L CNN
 F 2 "Package_DIP:DIP-16_W7.62mm" H 11750 4450 50  0001 C CNN
@@
 	8050 4950 8050 5200
 $Comp
-L 74xx:74LS161 U46
+L 74xx:74LS161 U32
 U 1 1 5F77E072
 P 8050 4450
-F 0 "U46" V 8004 5294 50  0000 L CNN
+F 0 "U32" V 8004 5294 50  0000 L CNN
 F 1 "74LS161" V 8095 5294 50  0000 L CNN
 F 2 "Package_DIP:DIP-16_W7.62mm" H 8050 4450 50  0001 C CNN
@@
 	6900 4450 6900 4250
 $Comp
-L power:+5V #PWR0125
+L power:+5V #PWR094
 U 1 1 5F9A8E46
 P 6900 4250
-F 0 "#PWR0125" H 6900 4100 50  0001 C CNN
+F 0 "#PWR094" H 6900 4100 50  0001 C CNN
 F 1 "+5V" H 6915 4423 50  0000 C CNN
 F 2 "" H 6900 4250 50  0001 C CNN
@@
 $EndComp
 $Comp
-L power:+5V #PWR0127
+L power:+5V #PWR096
 U 1 1 5F9B1DDA
 P 8850 4400
-F 0 "#PWR0127" H 8850 4250 50  0001 C CNN
+F 0 "#PWR096" H 8850 4250 50  0001 C CNN
 F 1 "+5V" H 8865 4573 50  0000 C CNN
 F 2 "" H 8850 4400 50  0001 C CNN
@@
 	8850 4400 8850 4450
 $Comp
-L power:+5V #PWR0129
+L power:+5V #PWR098
 U 1 1 5F9BCAE2
 P 10700 4450
-F 0 "#PWR0129" H 10700 4300 50  0001 C CNN
+F 0 "#PWR098" H 10700 4300 50  0001 C CNN
 F 1 "+5V" H 10715 4623 50  0000 C CNN
 F 2 "" H 10700 4450 50  0001 C CNN
@@
 $EndComp
 $Comp
-L power:+5V #PWR0131
+L power:+5V #PWR0100
 U 1 1 5F9BD87F
 P 12550 4450
-F 0 "#PWR0131" H 12550 4300 50  0001 C CNN
+F 0 "#PWR0100" H 12550 4300 50  0001 C CNN
 F 1 "+5V" H 12565 4623 50  0000 C CNN
 F 2 "" H 12550 4450 50  0001 C CNN
@@
 $EndComp
 $Comp
-L power:GND #PWR0124
+L power:GND #PWR093
 U 1 1 5F9BEDE2
 P 5300 4450
-F 0 "#PWR0124" H 5300 4200 50  0001 C CNN
+F 0 "#PWR093" H 5300 4200 50  0001 C CNN
 F 1 "GND" H 5305 4277 50  0000 C CNN
 F 2 "" H 5300 4450 50  0001 C CNN
@@
 $EndComp
 $Comp
-L power:GND #PWR0126
+L power:GND #PWR095
 U 1 1 5F9C426E
 P 7250 4450
-F 0 "#PWR0126" H 7250 4200 50  0001 C CNN
+F 0 "#PWR095" H 7250 4200 50  0001 C CNN
 F 1 "GND" H 7255 4277 50  0000 C CNN
 F 2 "" H 7250 4450 50  0001 C CNN
@@
 $EndComp
 $Comp
-L power:GND #PWR0128
+L power:GND #PWR097
 U 1 1 5F9CE333
 P 9100 4450
-F 0 "#PWR0128" H 9100 4200 50  0001 C CNN
+F 0 "#PWR097" H 9100 4200 50  0001 C CNN
 F 1 "GND" H 9105 4277 50  0000 C CNN
 F 2 "" H 9100 4450 50  0001 C CNN
@@
 $EndComp
 $Comp
-L power:GND #PWR0130
+L power:GND #PWR099
 U 1 1 5F9D8AA1
 P 10950 4450
-F 0 "#PWR0130" H 10950 4200 50  0001 C CNN
+F 0 "#PWR099" H 10950 4200 50  0001 C CNN
 F 1 "GND" H 10955 4277 50  0000 C CNN
 F 2 "" H 10950 4450 50  0001 C CNN

Commit message: Fixed ZIF
Parts:
- U29, U30: symbol 74xx:74LS245 -> 16bitCpu-rescue:74LS245-74xx
- U31, U32, U33, U34: symbol 74xx:74LS161 -> 16bitCpu-rescue:74LS161-74xx
Changed lines of the file:
@@
 	4150 3950 4150 2500
 $Comp
-L power:GND #PWR?
+L 16bitCpu-rescue:GND-power #PWR?
 U 1 1 5F6D5FCC
 P 4750 4450
@@
 $EndComp
 $Comp
-L power:GND #PWR?
+L 16bitCpu-rescue:GND-power #PWR?
 U 1 1 5F6D5FE4
 P 3150 3650
@@
 $EndComp
 $Comp
-L power:+5V #PWR?
+L 16bitCpu-rescue:+5V-power #PWR?
 U 1 1 5F6D5FF6
 P 3150 4450
@@
 Connection ~ 3150 4450
 $Comp
-L 74xx:74LS245 U?
+L 16bitCpu-rescue:74LS245-74xx U?
 U 1 1 5F6D6094
 P 2350 3650
@@
 $EndComp
 $Comp
-L power:GND #PWR?
+L 16bitCpu-rescue:GND-power #PWR?
 U 1 1 5F6D60A0
 P 4750 4450
@@
 $EndComp
 $Comp
-L power:GND #PWR?
+L 16bitCpu-rescue:GND-power #PWR?
 U 1 1 5F6D60B8
 P 3150 3650
@@
 $EndComp
 $Comp
-L power:+5V #PWR?
+L 16bitCpu-rescue:+5V-power #PWR?
 U 1 1 5F6D60C4
 P 1550 3650
@@
 $EndComp
 $Comp
-L power:+5V #PWR?
+L 16bitCpu-rescue:+5V-power #PWR?
 U 1 1 5F6D60D0
 P 3150 4450
@@
 Bus14
 $Comp
-L 74xx:74LS245 U?
+L 16bitCpu-rescue:74LS245-74xx U?
 U 1 1 5F6D6117
 P 3950 4450
@@
 Connection ~ 2550 1700
 $Comp
-L power:+5V #PWR?
+L 16bitCpu-rescue:+5V-power #PWR?
 U 1 1 5F6D6186
 P 1550 3650
@@
 	1550 4650 1550 3650
 $Comp
-L 74xx:74LS161 U31
+L 16bitCpu-rescue:74LS161-74xx U31
 U 1 1 5F779E04
 P 6100 4450
+AR Path="/5F779E04" Ref="U31"  Part="1"
+AR Path="/5F6ACD14/5F779E04" Ref="U31"  Part="1"
 F 0 "U31" V 6054 5294 50  0000 L CNN
 F 1 "74LS161" V 6145 5294 50  0000 L CNN
@@
 $EndComp
 $Comp
-L 74xx:74LS161 U33
+L 16bitCpu-rescue:74LS161-74xx U33
 U 1 1 5F77F8AA
 P 9900 4450
+AR Path="/5F77F8AA" Ref="U33"  Part="1"
+AR Path="/5F6ACD14/5F77F8AA" Ref="U33"  Part="1"
 F 0 "U33" V 9854 5294 50  0000 L CNN
 F 1 "74LS161" V 9945 5294 50  0000 L CNN
@@
 $EndComp
 $Comp
-L 74xx:74LS161 U34
+L 16bitCpu-rescue:74LS161-74xx U34
 U 1 1 5F780CA7
 P 11750 4450
+AR Path="/5F780CA7" Ref="U34"  Part="1"
+AR Path="/5F6ACD14/5F780CA7" Ref="U34"  Part="1"
 F 0 "U34" V 11704 5294 50  0000 L CNN
 F 1 "74LS161" V 11795 5294 50  0000 L CNN
@@
 	8050 4950 8050 5200
 $Comp
-L 74xx:74LS161 U32
+L 16bitCpu-rescue:74LS161-74xx U32
 U 1 1 5F77E072
 P 8050 4450
+AR Path="/5F77E072" Ref="U32"  Part="1"
+AR Path="/5F6ACD14/5F77E072" Ref="U32"  Part="1"
 F 0 "U32" V 8004 5294 50  0000 L CNN
 F 1 "74LS161" V 8095 5294 50  0000 L CNN
@@
 	6900 4450 6900 4250
 $Comp
-L power:+5V #PWR094
+L 16bitCpu-rescue:+5V-power #PWR094
 U 1 1 5F9A8E46
 P 6900 4250
+AR Path="/5F9A8E46" Ref="#PWR094"  Part="1"
+AR Path="/5F6ACD14/5F9A8E46" Ref="#PWR094"  Part="1"
 F 0 "#PWR094" H 6900 4100 50  0001 C CNN
 F 1 "+5V" H 6915 4423 50  0000 C CNN
@@
 $EndComp
 $Comp
-L power:+5V #PWR096
+L 16bitCpu-rescue:+5V-power #PWR096
 U 1 1 5F9B1DDA
 P 8850 4400
+AR Path="/5F9B1DDA" Ref="#PWR096"  Part="1"
+AR Path="/5F6ACD14/5F9B1DDA" Ref="#PWR096"  Part="1"
 F 0 "#PWR096" H 8850 4250 50  0001 C CNN
 F 1 "+5V" H 8865 4573 50  0000 C CNN
@@
 	8850 4400 8850 4450
 $Comp
-L power:+5V #PWR098
+L 16bitCpu-rescue:+5V-power #PWR098
 U 1 1 5F9BCAE2
 P 10700 4450
+AR Path="/5F9BCAE2" Ref="#PWR098"  Part="1"
+AR Path="/5F6ACD14/5F9BCAE2" Ref="#PWR098"  Part="1"
 F 0 "#PWR098" H 10700 4300 50  0001 C CNN
 F 1 "+5V" H 10715 4623 50  0000 C CNN
@@
 $EndComp
 $Comp
-L power:+5V #PWR0100
+L 16bitCpu-rescue:+5V-power #PWR0100
 U 1 1 5F9BD87F
 P 12550 4450
+AR Path="/5F9BD87F" Ref="#PWR0100"  Part="1"
+AR Path="/5F6ACD14/5F9BD87F" Ref="#PWR0100"  Part="1"
 F 0 "#PWR0100" H 12550 4300 50  0001 C CNN
 F 1 "+5V" H 12565 4623 50  0000 C CNN
@@
 $EndComp
 $Comp
-L power:GND #PWR093
+L 16bitCpu-rescue:GND-power #PWR093
 U 1 1 5F9BEDE2
 P 5300 4450
+AR Path="/5F9BEDE2" Ref="#PWR093"  Part="1"
+AR Path="/5F6ACD14/5F9BEDE2" Ref="#PWR093"  Part="1"
 F 0 "#PWR093" H 5300 4200 50  0001 C CNN
 F 1 "GND" H 5305 4277 50  0000 C CNN
@@
 $EndComp
 $Comp
-L power:GND #PWR095
+L 16bitCpu-rescue:GND-power #PWR095
 U 1 1 5F9C426E
 P 7250 4450
+AR Path="/5F9C426E" Ref="#PWR095"  Part="1"
+AR Path="/5F6ACD14/5F9C426E" Ref="#PWR095"  Part="1"
 F 0 "#PWR095" H 7250 4200 50  0001 C CNN
 F 1 "GND" H 7255 4277 50  0000 C CNN
@@
 $EndComp
 $Comp
-L power:GND #PWR097
+L 16bitCpu-rescue:GND-power #PWR097
 U 1 1 5F9CE333
 P 9100 4450
+AR Path="/5F9CE333" Ref="#PWR097"  Part="1"
+AR Path="/5F6ACD14/5F9CE333" Ref="#PWR097"  Part="1"
 F 0 "#PWR097" H 9100 4200 50  0001 C CNN
 F 1 "GND" H 9105 4277 50  0000 C CNN
@@
 $EndComp
 $Comp
-L power:GND #PWR099
+L 16bitCpu-rescue:GND-power #PWR099
 U 1 1 5F9D8AA1
 P 10950 4450
+AR Path="/5F9D8AA1" Ref="#PWR099"  Part="1"
+AR Path="/5F6ACD14/5F9D8AA1" Ref="#PWR099"  Part="1"
 F 0 "#PWR099" H 10950 4200 50  0001 C CNN
 F 1 "GND" H 10955 4277 50  0000 C CNN
