File: ProgramCounter.sch (KiCad schematic (older format))
At the start: 6 parts, among them U29 74LS245, U30 74LS245, U31 74LS161, U32 74LS161, U33 74LS161, U34 74LS161

Commit message: Let there be light
Connections:
- wire segments 207 -> 239
- no-connect marks 0 -> 1
Changed lines of the file:
@@
 $Descr A3 16535 11693
 encoding utf-8
-Sheet 6 11
+Sheet 9 20
 Title ""
 Date ""
@@
 	6600 6750 6600 4950
 Wire Wire Line
-	1850 6750 6600 6750
+	1850 6750 4600 6750
 Wire Wire Line
 	6500 4950 6500 6700
 Wire Wire Line
-	6500 6700 1950 6700
+	6500 6700 4700 6700
 Wire Wire Line
 	1950 6700 1950 4150
@@
 	2050 4150 2050 6650
 Wire Wire Line
-	2050 6650 6400 6650
-Wire Wire Line
 	6400 6650 6400 4950
 Wire Wire Line
@@
 	2150 6600 2150 4150
 Wire Wire Line
-	6300 6600 2150 6600
+	6300 6600 4900 6600
 Wire Wire Line
 	2250 4150 2250 6550
 Wire Wire Line
-	2250 6550 8550 6550
-Wire Wire Line
-	8450 6500 2350 6500
+	2250 6550 5000 6550
+Wire Wire Line
+	8450 6500 5100 6500
 Wire Wire Line
 	2350 6500 2350 4150
@@
 	2450 4150 2450 6450
 Wire Wire Line
-	2450 6450 8350 6450
-Wire Wire Line
-	8250 6400 2550 6400
+	2450 6450 5200 6450
+Wire Wire Line
+	8250 6400 5300 6400
 Wire Wire Line
 	2550 6400 2550 4150
@@
 	3450 4950 3450 6350
 Wire Wire Line
-	3450 6350 10400 6350
-Wire Wire Line
 	10400 6350 10400 4950
 Wire Wire Line
 	10300 4950 10300 6300
 Wire Wire Line
-	10300 6300 3550 6300
+	10300 6300 5500 6300
 Wire Wire Line
 	3550 6300 3550 4950
@@
 	3650 4950 3650 6250
 Wire Wire Line
-	3650 6250 10200 6250
+	3650 6250 5600 6250
 Wire Wire Line
 	10200 6250 10200 4950
@@
 	10100 4950 10100 6200
 Wire Wire Line
-	10100 6200 3750 6200
-Wire Wire Line
 	3750 6200 3750 4950
 Wire Wire Line
 	3850 4950 3850 6150
 Wire Wire Line
-	3850 6150 12250 6150
+	3850 6150 5800 6150
 Wire Wire Line
 	12250 6150 12250 4950
@@
 	12150 4950 12150 6100
 Wire Wire Line
-	12150 6100 3950 6100
+	12150 6100 5900 6100
 Wire Wire Line
 	3950 6100 3950 4950
@@
 	4050 4950 4050 6050
 Wire Wire Line
-	4050 6050 12050 6050
+	4050 6050 6000 6050
 Wire Wire Line
 	12050 6050 12050 4950
@@
 	11950 4950 11950 6000
 Wire Wire Line
-	11950 6000 4150 6000
+	11950 6000 6100 6000
 Wire Wire Line
 	4150 6000 4150 4950
@@
 Text HLabel 1150 2500 0    50   3State ~ 0
 Bus15
+NoConn ~ 11750 4950
+$Sheet
+S 4350 7100 1800 550
+U 6156E9B6
+F0 "sheet6156E9A4" 50
+F1 "led16.sch" 50
+F2 "I0" I T 4600 7100 50
+F3 "I1" I T 4700 7100 50
+F4 "I2" I T 4800 7100 50
+F5 "I3" I T 4900 7100 50
+F6 "I4" I T 5000 7100 50
+F7 "I5" I T 5100 7100 50
+F8 "I6" I T 5200 7100 50
+F9 "I7" I T 5300 7100 50
+F10 "I8" I T 5400 7100 50
+F11 "I9" I T 5500 7100 50
+F12 "I10" I T 5600 7100 50
+F13 "I11" I T 5700 7100 50
+F14 "I12" I T 5800 7100 50
+F15 "I13" I T 5900 7100 50
+F16 "I14" I T 6000 7100 50
+F17 "I15" I T 6100 7100 50
+$EndSheet
+Wire Wire Line
+	4600 7100 4600 6750
+Connection ~ 4600 6750
+Wire Wire Line
+	4600 6750 6600 6750
+Wire Wire Line
+	4700 7100 4700 6700
+Connection ~ 4700 6700
+Wire Wire Line
+	4700 6700 1950 6700
+Wire Wire Line
+	4800 7100 4800 6650
+Wire Wire Line
+	2050 6650 4800 6650
+Connection ~ 4800 6650
+Wire Wire Line
+	4800 6650 6400 6650
+Wire Wire Line
+	4900 7100 4900 6600
+Connection ~ 4900 6600
+Wire Wire Line
+	4900 6600 2150 6600
+Wire Wire Line
+	5000 7100 5000 6550
+Connection ~ 5000 6550
+Wire Wire Line
+	5000 6550 8550 6550
+Wire Wire Line
+	5100 7100 5100 6500
+Connection ~ 5100 6500
+Wire Wire Line
+	5100 6500 2350 6500
+Wire Wire Line
+	5200 7100 5200 6450
+Connection ~ 5200 6450
+Wire Wire Line
+	5200 6450 8350 6450
+Wire Wire Line
+	3450 6350 5400 6350
+Wire Wire Line
+	5300 7100 5300 6400
+Connection ~ 5300 6400
+Wire Wire Line
+	5300 6400 2550 6400
+Wire Wire Line
+	5400 7100 5400 6350
+Connection ~ 5400 6350
+Wire Wire Line
+	5400 6350 10400 6350
+Wire Wire Line
+	5500 7100 5500 6300
+Connection ~ 5500 6300
+Wire Wire Line
+	5500 6300 3550 6300
+Wire Wire Line
+	5600 7100 5600 6250
+Connection ~ 5600 6250
+Wire Wire Line
+	5600 6250 10200 6250
+Wire Wire Line
+	5700 7100 5700 6200
+Wire Wire Line
+	3750 6200 5700 6200
+Connection ~ 5700 6200
+Wire Wire Line
+	5700 6200 10100 6200
+Wire Wire Line
+	5800 7100 5800 6150
+Connection ~ 5800 6150
+Wire Wire Line
+	5800 6150 12250 6150
+Wire Wire Line
+	5900 7100 5900 6100
+Connection ~ 5900 6100
+Wire Wire Line
+	5900 6100 3950 6100
+Wire Wire Line
+	6000 7100 6000 6050
+Connection ~ 6000 6050
+Wire Wire Line
+	6000 6050 12050 6050
+Wire Wire Line
+	6100 7100 6100 6000
+Connection ~ 6100 6000
+Wire Wire Line
+	6100 6000 4150 6000
 $EndSCHEMATC
