File: ALU.sch (KiCad schematic (older format))
At the start: 15 parts, among them U1 74LS245, U10 74LS86, U2 74LS245, U3 74LS283, U4 74LS283, U5 74LS283, U53 74LS173, U54 74HC02, U55 74HC02, U56 74LS08, U57 74LS08, U6 74LS283, U7 74LS86, U8 74LS86, U9 74LS86

Commit message: Let there be light
Connections:
- net sheet61054F43/I1: now reaches U1.3 (A1), U3.1 (S2), U54.2
- net sheet61054F43/I3: now reaches U1.5 (A3), U3.10 (S4), U54.5
- net sheet61054F43/I2: now reaches U1.4 (A2), U3.13 (S3), U54.6
- net sheet61054F43/I0: now reaches U1.2 (A0), U3.4 (S1), U54.3
- net sheet61054F43/I5: now reaches U1.7 (A5), U5.1 (S2), U54.8
- net sheet61054F43/I7: now reaches U1.9 (A7), U5.10 (S4), U54.11
- net sheet61054F43/I6: now reaches U1.8 (A6), U5.13 (S3), U54.12
- net sheet61054F43/I4: now reaches U1.6 (A4), U5.4 (S1), U54.9
- net sheet61054F43/I13: now reaches U2.7 (A5), U55.8, U6.1 (S2)
- net sheet61054F43/I15: now reaches U2.9 (A7), U55.11, U6.10 (S4)
- net sheet61054F43/I14: now reaches U2.8 (A6), U55.12, U6.13 (S3)
- net sheet61054F43/I12: now reaches U2.6 (A4), U55.9, U6.4 (S1)
- net sheet61054F43/I9: now reaches U2.3 (A1), U4.1 (S2), U55.2
- net sheet61054F43/I11: now reaches U2.5 (A3), U4.10 (S4), U55.5
- net sheet61054F43/I10: now reaches U2.4 (A2), U4.13 (S3), U55.6
- net sheet61054F43/I8: now reaches U2.2 (A0), U4.4 (S1), U55.3
- no-connect marks 5 -> 4
Changed lines of the file:
@@
 $Descr A3 16535 11693
 encoding utf-8
-Sheet 2 11
+Sheet 2 20
 Title ""
 Date ""
@@
 NoConn ~ 1900 7000
 NoConn ~ 1900 6900
-NoConn ~ 4350 6800
 Wire Wire Line
 	2400 5700 2550 5700
@@
 	1    0    0    1
 $EndComp
+$Sheet
+S 8250 10400 1800 550
+U 61054F55
+F0 "sheet61054F43" 50
+F1 "led16.sch" 50
+F2 "I0" I T 9800 10400 50
+F3 "I1" I T 9700 10400 50
+F4 "I2" I T 9600 10400 50
+F5 "I3" I T 9500 10400 50
+F6 "I4" I T 9400 10400 50
+F7 "I5" I T 9300 10400 50
+F8 "I6" I T 9200 10400 50
+F9 "I7" I T 9100 10400 50
+F10 "I8" I T 9000 10400 50
+F11 "I9" I T 8900 10400 50
+F12 "I10" I T 8800 10400 50
+F13 "I11" I T 8700 10400 50
+F14 "I12" I T 8600 10400 50
+F15 "I13" I T 8500 10400 50
+F16 "I14" I T 8400 10400 50
+F17 "I15" I T 8300 10400 50
+$EndSheet
+Wire Wire Line
+	8300 10200 8300 10400
+Connection ~ 8300 10200
+Wire Wire Line
+	8350 10000 8350 10350
+Wire Wire Line
+	8350 10350 8400 10350
+Wire Wire Line
+	8400 10350 8400 10400
+Connection ~ 8350 10000
+Wire Wire Line
+	8400 9850 8400 10300
+Wire Wire Line
+	8400 10300 8500 10300
+Wire Wire Line
+	8500 10300 8500 10400
+Connection ~ 8400 9850
+Wire Wire Line
+	8450 9650 8450 10250
+Wire Wire Line
+	8450 10250 8600 10250
+Wire Wire Line
+	8600 10250 8600 10400
+Connection ~ 8450 9650
+Wire Wire Line
+	8500 9500 8500 10200
+Wire Wire Line
+	8500 10200 8700 10200
+Wire Wire Line
+	8700 10200 8700 10400
+Connection ~ 8500 9500
+Wire Wire Line
+	8550 9300 8550 10150
+Wire Wire Line
+	8550 10150 8800 10150
+Wire Wire Line
+	8800 10150 8800 10400
+Connection ~ 8550 9300
+Wire Wire Line
+	8900 10400 8900 10100
+Wire Wire Line
+	8900 10100 8600 10100
+Wire Wire Line
+	8600 10100 8600 9150
+Connection ~ 8600 9150
+Wire Wire Line
+	8650 8950 8650 10050
+Wire Wire Line
+	8650 10050 9000 10050
+Wire Wire Line
+	9000 10050 9000 10400
+Connection ~ 8650 8950
+Wire Wire Line
+	9100 10400 9100 10000
+Wire Wire Line
+	9100 10000 8700 10000
+Wire Wire Line
+	8700 10000 8700 8800
+Connection ~ 8700 8800
+Wire Wire Line
+	8750 8600 8750 9950
+Wire Wire Line
+	8750 9950 9200 9950
+Wire Wire Line
+	9200 9950 9200 10400
+Connection ~ 8750 8600
+Wire Wire Line
+	9300 10400 9300 9900
+Wire Wire Line
+	9300 9900 8800 9900
+Wire Wire Line
+	8800 9900 8800 8450
+Connection ~ 8800 8450
+Wire Wire Line
+	8850 8250 8850 9850
+Wire Wire Line
+	8850 9850 9400 9850
+Wire Wire Line
+	9400 9850 9400 10400
+Connection ~ 8850 8250
+Wire Wire Line
+	9500 10400 9500 9800
+Wire Wire Line
+	9500 9800 8900 9800
+Wire Wire Line
+	8900 9800 8900 8100
+Connection ~ 8900 8100
+Wire Wire Line
+	8950 7900 8950 9750
+Wire Wire Line
+	8950 9750 9600 9750
+Wire Wire Line
+	9600 9750 9600 10400
+Connection ~ 8950 7900
+Wire Wire Line
+	9700 10400 9700 9700
+Wire Wire Line
+	9700 9700 9000 9700
+Wire Wire Line
+	9000 9700 9000 7750
+Connection ~ 9000 7750
+Wire Wire Line
+	9050 7550 9050 9650
+Wire Wire Line
+	9050 9650 9800 9650
+Wire Wire Line
+	9800 9650 9800 10400
+Connection ~ 9050 7550
 $EndSCHEMATC

Commit message: better alu :
Parts:
- removed unit 1 of U54
- removed unit 2 of U54
- removed unit 3 of U54
- removed unit 4 of U54
- removed U55: 74HC02, Package_DIP:DIP-14_W7.62mm, symbol 16bitCpu-rescue:74HC02-74xx
- removed U56, U57: 74LS08, Package_DIP:DIP-14_W7.62mm, symbol 16bitCpu-rescue:74LS08-74xx
- added U? (x4): 74LS85, symbol 74xx:74LS85
Connections:
- net +5V: now also U?.16 (VCC), U?.16 (VCC), U?.16 (VCC), U?.16 (VCC)
- net A0: now also U?.15 (A3)
- net A1: now also U?.13 (A2)
- net A10: now also U?.13 (A2)
- net A11: now also U?.15 (A3)
- net A12: now also U?.10 (A0)
- net A13: now also U?.12 (A1)
- net A14: now also U?.13 (A2)
- net A15: now also U?.15 (A3)
- net A2: now also U?.12 (A1)
- net A3: now also U?.10 (A0)
- net A4: now also U?.10 (A0)
- net A5: now also U?.12 (A1)
- net A6: now also U?.13 (A2)
- net A7: now also U?.15 (A3)
- net A8: now also U?.10 (A0)
- net A9: now also U?.12 (A1)
- net CF: now also U53.6 (Q3); no longer U53.3 (Q0)
- net GND: now also U?.8 (GND), U?.8 (GND), U?.8 (GND)
- net SU: no longer U3.7 (C0)
- net ZF: now also U53.5 (Q2); no longer U53.4 (Q1)
- net at U3.6 (B1), U7.3: now also U?.9 (B0)
- net at U3.2 (B2), U7.6: now also U?.11 (B1)
- net at U3.15 (B3), U7.8: now also U?.14 (B2)
- net at U3.11 (B4), U7.11: now also U?.1 (B3)
- net at U5.6 (B1), U8.3: now also U?.9 (B0)
- net at U5.2 (B2), U8.6: now also U?.11 (B1)
- net at U5.15 (B3), U8.8: now also U?.14 (B2)
- net at U5.11 (B4), U8.11: now also U?.1 (B3)
- net at U4.6 (B1), U9.3: now also U?.9 (B0)
- net at U4.2 (B2), U9.6: now also U?.11 (B1)
- net at U4.15 (B3), U9.8: now also U?.14 (B2)
- net at U4.11 (B4), U9.11: now also U?.1 (B3)
- net at U10.3, U6.6 (B1): now also U?.9 (B0)
- net at U10.6, U6.2 (B2): now also U?.11 (B1)
- net at U10.8, U6.15 (B3): now also U?.14 (B2)
- net at U10.11, U6.11 (B4): now also U?.1 (B3)
- net at U6.9 (C4): now also U53.11 (D3); no longer U53.14 (D0)
- net at U53.12 (D2): now also U?.6 (Oa=b)
- net at U53.13 (D1): now also U?.7 (Oa<b)
- new net: U53.14 (D0), U?.5 (Oa>b)
- new net: U?.5 (Oa>b), U?.5 (Oa>b)
- new net: U?.6 (Oa=b), U?.6 (Oa=b)
- new net: U?.7 (Oa<b), U?.7 (Oa<b)
- new net: U?.2 (Ia<b), U?.2 (Ia<b)
- new net: U?.3 (Ia=b), U?.3 (Ia=b)
- new net: U?.4 (Ia>b), U?.4 (Ia>b)
- new net: U?.4 (Ia>b), U?.5 (Oa>b)
- new net: U?.3 (Ia=b), U?.6 (Oa=b)
- new net: U?.2 (Ia<b), U?.7 (Oa<b)
- new net AGTBF: U53.3 (Q0)
- new net ALTBF: U53.4 (Q1)
- no-connect marks 4 -> 3
Other:
- moved on the sheet: U1, U10A, U10B, U10C, U10D, U10E, U2, U3, U4, U5, U53, U54E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

Commit message: Added NAND GATES in ALU
Parts:
- added D103, D104, D105, D106: LED, LED_THT:LED_D3.0mm, symbol Device:LED
- added R110, R111, R112, R113: 220, Resistor_THT:R_Axial_DIN0204_L3.6mm_D1.6mm_P7.62mm_Horizontal, symbol Device:R
- added U42, U62: 74LS245, Package_DIP:DIP-20_W7.62mm, symbol 16bitCpu-rescue:74LS245-74xx
- added U43, U47, U50, U51: 74LS00, Package_DIP:DIP-14_W7.62mm, symbol 74xx:74LS00
- U53, U56, U59, U63: renamed from U?; footprint (none) -> Package_DIP:DIP-16_W7.62mm
- renumbered U10 to U44, U9 to U45, U8 to U46, U7 to U48, U54 to U49, U3 to U52, U5 to U54, U1 to U55, U2 to U57, U4 to U58, U53 to U60, U6 to U61
Connections:
- net +5V: now also U42.1 (A->B), U42.20 (VCC), U43.7 (GND), U47.7 (GND), U50.7 (GND), U51.7 (GND), U62.1 (A->B), U62.20 (VCC)
- net A0: now also U50.1
- net A1: now also U48.3, U52.6 (B1), U53.9 (B0), U50.2, U50.4
- net A10: now also U43.9
- net A11: now also U43.12
- net A12: now also U47.1
- net A13: now also U47.4
- net A14: now also U47.9
- net A15: now also U47.12
- net A2: now also U50.9
- net A3: now also U46.6, U54.2 (B2), U56.11 (B1), U50.12, U51.5
- net A4: now also U51.1
- net A5: now also U51.4
- net A6: now also U51.9
- net A7: now also U51.12
- net A8: now also U43.1
- net A9: now also U43.4
- net AGTBF: now also D106.2 (A)
- net ALTBF: now also D105.2 (A)
- net BUS0: now also U62.18 (B0)
- net BUS1: now also U62.17 (B1)
- net BUS10: now also U42.16 (B2)
- net BUS11: now also U42.15 (B3)
- net BUS12: now also U42.14 (B4)
- net BUS13: now also U42.13 (B5)
- net BUS14: now also U42.12 (B6)
- net BUS15: now also U42.11 (B7)
- net BUS2: now also U62.16 (B2)
- net BUS3: now also U62.15 (B3)
- net BUS4: now also U62.14 (B4)
- net BUS5: now also U62.13 (B5)
- net BUS6: now also U62.12 (B6)
- net BUS7: now also U62.11 (B7)
- net BUS8: now also U42.18 (B0)
- net BUS9: now also U42.17 (B1)
- net CF: now also D103.2 (A)
- net GND: now also R110.2, R111.2, R112.2, R113.2, U42.10 (GND), U43.14 (VCC), U47.14 (VCC), U50.14 (VCC), U51.14 (VCC), U62.10 (GND)
- net ZF: now also D104.2 (A)
- net at U48.6, U52.2 (B2), U53.11 (B1): now also U50.5
- net at U48.8, U52.15 (B3), U53.14 (B2): now also U50.10
- net at U48.11, U52.11 (B4), U53.1 (B3): now also U50.13
- net at U46.3, U54.6 (B1), U56.9 (B0): now also U51.2
- net at U46.8, U54.15 (B3), U56.14 (B2): now also U51.10
- net at U46.11, U54.11 (B4), U56.1 (B3): now also U45.3, U58.6 (B1), U59.9 (B0), U43.2, U51.13
- net at U45.6, U58.2 (B2), U59.11 (B1): now also U43.5
- net at U45.8, U58.15 (B3), U59.14 (B2): now also U43.10
- net at U45.11, U58.11 (B4), U59.1 (B3): now also U43.13
- net at U44.3, U61.6 (B1), U63.9 (B0): now also U47.2
- net at U44.6, U61.2 (B2), U63.11 (B1): now also U47.5
- net at U44.8, U61.15 (B3), U63.14 (B2): now also U47.10
- net at U44.11, U61.11 (B4), U63.1 (B3): now also U47.13
- new net: D104.1 (K), R111.1
- new net: D105.1 (K), R112.1
- new net: D106.1 (K), R113.1
- new net: D103.1 (K), R110.1
- new net sheet67DDEE7E/I0: U50.3, U62.2 (A0)
- new net sheet67DDEE7E/I1: U50.6, U62.3 (A1)
- new net sheet67DDEE7E/I10: U42.4 (A2), U43.8
- new net sheet67DDEE7E/I11: U42.5 (A3), U43.11
- new net sheet67DDEE7E/I12: U42.6 (A4), U47.3
- new net sheet67DDEE7E/I13: U42.7 (A5), U47.6
- new net sheet67DDEE7E/I14: U42.8 (A6), U47.8
- new net sheet67DDEE7E/I15: U42.9 (A7), U47.11
- new net sheet67DDEE7E/I2: U50.8, U62.4 (A2)
- new net sheet67DDEE7E/I3: U50.11, U62.5 (A3)
- new net sheet67DDEE7E/I4: U51.3, U62.6 (A4)
- new net sheet67DDEE7E/I5: U51.6, U62.7 (A5)
- new net sheet67DDEE7E/I6: U51.8, U62.8 (A6)
- new net sheet67DDEE7E/I7: U51.11, U62.9 (A7)
- new net sheet67DDEE7E/I8: U42.2 (A0), U43.3
- new net sheet67DDEE7E/I9: U42.3 (A1), U43.6
- new net ~NAND: U42.19 (CE), U62.19 (CE)
Other:
- moved on the sheet: U44A, U44B, U44C, U44D, U44E, U45A, U45B, U45C, U45D, U45E, U46A, U46B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
