File: Control Unit.sch (KiCad schematic (older format))
At the start: 53 parts, among them SW1 SW_Push-Switch, U19 7400, U20 74LS161-74xx, U21 AT28C256, U22 AT28C256, U23 74LS138, U24 74LS138, U25 74LS138

Commit message: fixed almost all errors
Parts:
- removed D63: LED, LED_THT:LED_D3.0mm, symbol Device:LED
- removed R64: 220, Resistor_THT:R_Axial_DIN0204_L3.6mm_D1.6mm_P7.62mm_Horizontal, symbol Device:R
Connections:
- net ~ALU_EO: now also D61.2 (A), U24.13 (O2); no longer D62.2 (A), U24.12 (O3)
- net ~ALU_NAND_O: now also D62.2 (A), U24.12 (O3); no longer U24.11 (O4)
- net ~SO: no longer D61.2 (A), U24.13 (O2)
- no-connect marks 8 -> 17
Changed lines of the file:
@@
-$Comp
-L Device:LED D?
-U 1 1 625D64E8
-P 11600 10400
-AR Path="/5F926C74/625D64E8" Ref="D?"  Part="1"
-AR Path="/61968B9B/60C9B37A/625D64E8" Ref="D?"  Part="1"
-AR Path="/5F67C726/60E31E38/625D64E8" Ref="D?"  Part="1"
-AR Path="/5F74778C/60E31E38/625D64E8" Ref="D?"  Part="1"
-AR Path="/5F5F4A69/61054F55/625D64E8" Ref="D?"  Part="1"
-AR Path="/5F6ACD14/6156E9B6/625D64E8" Ref="D?"  Part="1"
-AR Path="/5F681977/6183038C/625D64E8" Ref="D?"  Part="1"
-AR Path="/5F681977/61B5B13E/625D64E8" Ref="D?"  Part="1"
-AR Path="/5F79B702/621E2556/625D64E8" Ref="D?"  Part="1"
-AR Path="/61DF6CC7/623AC6EB/625D64E8" Ref="D?"  Part="1"
-AR Path="/5FD099BF/625B6FDA/625D64E8" Ref="D?"  Part="1"
-AR Path="/5FD099BF/625D64E8" Ref="D63"  Part="1"
-F 0 "D63" V 11639 10282 50  0000 R CNN
-F 1 "LED" V 11548 10282 50  0000 R CNN
-F 2 "LED_THT:LED_D3.0mm" H 11600 10400 50  0001 C CNN
-F 3 "" H 11600 10400 50  0001 C CNN
-	1    11600 10400
-	0    -1   -1   0
-$EndComp
 $Comp
 L Device:LED D?
@@
 	11300 10550 11300 10700
 Wire Wire Line
-	11600 10550 11600 10700
-Wire Wire Line
 	11900 10550 11900 10700
 Wire Wire Line
@@
 $Comp
 L Device:R R?
-U 1 1 625D657C
-P 11600 10850
-AR Path="/5F926C74/625D657C" Ref="R?"  Part="1"
-AR Path="/61968B9B/60C9B37A/625D657C" Ref="R?"  Part="1"
-AR Path="/5F67C726/60E31E38/625D657C" Ref="R?"  Part="1"
-AR Path="/5F74778C/60E31E38/625D657C" Ref="R?"  Part="1"
-AR Path="/5F5F4A69/61054F55/625D657C" Ref="R?"  Part="1"
-AR Path="/5F6ACD14/6156E9B6/625D657C" Ref="R?"  Part="1"
-AR Path="/5F681977/6183038C/625D657C" Ref="R?"  Part="1"
-AR Path="/5F681977/61B5B13E/625D657C" Ref="R?"  Part="1"
-AR Path="/5F79B702/621E2556/625D657C" Ref="R?"  Part="1"
-AR Path="/61DF6CC7/623AC6EB/625D657C" Ref="R?"  Part="1"
-AR Path="/5FD099BF/625B6FDA/625D657C" Ref="R?"  Part="1"
-AR Path="/5FD099BF/625D657C" Ref="R64"  Part="1"
-F 0 "R64" H 11670 10896 50  0000 L CNN
-F 1 "220" H 11670 10805 50  0000 L CNN
-F 2 "Resistor_THT:R_Axial_DIN0204_L3.6mm_D1.6mm_P7.62mm_Horizontal" V 11530 10850 50  0001 C CNN
-F 3 "" H 11600 10850 50  0001 C CNN
-	1    11600 10850
-	1    0    0    -1
-$EndComp
-$Comp
-L Device:R R?
 U 1 1 625D6582
 P 11900 10850
@@
 	11000 11000 11300 11000
 Connection ~ 11300 11000
-Wire Wire Line
-	11300 11000 11600 11000
-Connection ~ 11600 11000
-Wire Wire Line
-	11600 11000 11900 11000
 Connection ~ 12200 11000
 Wire Wire Line
@@
 	1    0    0    -1
 $EndComp
-Text HLabel 13600 4800 2    50   Output ~ 0
-~SO
 Text HLabel 13600 7400 2    50   Output ~ 0
 ~SI
@@
 Wire Wire Line
 	12300 4900 12850 4900
-Text HLabel 13600 4900 2    50   Output ~ 0
+Text HLabel 13600 4800 2    50   Output ~ 0
 ~ALU_EO
 Text HLabel 8450 3300 2    50   Output ~ 0
 ALU_SU
-Wire Wire Line
-	13600 4800 12800 4800
 Wire Wire Line
 	11300 3200 11300 3300
@@
 	11150 3100 11300 3100
 Connection ~ 11800 2300
-Wire Wire Line
-	12300 5000 12900 5000
-Text HLabel 13600 5000 2    50   Output ~ 0
+Text HLabel 13600 4900 2    50   Output ~ 0
 ~ALU_NAND_O
 $Comp
@@
 Wire Wire Line
 	12800 8600 12800 4800
-Connection ~ 12800 4800
 Wire Wire Line
 	12800 4800 12300 4800
@@
 Wire Wire Line
 	12850 8650 12850 4900
-Connection ~ 12850 4900
-Wire Wire Line
-	12850 4900 13600 4900
-Wire Wire Line
-	11600 10250 11600 8700
-Wire Wire Line
-	11600 8700 12900 8700
-Wire Wire Line
-	12900 8700 12900 5000
-Connection ~ 12900 5000
-Wire Wire Line
-	12900 5000 13600 5000
 Wire Wire Line
 	11900 10250 11900 8750
@@
 Wire Wire Line
 	2500 4900 4150 4900
+Wire Wire Line
+	12850 4900 13600 4900
+Connection ~ 12850 4900
+Wire Wire Line
+	12800 4800 13600 4800
+Connection ~ 12800 4800
+Wire Wire Line
+	11300 11000 11900 11000
+NoConn ~ 12300 6700
+NoConn ~ 12300 5300
+NoConn ~ 12300 5200
+NoConn ~ 12300 5100
+NoConn ~ 12300 5000
+NoConn ~ 12300 4600
+NoConn ~ 7150 5550
+NoConn ~ 7150 5450
+NoConn ~ 4050 2050
 $EndSCHEMATC
