File: stack.sch (KiCad schematic (older format))
At the start: 6 parts, among them U11 74LS245, U12 74LS173, U13 74LS173, U14 74LS245, U15 74LS173, U16 74LS173

Commit message: back to 13 bit addresses
Changed lines of the file:
@@
 Wire Wire Line
 	2300 5700 3800 5700
-Wire Wire Line
-	9450 5350 9550 5350
-Wire Wire Line
-	9550 4800 9550 5350
-Wire Wire Line
-	9450 4800 9450 5350
-Wire Wire Line
-	9650 5350 9550 5350
-Wire Wire Line
-	9650 4800 9650 5350
-Connection ~ 9550 5350
-Wire Wire Line
-	9550 5350 9550 5500
 $Comp
 L 16bitCpu-rescue:GND-power #PWR0211
@@
 	1    0    0    -1
 $EndComp
+Wire Wire Line
+	9550 5350 9550 5500
+Wire Wire Line
+	9450 4800 9450 5350
+Connection ~ 9550 5350
+Wire Wire Line
+	9550 4800 9550 5350
+Wire Wire Line
+	9450 5350 9550 5350
+Wire Wire Line
+	6600 5000 9650 5000
+Wire Wire Line
+	9650 5000 9650 4800
 $EndSCHEMATC

Commit message: Let there be light
Connections:
- wire segments 203 -> 250
- no-connect marks 0 -> 2
Changed lines of the file:
@@
 $Descr A3 16535 11693
 encoding utf-8
-Sheet 10 11
+Sheet 10 20
 Title ""
 Date ""
@@
 Wire Wire Line
 	6200 6800 6200 4800
-Wire Wire Line
-	6300 4800 6300 6650
 Wire Wire Line
 	8000 6650 8000 6150
@@
 	6400 6500 7900 6500
 Wire Wire Line
-	2700 4100 5350 4100
-Wire Wire Line
 	2600 4150 5450 4150
 Wire Wire Line
@@
 Wire Wire Line
 	9650 5000 9650 4800
+NoConn ~ 6700 4950
+NoConn ~ 6800 4900
+$Sheet
+S 4300 9100 1800 550
+U 60C9B37A
+F0 "sheet60C9B368" 50
+F1 "led16.sch" 50
+F2 "I0" I T 4550 9100 50
+F3 "I1" I T 4650 9100 50
+F4 "I2" I T 4750 9100 50
+F5 "I3" I T 4850 9100 50
+F6 "I4" I T 4950 9100 50
+F7 "I5" I T 5050 9100 50
+F8 "I6" I T 5150 9100 50
+F9 "I7" I T 5250 9100 50
+F10 "I8" I T 5350 9100 50
+F11 "I9" I T 5450 9100 50
+F12 "I10" I T 5550 9100 50
+F13 "I11" I T 5650 9100 50
+F14 "I12" I T 5750 9100 50
+F15 "I13" I T 5850 9100 50
+F16 "I14" I T 5950 9100 50
+F17 "I15" I T 6050 9100 50
+$EndSheet
+Wire Wire Line
+	2000 6100 2000 8750
+Wire Wire Line
+	2000 8750 4550 8750
+Wire Wire Line
+	4550 8750 4550 9100
+Connection ~ 2000 6100
+Wire Wire Line
+	2100 6000 2100 8700
+Wire Wire Line
+	2100 8700 4650 8700
+Wire Wire Line
+	4650 8700 4650 9100
+Connection ~ 2100 6000
+Wire Wire Line
+	2200 5850 2200 8500
+Wire Wire Line
+	2200 8500 4750 8500
+Wire Wire Line
+	4750 8500 4750 9100
+Connection ~ 2200 5850
+Wire Wire Line
+	2300 5700 2300 8400
+Wire Wire Line
+	2300 8400 4850 8400
+Wire Wire Line
+	4850 8400 4850 9100
+Connection ~ 2300 5700
+Wire Wire Line
+	5650 4250 5650 8400
+Wire Wire Line
+	5650 8400 4950 8400
+Wire Wire Line
+	4950 8400 4950 9100
+Connection ~ 5650 4250
+Wire Wire Line
+	5550 4200 5550 8500
+Wire Wire Line
+	5550 8500 5050 8500
+Wire Wire Line
+	5050 8500 5050 9100
+Connection ~ 5550 4200
+Wire Wire Line
+	5450 4150 5450 8700
+Wire Wire Line
+	5450 8700 5150 8700
+Wire Wire Line
+	5150 8700 5150 9100
+Connection ~ 5450 4150
+Wire Wire Line
+	2700 4100 5350 4100
+Wire Wire Line
+	5250 9100 5250 8800
+Wire Wire Line
+	5250 8800 5350 8800
+Wire Wire Line
+	5350 8800 5350 4100
+Connection ~ 5350 4100
+Wire Wire Line
+	6100 6900 6100 8900
+Wire Wire Line
+	6100 8900 5350 8900
+Wire Wire Line
+	5350 8900 5350 9100
+Connection ~ 6100 6900
+Wire Wire Line
+	6200 6800 6200 9000
+Wire Wire Line
+	6200 9000 5450 9000
+Wire Wire Line
+	5450 9000 5450 9100
+Connection ~ 6200 6800
+Wire Wire Line
+	6300 8800 5550 8800
+Wire Wire Line
+	5550 8800 5550 9100
+Wire Wire Line
+	6300 4800 6300 6650
+Connection ~ 6300 6650
+Wire Wire Line
+	6300 6650 6300 8800
+Wire Wire Line
+	6400 6500 6400 8700
+Wire Wire Line
+	6400 8700 5650 8700
+Wire Wire Line
+	5650 8700 5650 9100
+Connection ~ 6400 6500
+Wire Wire Line
+	5750 9100 5750 8500
+Wire Wire Line
+	5750 8500 9750 8500
+Wire Wire Line
+	9750 8500 9750 5050
+Connection ~ 9750 5050
+Wire Wire Line
+	9650 5000 9650 8400
+Wire Wire Line
+	9650 8400 5850 8400
+Wire Wire Line
+	5850 8400 5850 9100
+Connection ~ 9650 5000
+Wire Wire Line
+	9450 5350 9450 8300
+Wire Wire Line
+	9450 8300 6050 8300
+Wire Wire Line
+	5950 8300 5950 9100
+Connection ~ 9450 5350
+Wire Wire Line
+	6050 8300 6050 9100
+Connection ~ 6050 8300
+Wire Wire Line
+	6050 8300 5950 8300
 $EndSCHEMATC

Commit message: Added NAND GATES in ALU
Parts:
- renumbered U11 to U24, U12 to U25, U13 to U26, U14 to U27, U15 to U28, U16 to U29

Commit message: using new RAM and ROM,15bits baby
Parts:
- renumbered U24 to U27, U25 to U28, U26 to U29, U27 to U30, U28 to U31, U29 to U32
Connections:
- net labels removed: GND-power
- wire segments 250 -> 251
- no-connect marks 2 -> 0

Commit message: using new ROM in CU and more jumps
Parts:
- renumbered U27 to U26, U28 to U27, U29 to U28, U30 to U29, U31 to U30, U32 to U31
Changed lines of the file:
@@
 AR Path="/5F74778C/616C378C" Ref="U?"  Part="1"
 AR Path="/5FB94562/616C378C" Ref="U?"  Part="1"
-AR Path="/61968B9B/616C378C" Ref="U28"  Part="1"
-F 0 "U28" H 3500 5931 50  0000 C CNN
+AR Path="/61968B9B/616C378C" Ref="U27"  Part="1"
+F 0 "U27" H 3500 5931 50  0000 C CNN
 F 1 "74LS173" H 3500 5840 50  0000 C CNN
 F 2 "Package_DIP:DIP-16_W7.62mm" H 3500 4850 50  0001 C CNN
@@
 AR Path="/5F74778C/616C378D" Ref="U?"  Part="1"
 AR Path="/5FB94562/616C378D" Ref="U?"  Part="1"
-AR Path="/61968B9B/616C378D" Ref="U27"  Part="1"
-F 0 "U27" V 2546 2656 50  0000 R CNN
+AR Path="/61968B9B/616C378D" Ref="U26"  Part="1"
+F 0 "U26" V 2546 2656 50  0000 R CNN
 F 1 "74LS245" V 2455 2656 50  0000 R CNN
 F 2 "Package_DIP:DIP-20_W7.62mm" H 2500 3500 50  0001 C CNN
@@
 AR Path="/5F74778C/5F73559F" Ref="U?"  Part="1"
 AR Path="/5FB94562/5F73559F" Ref="U?"  Part="1"
-AR Path="/61968B9B/5F73559F" Ref="U32"  Part="1"
-F 0 "U32" V 9104 5244 50  0000 L CNN
+AR Path="/61968B9B/5F73559F" Ref="U31"  Part="1"
+F 0 "U31" V 9104 5244 50  0000 L CNN
 F 1 "74LS173" V 9195 5244 50  0000 L CNN
 F 2 "Package_DIP:DIP-16_W7.62mm" H 9150 4300 50  0001 C CNN
@@
 AR Path="/5F74778C/62492011" Ref="U?"  Part="1"
 AR Path="/5FB94562/62492011" Ref="U?"  Part="1"
-AR Path="/61968B9B/62492011" Ref="U31"  Part="1"
-F 0 "U31" V 7554 6594 50  0000 L CNN
+AR Path="/61968B9B/62492011" Ref="U30"  Part="1"
+F 0 "U30" V 7554 6594 50  0000 L CNN
 F 1 "74LS173" V 7645 6594 50  0000 L CNN
 F 2 "Package_DIP:DIP-16_W7.62mm" H 7600 5650 50  0001 C CNN
@@
 AR Path="/5F74778C/616C379D" Ref="U?"  Part="1"
 AR Path="/5FB94562/616C379D" Ref="U?"  Part="1"
-AR Path="/61968B9B/616C379D" Ref="U29"  Part="1"
-F 0 "U29" V 5004 4444 50  0000 L CNN
+AR Path="/61968B9B/616C379D" Ref="U28"  Part="1"
+F 0 "U28" V 5004 4444 50  0000 L CNN
 F 1 "74LS173" V 5095 4444 50  0000 L CNN
 F 2 "Package_DIP:DIP-16_W7.62mm" H 5050 3500 50  0001 C CNN
@@
 AR Path="/5F74778C/616C379F" Ref="U?"  Part="1"
 AR Path="/5FB94562/616C379F" Ref="U?"  Part="1"
-AR Path="/61968B9B/616C379F" Ref="U30"  Part="1"
-F 0 "U30" V 6646 3456 50  0000 R CNN
+AR Path="/61968B9B/616C379F" Ref="U29"  Part="1"
+F 0 "U29" V 6646 3456 50  0000 R CNN
 F 1 "74LS245" V 6555 3456 50  0000 R CNN
 F 2 "Package_DIP:DIP-20_W7.62mm" H 6600 4300 50  0001 C CNN

Commit message: fixed more errors
Changed lines of the file:
@@
-$Comp
-L 16bitCpu-rescue:+5V-power #PWR?
-U 1 1 616C3797
-P 5800 4300
-AR Path="/616C3797" Ref="#PWR?"  Part="1"
-AR Path="/5F67C726/616C3797" Ref="#PWR?"  Part="1"
-AR Path="/5F70885A/616C3797" Ref="#PWR?"  Part="1"
-AR Path="/5F733C5E/616C3797" Ref="#PWR?"  Part="1"
-AR Path="/602D4838/616C3797" Ref="#PWR?"  Part="1"
-AR Path="/603B00C8/616C3797" Ref="#PWR?"  Part="1"
-AR Path="/603B766D/616C3797" Ref="#PWR?"  Part="1"
-AR Path="/5F74778C/616C3797" Ref="#PWR?"  Part="1"
-AR Path="/5FB94562/616C3797" Ref="#PWR?"  Part="1"
-AR Path="/61968B9B/616C3797" Ref="#PWR0110"  Part="1"
-F 0 "#PWR0110" H 5800 4150 50  0001 C CNN
-F 1 "+5V" H 5815 4473 50  0000 C CNN
-F 2 "" H 5800 4300 50  0001 C CNN
-F 3 "" H 5800 4300 50  0001 C CNN
-	1    5800 4300
-	1    0    0    -1
-$EndComp
 $Comp
 L 16bitCpu-rescue:+5V-power #PWR?
@@
 	1    0    0    -1
 $EndComp
-$Comp
-L 16bitCpu-rescue:+5V-power #PWR?
-U 1 1 616C379A
-P 5950 3500
-AR Path="/616C379A" Ref="#PWR?"  Part="1"
-AR Path="/5F67C726/616C379A" Ref="#PWR?"  Part="1"
-AR Path="/5F70885A/616C379A" Ref="#PWR?"  Part="1"
-AR Path="/5F733C5E/616C379A" Ref="#PWR?"  Part="1"
-AR Path="/602D4838/616C379A" Ref="#PWR?"  Part="1"
-AR Path="/603B00C8/616C379A" Ref="#PWR?"  Part="1"
-AR Path="/603B766D/616C379A" Ref="#PWR?"  Part="1"
-AR Path="/5F74778C/616C379A" Ref="#PWR?"  Part="1"
-AR Path="/5FB94562/616C379A" Ref="#PWR?"  Part="1"
-AR Path="/61968B9B/616C379A" Ref="#PWR0111"  Part="1"
-F 0 "#PWR0111" H 5950 3350 50  0001 C CNN
-F 1 "+5V" H 5965 3673 50  0000 C CNN
-F 2 "" H 5950 3500 50  0001 C CNN
-F 3 "" H 5950 3500 50  0001 C CNN
-	1    5950 3500
-	1    0    0    -1
-$EndComp
