File: resgister.sch (KiCad schematic (older format))
At the start: 6 parts, among them U11 74LS245, U12 74LS173, U13 74LS173, U14 74LS245, U15 74LS173, U16 74LS173

Commit message: Let there be light
Connections:
- wire segments 234 -> 277
Changed lines of the file:
@@
 $Descr A3 16535 11693
 encoding utf-8
-Sheet 4 11
+Sheet 6 20
 Title ""
 Date ""
@@
 	3250 6100 4100 6100
 Wire Wire Line
-	3350 7500 3350 6000
+	3350 7500 3350 6200
 Connection ~ 3350 6000
 Wire Wire Line
 	3350 6000 2100 6000
 Wire Wire Line
-	3450 7500 3450 5850
+	3450 7500 3450 6300
 Connection ~ 3450 5850
 Wire Wire Line
 	3450 5850 3900 5850
 Wire Wire Line
-	3550 7500 3550 5700
+	3550 7500 3550 6400
 Wire Wire Line
 	2300 5700 3550 5700
@@
 Wire Wire Line
 	3550 5700 3800 5700
-Wire Wire Line
-	5250 7500 5250 4100
 Connection ~ 5250 4100
 Wire Wire Line
@@
 	5150 4150 5450 4150
 Wire Wire Line
-	5150 7500 5150 4150
+	5150 7500 5150 6850
 Wire Wire Line
 	2500 4200 5050 4200
@@
 	5050 4200 5550 4200
 Wire Wire Line
-	4950 7500 4950 4250
+	4950 7500 4950 6550
 Wire Wire Line
 	2400 4250 4950 4250
 Connection ~ 4950 4250
 Wire Wire Line
-	5050 4200 5050 7500
+	5050 4200 5050 6600
 Wire Wire Line
 	4950 4250 5650 4250
 Wire Wire Line
 	6200 6800 7600 6800
-Wire Wire Line
-	7500 7500 7500 6900
 Connection ~ 7500 6900
 Wire Wire Line
 	7500 6900 8200 6900
 Wire Wire Line
-	7600 7500 7600 6800
+	7600 7500 7600 7050
 Connection ~ 7600 6800
 Wire Wire Line
 	7600 6800 8100 6800
-Wire Wire Line
-	7700 7500 7700 6650
 Wire Wire Line
 	6300 6650 7700 6650
@@
 	7700 6650 8000 6650
 Wire Wire Line
-	7800 7500 7800 6500
+	7800 7500 7800 7200
 Wire Wire Line
 	6400 6500 7800 6500
@@
 	6500 5050 9150 5050
 Wire Wire Line
-	9150 7500 9150 5050
+	9150 7500 9150 7300
 Connection ~ 9150 5050
 Wire Wire Line
 	9150 5050 9750 5050
 Wire Wire Line
-	9250 7500 9250 5000
+	9250 7500 9250 7400
 Connection ~ 9250 5000
 Wire Wire Line
 	9250 5000 9650 5000
 Wire Wire Line
-	9350 7500 9350 4950
+	9350 7500 9350 7450
 Connection ~ 9350 4950
 Wire Wire Line
 	9350 4950 6700 4950
 Wire Wire Line
-	9450 7500 9450 4900
+	9450 7500 9450 7350
 Connection ~ 9450 4900
 $Comp
@@
 Text HLabel 1300 2350 0    50   3State ~ 0
 Bus15
+$Sheet
+S 10800 5850 550  1800
+U 60E31E38
+F0 "sheet60E31E26" 50
+F1 "led16.sch" 50
+F2 "I0" I L 10800 6100 50
+F3 "I1" I L 10800 6200 50
+F4 "I2" I L 10800 6300 50
+F5 "I3" I L 10800 6400 50
+F6 "I4" I L 10800 6500 50
+F7 "I5" I L 10800 6600 50
+F8 "I6" I L 10800 6700 50
+F9 "I7" I L 10800 6800 50
+F10 "I8" I L 10800 6900 50
+F11 "I9" I L 10800 7000 50
+F12 "I10" I L 10800 7100 50
+F13 "I11" I L 10800 7200 50
+F14 "I12" I L 10800 7300 50
+F15 "I13" I L 10800 7400 50
+F16 "I14" I L 10800 7500 50
+F17 "I15" I L 10800 7600 50
+$EndSheet
+Wire Wire Line
+	4100 6100 10800 6100
+Connection ~ 4100 6100
+Wire Wire Line
+	10800 6200 3350 6200
+Connection ~ 3350 6200
+Wire Wire Line
+	3350 6200 3350 6000
+Connection ~ 3450 6300
+Wire Wire Line
+	3450 6300 3450 5850
+Wire Wire Line
+	3450 6300 10800 6300
+Wire Wire Line
+	10800 6400 3550 6400
+Connection ~ 3550 6400
+Wire Wire Line
+	3550 6400 3550 5700
+Wire Wire Line
+	4950 6550 10650 6550
+Wire Wire Line
+	10650 6550 10650 6500
+Wire Wire Line
+	10650 6500 10800 6500
+Connection ~ 4950 6550
+Wire Wire Line
+	4950 6550 4950 4250
+Wire Wire Line
+	5050 6600 10800 6600
+Connection ~ 5050 6600
+Wire Wire Line
+	5050 6600 5050 7500
+Wire Wire Line
+	5150 6700 10800 6700
+Connection ~ 5150 6700
+Wire Wire Line
+	5150 6700 5150 4150
+Wire Wire Line
+	5250 7500 5250 4100
+Wire Wire Line
+	5150 6850 10550 6850
+Wire Wire Line
+	10550 6850 10550 6800
+Wire Wire Line
+	10550 6800 10800 6800
+Connection ~ 5150 6850
+Wire Wire Line
+	5150 6850 5150 6700
+Wire Wire Line
+	7500 7500 7500 7000
+Wire Wire Line
+	7500 7000 10600 7000
+Wire Wire Line
+	10600 7000 10600 6900
+Wire Wire Line
+	10600 6900 10800 6900
+Connection ~ 7500 7000
+Wire Wire Line
+	7500 7000 7500 6900
+Wire Wire Line
+	10800 7000 10650 7000
+Wire Wire Line
+	10650 7000 10650 7050
+Wire Wire Line
+	10650 7050 7600 7050
+Connection ~ 7600 7050
+Wire Wire Line
+	7600 7050 7600 6800
+Wire Wire Line
+	7700 7100 10800 7100
+Connection ~ 7700 7100
+Wire Wire Line
+	7700 7100 7700 6650
+Wire Wire Line
+	7700 7500 7700 7100
+Wire Wire Line
+	10800 7200 7800 7200
+Connection ~ 7800 7200
+Wire Wire Line
+	7800 7200 7800 6500
+Wire Wire Line
+	9150 7300 10800 7300
+Connection ~ 9150 7300
+Wire Wire Line
+	9150 7300 9150 5050
+Wire Wire Line
+	9250 7400 10800 7400
+Connection ~ 9250 7400
+Wire Wire Line
+	9250 7400 9250 5000
+Wire Wire Line
+	9350 7450 10650 7450
+Wire Wire Line
+	10650 7450 10650 7500
+Wire Wire Line
+	10650 7500 10800 7500
+Connection ~ 9350 7450
+Wire Wire Line
+	9350 7450 9350 4950
+Wire Wire Line
+	9450 7350 10600 7350
+Wire Wire Line
+	10600 7350 10600 7600
+Wire Wire Line
+	10600 7600 10800 7600
+Connection ~ 9450 7350
+Wire Wire Line
+	9450 7350 9450 4900
 $EndSCHEMATC

Commit message: Fixes
Changed lines of the file:
@@
 	5150 4150 5450 4150
-Wire Wire Line
-	5150 7500 5150 6850
 Wire Wire Line
 	2500 4200 5050 4200
@@
 	5150 6700 5150 4150
 Wire Wire Line
-	5250 7500 5250 4100
-Wire Wire Line
-	5150 6850 10550 6850
+	5250 7500 5250 6850
 Wire Wire Line
 	10550 6850 10550 6800
 Wire Wire Line
 	10550 6800 10800 6800
-Connection ~ 5150 6850
-Wire Wire Line
-	5150 6850 5150 6700
 Wire Wire Line
 	7500 7500 7500 7000
@@
 Wire Wire Line
 	9450 7350 9450 4900
+Wire Wire Line
+	5150 6700 5150 7500
+Connection ~ 5250 6850
+Wire Wire Line
+	5250 6850 5250 4100
+Wire Wire Line
+	5250 6850 10550 6850
 $EndSCHEMATC

Commit message: Added NAND GATES in ALU
Parts:
- renumbered U11 to U1, U12 to U2, U13 to U3, U14 to U4, U15 to U5, U16 to U6

Commit message: fixed almost all errors
Changed lines of the file:
@@
 $Descr A3 16535 11693
 encoding utf-8
-Sheet 4 21
+Sheet 2 21
 Title ""
 Date ""
@@
 AR Path="/5FB94562/5F6AAB55" Ref="U?"  Part="1"
 AR Path="/616D5CDC/5F6AAB55" Ref="U?"  Part="1"
-F 0 "U8" H 3500 5931 50  0000 C CNN
+F 0 "U2" H 3500 5931 50  0000 C CNN
 F 1 "74LS173" H 3500 5840 50  0000 C CNN
 F 2 "Package_DIP:DIP-16_W7.62mm" H 3500 4850 50  0001 C CNN
@@
 AR Path="/5FB94562/5F6AAB61" Ref="U?"  Part="1"
 AR Path="/616D5CDC/5F6AAB61" Ref="U?"  Part="1"
-F 0 "U7" V 2546 2656 50  0000 R CNN
+F 0 "U1" V 2546 2656 50  0000 R CNN
 F 1 "74LS245" V 2455 2656 50  0000 R CNN
 F 2 "Package_DIP:DIP-20_W7.62mm" H 2500 3500 50  0001 C CNN
@@
 AR Path="/5FB94562/616C379E" Ref="U?"  Part="1"
 AR Path="/616D5CDC/616C379E" Ref="U?"  Part="1"
-F 0 "U12" V 9104 5244 50  0000 L CNN
+F 0 "U6" V 9104 5244 50  0000 L CNN
 F 1 "74LS173" V 9195 5244 50  0000 L CNN
 F 2 "Package_DIP:DIP-16_W7.62mm" H 9150 4300 50  0001 C CNN
@@
 AR Path="/5FB94562/61968D33" Ref="U?"  Part="1"
 AR Path="/616D5CDC/61968D33" Ref="U?"  Part="1"
-F 0 "U11" V 7554 6594 50  0000 L CNN
+F 0 "U5" V 7554 6594 50  0000 L CNN
 F 1 "74LS173" V 7645 6594 50  0000 L CNN
 F 2 "Package_DIP:DIP-16_W7.62mm" H 7600 5650 50  0001 C CNN
@@
 AR Path="/5FB94562/5F73559C" Ref="U?"  Part="1"
 AR Path="/616D5CDC/5F73559C" Ref="U?"  Part="1"
-F 0 "U9" V 5004 4444 50  0000 L CNN
+F 0 "U3" V 5004 4444 50  0000 L CNN
 F 1 "74LS173" V 5095 4444 50  0000 L CNN
 F 2 "Package_DIP:DIP-16_W7.62mm" H 5050 3500 50  0001 C CNN
@@
 AR Path="/5FB94562/62492020" Ref="U?"  Part="1"
 AR Path="/616D5CDC/62492020" Ref="U?"  Part="1"
-F 0 "U10" V 6646 3456 50  0000 R CNN
+F 0 "U4" V 6646 3456 50  0000 R CNN
 F 1 "74LS245" V 6555 3456 50  0000 R CNN
 F 2 "Package_DIP:DIP-20_W7.62mm" H 6600 4300 50  0001 C CNN

Commit message: fixed more errors
Changed lines of the file:
@@
-$Comp
-L 16bitCpu-rescue:GND-power #PWR?
-U 1 1 61968D2B
-P 7400 4300
-AR Path="/61968D2B" Ref="#PWR?"  Part="1"
-AR Path="/5F67C726/61968D2B" Ref="#PWR026"  Part="1"
-AR Path="/5F70885A/61968D2B" Ref="#PWR?"  Part="1"
-AR Path="/5F733C5E/61968D2B" Ref="#PWR?"  Part="1"
-AR Path="/602D4838/61968D2B" Ref="#PWR?"  Part="1"
-AR Path="/603B00C8/61968D2B" Ref="#PWR?"  Part="1"
-AR Path="/603B766D/61968D2B" Ref="#PWR?"  Part="1"
-AR Path="/5F74778C/61968D2B" Ref="#PWR055"  Part="1"
-AR Path="/5FB94562/61968D2B" Ref="#PWR?"  Part="1"
-AR Path="/616D5CDC/61968D2B" Ref="#PWR?"  Part="1"
-F 0 "#PWR055" H 7400 4050 50  0001 C CNN
-F 1 "GND" H 7405 4127 50  0000 C CNN
-F 2 "" H 7400 4300 50  0001 C CNN
-F 3 "" H 7400 4300 50  0001 C CNN
-	1    7400 4300
-	1    0    0    -1
-$EndComp
-$Comp
-L 16bitCpu-rescue:GND-power #PWR?
-U 1 1 61968D2C
-P 8250 4300
-AR Path="/61968D2C" Ref="#PWR?"  Part="1"
-AR Path="/5F67C726/61968D2C" Ref="#PWR031"  Part="1"
-AR Path="/5F70885A/61968D2C" Ref="#PWR?"  Part="1"
-AR Path="/5F733C5E/61968D2C" Ref="#PWR?"  Part="1"
-AR Path="/602D4838/61968D2C" Ref="#PWR?"  Part="1"
-AR Path="/603B00C8/61968D2C" Ref="#PWR?"  Part="1"
-AR Path="/603B766D/61968D2C" Ref="#PWR?"  Part="1"
-AR Path="/5F74778C/61968D2C" Ref="#PWR060"  Part="1"
-AR Path="/5FB94562/61968D2C" Ref="#PWR?"  Part="1"
-AR Path="/616D5CDC/61968D2C" Ref="#PWR?"  Part="1"
-F 0 "#PWR060" H 8250 4050 50  0001 C CNN
-F 1 "GND" H 8255 4127 50  0000 C CNN
-F 2 "" H 8250 4300 50  0001 C CNN
-F 3 "" H 8250 4300 50  0001 C CNN
-	1    8250 4300
-	1    0    0    -1
-$EndComp
-$Comp
-L 16bitCpu-rescue:GND-power #PWR?
-U 1 1 5F7355A3
-P 6700 5650
-AR Path="/5F7355A3" Ref="#PWR?"  Part="1"
-AR Path="/5F67C726/5F7355A3" Ref="#PWR024"  Part="1"
-AR Path="/5F70885A/5F7355A3" Ref="#PWR?"  Part="1"
-AR Path="/5F733C5E/5F7355A3" Ref="#PWR?"  Part="1"
-AR Path="/602D4838/5F7355A3" Ref="#PWR?"  Part="1"
-AR Path="/603B00C8/5F7355A3" Ref="#PWR?"  Part="1"
-AR Path="/603B766D/5F7355A3" Ref="#PWR?"  Part="1"
-AR Path="/5F74778C/5F7355A3" Ref="#PWR053"  Part="1"
-AR Path="/5FB94562/5F7355A3" Ref="#PWR?"  Part="1"
-AR Path="/616D5CDC/5F7355A3" Ref="#PWR?"  Part="1"
-F 0 "#PWR053" H 6700 5400 50  0001 C CNN
-F 1 "GND" H 6705 5477 50  0000 C CNN
-F 2 "" H 6700 5650 50  0001 C CNN
-F 3 "" H 6700 5650 50  0001 C CNN
-	1    6700 5650
-	1    0    0    -1
-$EndComp
 $Comp
 L 16bitCpu-rescue:GND-power #PWR?
@@
 	9150 3800 9250 3800
 Connection ~ 9250 3800
-$Comp
-L 16bitCpu-rescue:GND-power #PWR?
-U 1 1 6249201D
-P 7800 3650
-AR Path="/6249201D" Ref="#PWR?"  Part="1"
-AR Path="/5F67C726/6249201D" Ref="#PWR029"  Part="1"
-AR Path="/5F70885A/6249201D" Ref="#PWR?"  Part="1"
-AR Path="/5F733C5E/6249201D" Ref="#PWR?"  Part="1"
-AR Path="/602D4838/6249201D" Ref="#PWR?"  Part="1"
-AR Path="/603B00C8/6249201D" Ref="#PWR?"  Part="1"
-AR Path="/603B766D/6249201D" Ref="#PWR?"  Part="1"
-AR Path="/5F74778C/6249201D" Ref="#PWR058"  Part="1"
-AR Path="/5FB94562/6249201D" Ref="#PWR?"  Part="1"
-AR Path="/616D5CDC/6249201D" Ref="#PWR?"  Part="1"
-F 0 "#PWR058" H 7800 3400 50  0001 C CNN
-F 1 "GND" H 7805 3477 50  0000 C CNN
-F 2 "" H 7800 3650 50  0001 C CNN
-F 3 "" H 7800 3650 50  0001 C CNN
-	1    7800 3650
-	1    0    0    -1
-$EndComp
 Connection ~ 7800 3650
 Wire Wire Line
@@
 $Comp
 L 16bitCpu-rescue:GND-power #PWR?
-U 1 1 61968D2E
-P 2600 4850
-AR Path="/61968D2E" Ref="#PWR?"  Part="1"
-AR Path="/5F67C726/61968D2E" Ref="#PWR010"  Part="1"
-AR Path="/5F70885A/61968D2E" Ref="#PWR?"  Part="1"
-AR Path="/5F733C5E/61968D2E" Ref="#PWR?"  Part="1"
-AR Path="/602D4838/61968D2E" Ref="#PWR?"  Part="1"
-AR Path="/603B00C8/61968D2E" Ref="#PWR?"  Part="1"
-AR Path="/603B766D/61968D2E" Ref="#PWR?"  Part="1"
-AR Path="/5F74778C/61968D2E" Ref="#PWR039"  Part="1"
-AR Path="/5FB94562/61968D2E" Ref="#PWR?"  Part="1"
-AR Path="/616D5CDC/61968D2E" Ref="#PWR?"  Part="1"
-F 0 "#PWR039" H 2600 4600 50  0001 C CNN
-F 1 "GND" H 2605 4677 50  0000 C CNN
-F 2 "" H 2600 4850 50  0001 C CNN
-F 3 "" H 2600 4850 50  0001 C CNN
-	1    2600 4850
-	1    0    0    -1
-$EndComp
-$Comp
-L 16bitCpu-rescue:GND-power #PWR?
-U 1 1 61968D3B
-P 3300 3500
-AR Path="/61968D3B" Ref="#PWR?"  Part="1"
-AR Path="/5F67C726/61968D3B" Ref="#PWR013"  Part="1"
-AR Path="/5F70885A/61968D3B" Ref="#PWR?"  Part="1"
-AR Path="/5F733C5E/61968D3B" Ref="#PWR?"  Part="1"
-AR Path="/602D4838/61968D3B" Ref="#PWR?"  Part="1"
-AR Path="/603B00C8/61968D3B" Ref="#PWR?"  Part="1"
-AR Path="/603B766D/61968D3B" Ref="#PWR?"  Part="1"
-AR Path="/5F74778C/61968D3B" Ref="#PWR042"  Part="1"
-AR Path="/5FB94562/61968D3B" Ref="#PWR?"  Part="1"
-AR Path="/616D5CDC/61968D3B" Ref="#PWR?"  Part="1"
-F 0 "#PWR042" H 3300 3250 50  0001 C CNN
-F 1 "GND" H 3305 3327 50  0000 C CNN
-F 2 "" H 3300 3500 50  0001 C CNN
-F 3 "" H 3300 3500 50  0001 C CNN
-	1    3300 3500
-	1    0    0    -1
-$EndComp
-$Comp
-L 16bitCpu-rescue:GND-power #PWR?
 U 1 1 62492023
 P 4150 3500
@@
 $Comp
 L 16bitCpu-rescue:+5V-power #PWR?
-U 1 1 62492018
-P 1700 3500
-AR Path="/62492018" Ref="#PWR?"  Part="1"
-AR Path="/5F67C726/62492018" Ref="#PWR09"  Part="1"
-AR Path="/5F70885A/62492018" Ref="#PWR?"  Part="1"
-AR Path="/5F733C5E/62492018" Ref="#PWR?"  Part="1"
-AR Path="/602D4838/62492018" Ref="#PWR?"  Part="1"
-AR Path="/603B00C8/62492018" Ref="#PWR?"  Part="1"
-AR Path="/603B766D/62492018" Ref="#PWR?"  Part="1"
-AR Path="/5F74778C/62492018" Ref="#PWR038"  Part="1"
-AR Path="/5FB94562/62492018" Ref="#PWR?"  Part="1"
-AR Path="/616D5CDC/62492018" Ref="#PWR?"  Part="1"
-F 0 "#PWR038" H 1700 3350 50  0001 C CNN
-F 1 "+5V" H 1715 3673 50  0000 C CNN
-F 2 "" H 1700 3500 50  0001 C CNN
-F 3 "" H 1700 3500 50  0001 C CNN
-	1    1700 3500
-	1    0    0    -1
-$EndComp
-$Comp
-L 16bitCpu-rescue:+5V-power #PWR?
 U 1 1 62492019
 P 4400 4850
@@
 F 3 "" H 10050 4300 50  0001 C CNN
 	1    10050 4300
-	1    0    0    -1
-$EndComp
-$Comp
-L 16bitCpu-rescue:+5V-power #PWR?
-U 1 1 5F6AAC6B
-P 5950 3500
-AR Path="/5F6AAC6B" Ref="#PWR?"  Part="1"
-AR Path="/5F67C726/5F6AAC6B" Ref="#PWR022"  Part="1"
-AR Path="/5F70885A/5F6AAC6B" Ref="#PWR?"  Part="1"
-AR Path="/5F733C5E/5F6AAC6B" Ref="#PWR?"  Part="1"
-AR Path="/602D4838/5F6AAC6B" Ref="#PWR?"  Part="1"
-AR Path="/603B00C8/5F6AAC6B" Ref="#PWR?"  Part="1"
-AR Path="/603B766D/5F6AAC6B" Ref="#PWR?"  Part="1"
-AR Path="/5F74778C/5F6AAC6B" Ref="#PWR051"  Part="1"
-AR Path="/5FB94562/5F6AAC6B" Ref="#PWR?"  Part="1"
-AR Path="/616D5CDC/5F6AAC6B" Ref="#PWR?"  Part="1"
-F 0 "#PWR051" H 5950 3350 50  0001 C CNN
-F 1 "+5V" H 5965 3673 50  0000 C CNN
-F 2 "" H 5950 3500 50  0001 C CNN
-F 3 "" H 5950 3500 50  0001 C CNN
-	1    5950 3500
-	1    0    0    -1
-$EndComp
-$Comp
-L 16bitCpu-rescue:GND-power #PWR?
-U 1 1 61968D27
-P 4250 2800
-AR Path="/61968D27" Ref="#PWR?"  Part="1"
-AR Path="/5F67C726/61968D27" Ref="#PWR016"  Part="1"
-AR Path="/5F70885A/61968D27" Ref="#PWR?"  Part="1"
-AR Path="/5F733C5E/61968D27" Ref="#PWR?"  Part="1"
-AR Path="/602D4838/61968D27" Ref="#PWR?"  Part="1"
-AR Path="/603B00C8/61968D27" Ref="#PWR?"  Part="1"
-AR Path="/603B766D/61968D27" Ref="#PWR?"  Part="1"
-AR Path="/5F74778C/61968D27" Ref="#PWR045"  Part="1"
-AR Path="/5FB94562/61968D27" Ref="#PWR?"  Part="1"
-AR Path="/616D5CDC/61968D27" Ref="#PWR?"  Part="1"
-F 0 "#PWR045" H 4250 2550 50  0001 C CNN
-F 1 "GND" H 4255 2627 50  0000 C CNN
-F 2 "" H 4250 2800 50  0001 C CNN
-F 3 "" H 4250 2800 50  0001 C CNN
-	1    4250 2800
 	1    0    0    -1
 $EndComp
@@
 Connection ~ 3600 4350
 Connection ~ 4400 4850
-Connection ~ 2600 4850
 Wire Wire Line
 	10250 3050 10250 7750
